Commit message: Edit location of the images

File: src/mobRobURDF_wizard/mobRobURDF_wizard/classes/temp/2_wheeled_caster/wheels.xacro (robot description, xacro)
@@ -3,5 +3,5 @@
   <!-- Include the inertial_macros.xacro file -->
   <xacro:include filename="$(find mobRobURDF_description)/urdf/macros/inertial_macros.xacro" />
-  <!-- Wheel Macro -->
+  <!-- Wheel Macro (Cylindrical Wheels) -->
   <xacro:macro name="wheel" params="name radius width mass material x y z joint_type">
     <link name="${name}_wheel">
@@ -33,3 +33,32 @@
     </joint>
   </xacro:macro>
+  <!-- Caster Macro (Spherical Wheel) -->
+  <xacro:macro name="caster" params="name radius mass material x y z">
+    <link name="${name}_wheel">
+      <inertial>
+        <mass value="${mass}" />
+        <origin xyz="0 0 0" rpy="0 0 0" />
+        <!-- Use the sphere_inertia macro from inertial_macros.xacro (assumed to exist) -->
+        <xacro:sphere_inertia mass="${mass}" r="${radius}" />
+      </inertial>
+      <visual>
+        <origin xyz="0 0 0" rpy="0 0 0" />
+        <geometry>
+          <sphere radius="${radius}" />
+        </geometry>
+        <material name="${material}" />
+      </visual>
+      <collision>
+        <origin xyz="0 0 0" rpy="0 0 0" />
+        <geometry>
+          <sphere radius="${radius}" />
+        </geometry>
+      </collision>
+    </link>
+    <joint name="${name}_joint" type="fixed">
+      <parent link="chassis" />
+      <child link="${name}_wheel" />
+      <origin xyz="${x} ${y} ${z}" rpy="0 0 0" />
+    </joint>
+  </xacro:macro>
 </robot>

File: src/mobRobURDF_wizard/mobRobURDF_wizard/classes/temp/4_wheeled/wheels.xacro (robot description, xacro)
@@ -4,5 +4,5 @@
   <xacro:include filename="$(find mobRobURDF_description)/urdf/macros/inertial_macros.xacro" />
   <!-- Wheel Macro -->
-  <xacro:macro name="wheel" params="name radius width mass material x y z joint_type">
+  <xacro:macro name="wheel" params="name radius width mass material x y z">
     <link name="${name}_wheel">
       <inertial>
@@ -26,5 +26,5 @@
       </collision>
     </link>
-    <joint name="${name}_joint" type="${joint_type}">
+    <joint name="${name}_joint" type="continuous">
       <parent link="chassis" />
       <child link="${name}_wheel" />
