Commit message: Edited xacro files

File: src/mobRobURDF_description/urdf/macros/inertial_macros.xacro (robot description, xacro)
@@ -14,3 +14,9 @@
              ixy="0" ixz="0" iyz="0" />
   </xacro:macro>
+  <xacro:macro name="sphere_inertia" params="mass r">
+    <inertia ixx="${mass * 2 * r * r / 5}"
+             iyy="${mass * 2 * r * r / 5}"
+             izz="${mass * 2 * r * r / 5}"
+             ixy="0" ixz="0" iyz="0" />
+  </xacro:macro>
 </robot>

File: src/mobRobURDF_description/urdf/submodules/2_wheeled_caster/base.xacro (robot description, xacro)
@@ -1,9 +1,9 @@
 <?xml version="1.0"?>
 <robot xmlns:xacro="http://www.ros.org/wiki/xacro">
-  <!-- Include the inertial_macros.xacro file for 2-wheeled with caster robot -->
+  <!-- Include the inertial_macros.xacro file -->
   <xacro:include filename="$(find mobRobURDF_description)/urdf/macros/inertial_macros.xacro" />
   <!-- Base Link -->
   <link name="base_link"></link>
-  <!-- Chassis -->
+  <!-- Chassis Macro -->
   <xacro:macro name="chassis" params="size mass material">
     <xacro:property name="size_list" value="${list(map(float, size.split()))}" />

File: src/mobRobURDF_description/urdf/submodules/2_wheeled_caster/mobRob.xacro (robot description, xacro)
@@ -13,7 +13,7 @@
   <xacro:chassis size="${chassis_size}" mass="${chassis_mass}" material="${chassis_material}" />
   <!-- Wheels -->
-  <xacro:wheel name="left" radius="${wheel_radius}" width="${wheel_width}" mass="${wheel_mass}" material="${wheel_material}" x="${l_x}" y="${l_y}" z="${l_z}" joint_type="continuous" />
-  <xacro:wheel name="right" radius="${wheel_radius}" width="${wheel_width}" mass="${wheel_mass}" material="${wheel_material}" x="${r_x}" y="${r_y}" z="${r_z}" joint_type="continuous" />
-  <xacro:caster name="front_caster" radius="${caster_radius}" mass="${wheel_mass}" material="${wheel_material}" x="${caster_x}" y="${caster_y}" z="${caster_z}" />
+  <xacro:wheel name="left" radius="${wheel_radius}" width="${wheel_width}" mass="${wheel_mass}" material="${wheel_material}" x="${l_x}" y="${l_y}" z="${l_z}" />
+  <xacro:wheel name="right" radius="${wheel_radius}" width="${wheel_width}" mass="${wheel_mass}" material="${wheel_material}" x="${r_x}" y="${r_y}" z="${r_z}" />
+  <xacro:caster name="front_caster" radius="${wheel_radius}" mass="${wheel_mass}" material="${wheel_material}" x="${caster_x}" y="${caster_y}" z="${caster_z}" />
   <!-- Sensors -->
   <xacro:lidar radius="${lidar_radius}" height="${lidar_height}" mass="${lidar_mass}" material="${lidar_material}" z="${lidar_z}" />

File: src/mobRobURDF_description/urdf/submodules/2_wheeled_caster/sensors.xacro (robot description, xacro)
@@ -1,5 +1,5 @@
 <?xml version="1.0"?>
 <robot xmlns:xacro="http://www.ros.org/wiki/xacro">
-  <!-- Include the inertial_macros.xacro file for 2-wheeled with caster robot -->
+  <!-- Include the inertial_macros.xacro file -->
   <xacro:include filename="$(find mobRobURDF_description)/urdf/macros/inertial_macros.xacro" />
   <!-- Lidar Macro -->

File: src/mobRobURDF_description/urdf/submodules/2_wheeled_caster/wheels.xacro (robot description, xacro)
@@ -3,6 +3,6 @@
   <!-- Include the inertial_macros.xacro file -->
   <xacro:include filename="$(find mobRobURDF_description)/urdf/macros/inertial_macros.xacro" />
-  <!-- Wheel Macro (Cylindrical Wheels) -->
-  <xacro:macro name="wheel" params="name radius width mass material x y z joint_type">
+  <!-- Wheel Macro (Cylindrical) -->
+  <xacro:macro name="wheel" params="name radius width mass material x y z">
     <link name="${name}_wheel">
       <inertial>
@@ -26,5 +26,5 @@
       </collision>
     </link>
-    <joint name="${name}_joint" type="${joint_type}">
+    <joint name="${name}_joint" type="continuous">
       <parent link="chassis" />
       <child link="${name}_wheel" />
@@ -33,5 +33,5 @@
     </joint>
   </xacro:macro>
-  <!-- Caster Macro (Spherical Wheel) -->
+  <!-- Caster Macro (Spherical) -->
   <xacro:macro name="caster" params="name radius mass material x y z">
     <link name="${name}_wheel">

File: src/mobRobURDF_description/urdf/submodules/3_wheeled/base.xacro (robot description, xacro)
@@ -1,5 +1,5 @@
 <?xml version="1.0"?>
 <robot xmlns:xacro="http://www.ros.org/wiki/xacro">
-  <!-- Include the inertial_macros.xacro file for 3-wheeled robot -->
+  <!-- Include the inertial_macros.xacro file -->
   <xacro:include filename="$(find mobRobURDF_description)/urdf/macros/inertial_macros.xacro" />
   <!-- Base Link -->
@@ -11,4 +11,5 @@
     <xacro:property name="w" value="${size_list[1]}" />
     <xacro:property name="h" value="${size_list[2]}" />
+    <!-- Chassis Link -->
     <link name="chassis">
       <inertial>
@@ -37,4 +38,22 @@
       <origin xyz="0 0 ${h/2}" rpy="0 0 0" />
     </joint>
+    <!-- Front Steering Link for 3-Wheeled Robot -->
+    <link name="front_steering_link">
+      <!-- No mass or geometry needed; this is a pivot point for steering -->
+      <inertial>
+        <mass value="0.001" /> <!-- Minimal mass to avoid simulation issues -->
+        <origin xyz="0 0 0" rpy="0 0 0" />
+        <inertia ixx="1e-6" ixy="0" ixz="0" iyy="1e-6" iyz="0" izz="1e-6" />
+      </inertial>
+      <!-- Optional: Add visual/collision if you want a visible steering component -->
+    </link>
+    <!-- Revolute Joint for Steering (z-axis rotation) -->
+    <joint name="chassis_to_front_steering" type="revolute">
+      <parent link="chassis" />
+      <child link="front_steering_link" />
+      <origin xyz="${l/2} 0 ${-h/2}" rpy="0 0 0" /> <!-- Position at front wheel base -->
+      <axis xyz="0 0 1" /> <!-- Rotation around z-axis for steering -->
+      <limit lower="${-pi/2}" upper="${pi/2}" effort="100" velocity="10" /> <!-- Steering range: ±90° -->
+    </joint>
   </xacro:macro>
 </robot>

File: src/mobRobURDF_description/urdf/submodules/3_wheeled/mobRob.xacro (robot description, xacro)
@@ -13,7 +13,7 @@
   <xacro:chassis size="${chassis_size}" mass="${chassis_mass}" material="${chassis_material}" />
   <!-- Wheels -->
-  <xacro:wheel name="front" radius="${wheel_radius}" width="${wheel_width}" mass="${wheel_mass}" material="${wheel_material}" x="${front_x}" y="${front_y}" z="${front_z}" />
-  <xacro:wheel name="rear_left" radius="${wheel_radius}" width="${wheel_width}" mass="${wheel_mass}" material="${wheel_material}" x="${rl_x}" y="${rl_y}" z="${rl_z}" />
-  <xacro:wheel name="rear_right" radius="${wheel_radius}" width="${wheel_width}" mass="${wheel_mass}" material="${wheel_material}" x="${rr_x}" y="${rr_y}" z="${rr_z}" />
+  <xacro:wheel name="front" radius="${wheel_radius}" width="${wheel_width}" mass="${wheel_mass}" material="${wheel_material}" x="0" y="0" z="0" parent="front_steering_link" />
+  <xacro:wheel name="rear_left" radius="${wheel_radius}" width="${wheel_width}" mass="${wheel_mass}" material="${wheel_material}" x="${rl_x}" y="${rl_y}" z="${rl_z}" parent="chassis" />
+  <xacro:wheel name="rear_right" radius="${wheel_radius}" width="${wheel_width}" mass="${wheel_mass}" material="${wheel_material}" x="${rr_x}" y="${rr_y}" z="${rr_z}" parent="chassis" />
   <!-- Sensors -->
   <xacro:lidar radius="${lidar_radius}" height="${lidar_height}" mass="${lidar_mass}" material="${lidar_material}" z="${lidar_z}" />

File: src/mobRobURDF_description/urdf/submodules/3_wheeled/sensors.xacro (robot description, xacro)
@@ -1,5 +1,5 @@
 <?xml version="1.0"?>
 <robot xmlns:xacro="http://www.ros.org/wiki/xacro">
-  <!-- Include the inertial_macros.xacro file for 3-wheeled robot -->
+  <!-- Include the inertial_macros.xacro file -->
   <xacro:include filename="$(find mobRobURDF_description)/urdf/macros/inertial_macros.xacro" />
   <!-- Lidar Macro -->

File: src/mobRobURDF_description/urdf/submodules/3_wheeled/wheels.xacro (robot description, xacro)
@@ -4,5 +4,5 @@
   <xacro:include filename="$(find mobRobURDF_description)/urdf/macros/inertial_macros.xacro" />
   <!-- Wheel Macro -->
-  <xacro:macro name="wheel" params="name radius width mass material x y z joint_type">
+  <xacro:macro name="wheel" params="name radius width mass material x y z parent">
     <link name="${name}_wheel">
       <inertial>
@@ -26,6 +26,6 @@
       </collision>
     </link>
-    <joint name="${name}_joint" type="${joint_type}">
-      <parent link="chassis" />
+    <joint name="${name}_joint" type="continuous">
+      <parent link="${parent}" />
       <child link="${name}_wheel" />
       <origin xyz="${x} ${y} ${z}" rpy="0 0 0" />

File: src/mobRobURDF_description/urdf/submodules/4_wheeled/base.xacro (robot description, xacro)
@@ -5,5 +5,5 @@
   <!-- Base Link -->
   <link name="base_link"></link>
-  <!-- Chassis -->
+  <!-- Chassis Macro -->
   <xacro:macro name="chassis" params="size mass material">
     <xacro:property name="size_list" value="${list(map(float, size.split()))}" />

File: src/mobRobURDF_wizard/mobRobURDF_wizard/classes/temp/2_wheeled_caster/mobRob.xacro (robot description, xacro)
@@ -11,11 +11,11 @@
   <xacro:define_materials/>
   <!-- Define the robot -->
-  <xacro:chassis size="1 1 1" mass="1.0" material="Gray" />
+  <xacro:chassis size="1.2 0.8 0.3" mass="1.0" material="Gray" />
   <!-- Wheels -->
-  <xacro:wheel name="left" radius="0.22" width="0.12" mass="0.5" material="Black" x="0" y="0.56" z="-0.5" joint_type="continuous" />
-  <xacro:wheel name="right" radius="0.22" width="0.12" mass="0.5" material="Black" x="0" y="-0.56" z="-0.5" joint_type="continuous" />
-  <xacro:caster name="front_caster" radius="1 1 1" mass="0.5" material="Black" x="0.5" y="0" z="-0.5" />
+  <xacro:wheel name="left" radius="0.1" width="0.12" mass="0.5" material="Black" x="0" y="0.46" z="-0.15" />
+  <xacro:wheel name="right" radius="0.1" width="0.12" mass="0.5" material="Black" x="0" y="-0.46" z="-0.15" />
+  <xacro:caster name="front_caster" radius="0.1" mass="0.5" material="Black" x="0.6" y="0" z="-0.15" />
   <!-- Sensors -->
-  <xacro:lidar radius="0.1" height="0.08" mass="0.2" material="Red" z="0.54" />
-  <xacro:camera size="0.08 0.2 0.08" mass="0.1" material="Blue" x="0.54" />
+  <xacro:lidar radius="0.1" height="0.08" mass="0.2" material="Red" z="0.19" />
+  <xacro:camera size="0.08 0.2 0.08" mass="0.1" material="Blue" x="0.64" />
 </robot>

File: src/mobRobURDF_wizard/mobRobURDF_wizard/classes/temp/3_wheeled/mobRob.xacro (robot description, xacro)
@@ -11,11 +11,11 @@
   <xacro:define_materials/>
   <!-- Define the robot -->
-  <xacro:chassis size="1 1 1" mass="1.0" material="Gray" />
+  <xacro:chassis size="1.2 0.8 0.3" mass="1.0" material="Gray" />
   <!-- Wheels -->
-  <xacro:wheel name="front" radius="0.22" width="0.12" mass="0.5" material="Black" x="0.5" y="0" z="-0.5" />
-  <xacro:wheel name="rear_left" radius="0.22" width="0.12" mass="0.5" material="Black" x="-0.5" y="0.56" z="-0.5" />
-  <xacro:wheel name="rear_right" radius="0.22" width="0.12" mass="0.5" material="Black" x="-0.5" y="-0.56" z="-0.5" />
+  <xacro:wheel name="front" radius="0.22" width="0.12" mass="0.5" material="1 1 1" x="0" y="0" z="0" parent="front_steering_link" />
+  <xacro:wheel name="rear_left" radius="0.22" width="0.12" mass="0.5" material="1 1 1" x="-0.6" y="0.46" z="-0.15" parent="chassis" />
+  <xacro:wheel name="rear_right" radius="0.22" width="0.12" mass="0.5" material="1 1 1" x="-0.6" y="-0.46" z="-0.15" parent="chassis" />
   <!-- Sensors -->
-  <xacro:lidar radius="0.1" height="0.08" mass="0.2" material="Red" z="0.54" />
-  <xacro:camera size="0.08 0.2 0.08" mass="0.1" material="Blue" x="0.54" />
+  <xacro:lidar radius="0.4" height="0.1" mass="0.2" material="Red" z="0.2" />
+  <xacro:camera size="0.08 0.2 0.08" mass="0.1" material="Red" x="0.64" />
 </robot>
