Commit message: Added more colors (materials) and a drop-down menu for choosing them

File: src/mobRobURDF_description/urdf/macros/material_macros.xacro (robot description, xacro)
@@ -1,24 +1,23 @@
 <?xml version="1.0"?>
 <robot xmlns:xacro="http://www.ros.org/wiki/xacro">
-  <!-- Define Material Colors -->
   <xacro:macro name="define_materials">
-    <material name="Gray">
-      <color rgba="0.5 0.5 0.5 1.0"/>
-    </material>
-    <material name="Black">
-      <color rgba="0.0 0.0 0.0 1.0"/>
-    </material>
-    <material name="Red">
-      <color rgba="1.0 0.0 0.0 1.0"/>
-    </material>
-    <material name="Blue">
-      <color rgba="0.0 0.0 1.0 1.0"/>
-    </material>
-    <material name="Green">
-      <color rgba="0.0 1.0 0.0 1.0"/>
-    </material>
-    <material name="White">
-      <color rgba="1.0 1.0 1.0 1.0"/>
-    </material>
+    <material name="Gray">      <color rgba="0.50 0.50 0.50 1.0"/> </material>
+    <material name="Silver">    <color rgba="0.75 0.75 0.75 1.0"/> </material>
+    <material name="Dark Gray"> <color rgba="0.25 0.25 0.25 1.0"/> </material>
+    <material name="Black">     <color rgba="0.00 0.00 0.00 1.0"/> </material>
+    <material name="White">     <color rgba="1.00 1.00 1.00 1.0"/> </material>
+    <material name="Red">       <color rgba="1.00 0.00 0.00 1.0"/> </material>
+    <material name="Maroon">    <color rgba="0.50 0.00 0.00 1.0"/> </material>
+    <material name="Orange">    <color rgba="1.00 0.50 0.00 1.0"/> </material>
+    <material name="Yellow">    <color rgba="1.00 1.00 0.00 1.0"/> </material>
+    <material name="Green">     <color rgba="0.00 0.80 0.00 1.0"/> </material>
+    <material name="Lime">      <color rgba="0.50 1.00 0.00 1.0"/> </material>
+    <material name="Teal">      <color rgba="0.00 0.50 0.50 1.0"/> </material>
+    <material name="Cyan">      <color rgba="0.00 1.00 1.00 1.0"/> </material>
+    <material name="Blue">      <color rgba="0.00 0.00 1.00 1.0"/> </material>
+    <material name="Navy">      <color rgba="0.00 0.00 0.50 1.0"/> </material>
+    <material name="Purple">    <color rgba="0.50 0.00 0.50 1.0"/> </material>
+    <material name="Pink">      <color rgba="1.00 0.40 0.70 1.0"/> </material>
+    <material name="Brown">     <color rgba="0.60 0.30 0.10 1.0"/> </material>
   </xacro:macro>
 </robot>

File: src/mobRobURDF_description/urdf/mobRob.urdf.xacro (robot description, xacro)
@@ -9,20 +9,18 @@
   <xacro:property name="wheel_mass" value="0.5"/>
   <xacro:property name="wheel_material" value="Black"/>
-  <xacro:property name="fl_x" value="0.4533333333333333"/>
-  <xacro:property name="fl_y" value="0.46"/>
-  <xacro:property name="fl_z" value="-0.15"/>
-  <xacro:property name="fr_x" value="0.4533333333333333"/>
-  <xacro:property name="fr_y" value="-0.46"/>
-  <xacro:property name="fr_z" value="-0.15"/>
-  <xacro:property name="rl_x" value="-0.4533333333333333"/>
-  <xacro:property name="rl_y" value="0.46"/>
-  <xacro:property name="rl_z" value="-0.15"/>
-  <xacro:property name="rr_x" value="-0.4533333333333333"/>
-  <xacro:property name="rr_y" value="-0.46"/>
-  <xacro:property name="rr_z" value="-0.15"/>
-  <xacro:property name="controller_type" value="mecanum"/>
+  <xacro:property name="caster_radius" value="0.22"/>
+  <xacro:property name="l_x" value="-0.3"/>
+  <xacro:property name="l_y" value="0.46"/>
+  <xacro:property name="l_z" value="-0.15"/>
+  <xacro:property name="r_x" value="-0.3"/>
+  <xacro:property name="r_y" value="-0.46"/>
+  <xacro:property name="r_z" value="-0.15"/>
+  <xacro:property name="caster_x" value="0.38"/>
+  <xacro:property name="caster_y" value="0"/>
+  <xacro:property name="caster_z" value="-0.15"/>
+  <xacro:property name="controller_type" value="diff_2wc"/>
   <xacro:property name="hardware_plugin" value="gz_ros2_control/GazeboSimSystem"/>
   <xacro:property name="use_gazebo_sim" value="1"/>
-  <xacro:include filename="$(find mobRobURDF_description)/urdf/submodules/4_wheeled/mobRob_4w_mec.xacro"/>
+  <xacro:include filename="$(find mobRobURDF_description)/urdf/submodules/2_wheeled_caster/mobRob_2wc_diff.xacro"/>
   <xacro:include filename="$(find mobRobURDF_description)/urdf/user_sensors.xacro"/>
 </robot>
