Commit message: Modified (and created) gazebo ros2 control files.

File: src/mobRobURDF_description/urdf/gazebo_files/control/gazebo_ros2_control_4w_acker.xacro (robot description, xacro)
@@ -5,5 +5,5 @@
             <plugin>gazebo_ros2_control/GazeboSystem</plugin>
         </hardware>
-        <joint name="left_joint">
+        <joint name="rear_left_joint">
             <command_interface name="velocity">
                 <param name="min">-50</param>
@@ -13,5 +13,5 @@
             <state_interface name="position"/>
         </joint>
-        <joint name="right_joint">
+        <joint name="rear_right_joint">
             <command_interface name="velocity">
                 <param name="min">-50</param>
@@ -21,19 +21,30 @@
             <state_interface name="position"/>
         </joint>
+        <joint name="chassis_to_front_left_steering">
+            <command_interface name="position">
+                <param name="min">-0.785</param>
+                <param name="max">0.785</param>
+            </command_interface>
+            <state_interface name="velocity"/>
+            <state_interface name="position"/>
+        </joint>
+        <joint name="chassis_to_front_right_steering">
+            <command_interface name="position">
+                <param name="min">-0.785</param>
+                <param name="max">0.785</param>
+            </command_interface>
+            <state_interface name="velocity"/>
+            <state_interface name="position"/>
+        </joint>
         <!-- - - - Not-motorized - - - -->
-        <joint name="front_caster_joint">
+        <joint name="front_left_joint">
             <command_interface name="velocity"></command_interface>
+            <state_interface name="velocity"/>
             <state_interface name="position"/>
+        </joint>
+        <joint name="front_right_joint">
+            <command_interface name="velocity"></command_interface>
             <state_interface name="velocity"/>
-        </joint>
-        <joint name="rotating_x_joint">
-            <command_interface name="velocity"></command_interface>
             <state_interface name="position"/>
-            <state_interface name="velocity"/>
-        </joint>
-        <joint name="rotating_y_joint">
-            <command_interface name="velocity"></command_interface>
-            <state_interface name="position"/>
-            <state_interface name="velocity"/>
         </joint>
         <!-- - - - - - - - - - - - - - -->
@@ -41,5 +52,5 @@
     <gazebo>
         <plugin name="gazebo_ros2_control" filename="libgazebo_ros2_control.so">
-            <parameters>$(find mobRobURDF_control)/config/drive/gazebo_controller_diffDrive_2wd_caster.yaml</parameters>
+            <parameters>$(find mobRobURDF_control)/config/steer/gazebo_controller_ackerSteer.yaml</parameters>
         </plugin>
     </gazebo>

File: src/mobRobURDF_description/urdf/gazebo_files/control/gazebo_ros2_control_4w_mec.xacro (robot description, xacro)
@@ -5,4 +5,20 @@
             <plugin>gazebo_ros2_control/GazeboSystem</plugin>
         </hardware>
+        <joint name="front_left_joint">
+            <command_interface name="velocity">
+                <param name="min">-50</param>
+                <param name="max">50</param>
+            </command_interface>
+            <state_interface name="velocity"/>
+            <state_interface name="position"/>
+        </joint>
+        <joint name="front_right_joint">
+            <command_interface name="velocity">
+                <param name="min">-50</param>
+                <param name="max">50</param>
+            </command_interface>
+            <state_interface name="velocity"/>
+            <state_interface name="position"/>
+        </joint>
         <joint name="rear_left_joint">
             <command_interface name="velocity">
@@ -21,25 +37,9 @@
             <state_interface name="position"/>
         </joint>
-        <joint name="front_joint">
-            <command_interface name="velocity">
-                <param name="min">-50</param>
-                <param name="max">50</param>
-            </command_interface>
-            <state_interface name="velocity"/>
-            <state_interface name="position"/>
-        </joint>
-        <joint name="chassis_to_front_steering">
-            <command_interface name="position">
-                <param name="min">-1.57</param>
-                <param name="max">1.57</param>
-            </command_interface>
-            <state_interface name="velocity"/>
-            <state_interface name="position"/>
-        </joint>
         <!-- - - - - - - - - - - - - - -->
     </ros2_control>
     <gazebo>
         <plugin name="gazebo_ros2_control" filename="libgazebo_ros2_control.so">
-            <parameters>$(find mobRobURDF_control)/config/gazebo_controller_tricycle.yaml</parameters>
+            <parameters>$(find mobRobURDF_control)/config/drive/gazebo_controller_mecDrive.yaml</parameters>
         </plugin>
     </gazebo>

File: src/mobRobURDF_description/urdf/submodules/2_wheeled_caster/mobRob.xacro (robot description, xacro)
@@ -7,5 +7,4 @@
   <xacro:include filename="$(find mobRobURDF_description)/urdf/macros/inertial_macros.xacro" />
   <xacro:include filename="$(find mobRobURDF_description)/urdf/macros/material_macros.xacro" />
-  <!-- <xacro:include filename="$(find mobRobURDF_description)/urdf/gazebo_files/gazebo_sensors.xacro" /> -->
   <!-- Call the macro to define materials -->
   <xacro:define_materials/>
@@ -19,3 +18,7 @@
   <xacro:lidar radius="${lidar_radius}" height="${lidar_height}" mass="${lidar_mass}" material="${lidar_material}" z="${lidar_z}" />
   <xacro:camera size="${camera_size}" mass="${camera_mass}" material="${camera_material}" x="${camera_x}" />
+  <!-- Include Gazebo Xacro files -->
+  <xacro:include filename="$(find mobRobURDF_description)/urdf/gazebo_files/control/gazebo_ros2_control_4w.xacro" />
+  <xacro:include filename="$(find mobRobURDF_description)/urdf/gazebo_files/gazebo_properties.xacro" />
+  <xacro:include filename="$(find mobRobURDF_description)/urdf/gazebo_files/gazebo_sensors.xacro" />
 </robot>
