Commit message: Fixed the issue with steering joints in tricycle kinematics

File: src/mobRobURDF_description/urdf/gazebo_files/control/gazebo_ros2_control_3w_triSteer.xacro (robot description, xacro)
@@ -29,7 +29,6 @@
             <state_interface name="position"/>
         </joint>
-        <!-- - - - Not-motorized - - - -->
+        <!-- Passive front wheel: state interfaces only — no command so gz rolls it freely -->
         <joint name="front_joint">
-            <command_interface name="velocity"></command_interface>
             <state_interface name="velocity"/>
             <state_interface name="position"/>

File: src/mobRobURDF_description/urdf/gazebo_files/control/gazebo_ros2_control_3w_tricycle.xacro (robot description, xacro)
@@ -21,12 +21,10 @@
             <state_interface name="position"/>
         </joint>
-        <!-- - - - Not-motorized - - - -->
+        <!-- Passive rear wheels: state interfaces only — no command so gz rolls them freely -->
         <joint name="rear_left_joint">
-            <command_interface name="velocity"></command_interface>
             <state_interface name="velocity"/>
             <state_interface name="position"/>
         </joint>
         <joint name="rear_right_joint">
-            <command_interface name="velocity"></command_interface>
             <state_interface name="velocity"/>
             <state_interface name="position"/>

File: src/mobRobURDF_description/urdf/mobRob.urdf (robot description, URDF)
Before this commit: robot mobRob, 12 links, 11 joints
Links:
- removed link camera_2
- removed link camera_2_optical
- removed link front_steering_link
- removed link front_wheel
- removed link lidar_2
- added link front_left_wheel, mass 0.5; collision cylinder length=0.12 radius=0.22; visual cylinder length=0.12 radius=0.22
- added link front_right_wheel, mass 0.5; collision cylinder length=0.12 radius=0.22; visual cylinder length=0.12 radius=0.22
Joints:
- removed joint camera_2_joint
- removed joint camera_2_optical_joint
- removed joint chassis_to_front_steering
- removed joint front_joint
- removed joint lidar_2_joint
- added joint front_left_joint: type continuous, parent chassis, child front_left_wheel, origin xyz=0.4533333333333333 0.46 -0.15 rpy=0 0 0, axis 0 1 0
- added joint front_right_joint: type continuous, parent chassis, child front_right_wheel, origin xyz=0.4533333333333333 -0.46 -0.15 rpy=0 0 0, axis 0 1 0

File: src/mobRobURDF_description/urdf/mobRob.urdf.xacro (robot description, xacro)
@@ -9,7 +9,10 @@
   <xacro:property name="wheel_mass" value="0.5"/>
   <xacro:property name="wheel_material" value="Black"/>
-  <xacro:property name="front_x" value="0.6"/>
-  <xacro:property name="front_y" value="0"/>
-  <xacro:property name="front_z" value="-0.15"/>
+  <xacro:property name="fl_x" value="0.4533333333333333"/>
+  <xacro:property name="fl_y" value="0.46"/>
+  <xacro:property name="fl_z" value="-0.15"/>
+  <xacro:property name="fr_x" value="0.4533333333333333"/>
+  <xacro:property name="fr_y" value="-0.46"/>
+  <xacro:property name="fr_z" value="-0.15"/>
   <xacro:property name="rl_x" value="-0.4533333333333333"/>
   <xacro:property name="rl_y" value="0.46"/>
@@ -18,6 +21,6 @@
   <xacro:property name="rr_y" value="-0.46"/>
   <xacro:property name="rr_z" value="-0.15"/>
-  <xacro:property name="controller_type" value="triSteer"/>
-  <xacro:include filename="$(find mobRobURDF_description)/urdf/submodules/3_wheeled/mobRob_3w_triSteer.xacro"/>
+  <xacro:property name="controller_type" value="mecanum"/>
+  <xacro:include filename="$(find mobRobURDF_description)/urdf/submodules/4_wheeled/mobRob_4w_mec.xacro"/>
   <xacro:include filename="$(find mobRobURDF_description)/urdf/user_sensors.xacro"/>
 </robot>

Commit message: Fixed the kinematics that didn't publish odom tf and topic

File: src/mobRobURDF_description/urdf/gazebo_files/control/gazebo_ros2_control_3w_triSteer.xacro (robot description, xacro)
@@ -39,4 +39,10 @@
         <plugin name="gz_ros2_control::GazeboSimROS2ControlPlugin" filename="libgz_ros2_control-system.so">
             <parameters>$(find mobRobURDF_control)/config/steer/gazebo_controller_triSteer.yaml</parameters>
+            <ros>
+                <!-- tricycle_steering_controller publishes to ~/tf_odometry and ~/odometry,
+                     not to /tf and /odom. Remap to the standard global topics. -->
+                <remapping>/triSteer_controller/tf_odometry:=/tf</remapping>
+                <remapping>/triSteer_controller/odometry:=/odom</remapping>
+            </ros>
         </plugin>
     </gazebo>

File: src/mobRobURDF_description/urdf/gazebo_files/control/gazebo_ros2_control_4w_acker.xacro (robot description, xacro)
@@ -51,4 +51,10 @@
         <plugin name="gz_ros2_control::GazeboSimROS2ControlPlugin" filename="libgz_ros2_control-system.so">
             <parameters>$(find mobRobURDF_control)/config/steer/gazebo_controller_ackerSteer.yaml</parameters>
+            <ros>
+                <!-- ackermann_steering_controller publishes to ~/tf_odometry and ~/odometry,
+                     not to /tf and /odom. Remap to the standard global topics. -->
+                <remapping>/ackerSteer_controller/tf_odometry:=/tf</remapping>
+                <remapping>/ackerSteer_controller/odometry:=/odom</remapping>
+            </ros>
         </plugin>
     </gazebo>

File: src/mobRobURDF_description/urdf/gazebo_files/control/gazebo_ros2_control_4w_mec.xacro (robot description, xacro)
@@ -42,4 +42,10 @@
         <plugin name="gz_ros2_control::GazeboSimROS2ControlPlugin" filename="libgz_ros2_control-system.so">
             <parameters>$(find mobRobURDF_control)/config/drive/gazebo_controller_mecDrive.yaml</parameters>
+            <ros>
+                <!-- mecanum_drive_controller publishes to ~/tf_odometry and ~/odometry,
+                     not to /tf and /odom. Remap to the standard global topics. -->
+                <remapping>/mecDrive_controller/tf_odometry:=/tf</remapping>
+                <remapping>/mecDrive_controller/odometry:=/odom</remapping>
+            </ros>
         </plugin>
     </gazebo>

File: src/mobRobURDF_description/urdf/mobRob.urdf (robot description, URDF)
Before this commit: robot mobRob, 9 links, 8 joints
Links:
- added link front_left_steering_link, mass 0.001
- added link front_right_steering_link, mass 0.001
Joints:
- added joint chassis_to_front_left_steering: type revolute, parent chassis, child front_left_steering_link, origin xyz=0.4533333333333333 0.46 -0.15 rpy=0 0 0, axis 0 0 1, limit lower=-0.7853981633974483 upper=0.7853981633974483 effort=100 velocity=10
- added joint chassis_to_front_right_steering: type revolute, parent chassis, child front_right_steering_link, origin xyz=0.4533333333333333 -0.46 -0.15 rpy=0 0 0, axis 0 0 1, limit lower=-0.7853981633974483 upper=0.7853981633974483 effort=100 velocity=10
- joint front_left_joint: origin xyz=0.4533333333333333 0.46 -0.15 rpy=0 0 0 -> xyz=0 0 0 rpy=0 0 0; parent chassis -> front_left_steering_link
- joint front_right_joint: origin xyz=0.4533333333333333 -0.46 -0.15 rpy=0 0 0 -> xyz=0 0 0 rpy=0 0 0; parent chassis -> front_right_steering_link

File: src/mobRobURDF_description/urdf/mobRob.urdf.xacro (robot description, xacro)
@@ -21,6 +21,6 @@
   <xacro:property name="rr_y" value="-0.46"/>
   <xacro:property name="rr_z" value="-0.15"/>
-  <xacro:property name="controller_type" value="mecanum"/>
-  <xacro:include filename="$(find mobRobURDF_description)/urdf/submodules/4_wheeled/mobRob_4w_mec.xacro"/>
+  <xacro:property name="controller_type" value="ackermann"/>
+  <xacro:include filename="$(find mobRobURDF_description)/urdf/submodules/4_wheeled/ackermann/mobRob_4w_acker.xacro"/>
   <xacro:include filename="$(find mobRobURDF_description)/urdf/user_sensors.xacro"/>
 </robot>
