Commit message: Modified xacro files (for controllers).

File: src/mobRobURDF_description/urdf/gazebo_files/control/gazebo_ros2_control_2wc_diff.xacro (robot description, xacro)
@@ -3,5 +3,5 @@
     <ros2_control name="GazeboSystem" type="system">
         <hardware>
-            <plugin>gazebo_ros2_control/GazeboSystem</plugin>
+            <plugin>gz_ros2_control/GazeboSimSystem</plugin>
         </hardware>
         <joint name="left_joint">
@@ -40,5 +40,5 @@
     </ros2_control>
     <gazebo>
-        <plugin name="gazebo_ros2_control" filename="libgazebo_ros2_control.so">
+        <plugin name="gz_ros2_control::GazeboSimROS2ControlPlugin" filename="libgz_ros2_control-system.so">
             <parameters>$(find mobRobURDF_control)/config/drive/gazebo_controller_diffDrive_2wd_caster.yaml</parameters>
         </plugin>

File: src/mobRobURDF_description/urdf/gazebo_files/control/gazebo_ros2_control_3w_triSteer.xacro (robot description, xacro)
@@ -3,5 +3,5 @@
     <ros2_control name="GazeboSystem" type="system">
         <hardware>
-            <plugin>gazebo_ros2_control/GazeboSystem</plugin>
+            <plugin>gz_ros2_control/GazeboSimSystem</plugin>
         </hardware>
         <joint name="rear_left_joint">
@@ -38,5 +38,5 @@
     </ros2_control>
     <gazebo>
-        <plugin name="gazebo_ros2_control" filename="libgazebo_ros2_control.so">
+        <plugin name="gz_ros2_control::GazeboSimROS2ControlPlugin" filename="libgz_ros2_control-system.so">
             <parameters>$(find mobRobURDF_control)/config/steer/gazebo_controller_triSteer.yaml</parameters>
         </plugin>

File: src/mobRobURDF_description/urdf/gazebo_files/control/gazebo_ros2_control_3w_tricycle.xacro (robot description, xacro)
@@ -3,5 +3,5 @@
     <ros2_control name="GazeboSystem" type="system">
         <hardware>
-            <plugin>gazebo_ros2_control/GazeboSystem</plugin>
+            <plugin>gz_ros2_control/GazeboSimSystem</plugin>
         </hardware>
         <joint name="front_joint">
@@ -35,5 +35,5 @@
     </ros2_control>
     <gazebo>
-        <plugin name="gazebo_ros2_control" filename="libgazebo_ros2_control.so">
+        <plugin name="gz_ros2_control::GazeboSimROS2ControlPlugin" filename="libgz_ros2_control-system.so">
             <parameters>$(find mobRobURDF_control)/config/gazebo_controller_tricycle.yaml</parameters>
         </plugin>

File: src/mobRobURDF_description/urdf/gazebo_files/control/gazebo_ros2_control_4w_acker.xacro (robot description, xacro)
@@ -3,5 +3,5 @@
     <ros2_control name="GazeboSystem" type="system">
         <hardware>
-            <plugin>gazebo_ros2_control/GazeboSystem</plugin>
+            <plugin>gz_ros2_control/GazeboSimSystem</plugin>
         </hardware>
         <joint name="rear_left_joint">
@@ -51,5 +51,5 @@
     </ros2_control>
     <gazebo>
-        <plugin name="gazebo_ros2_control" filename="libgazebo_ros2_control.so">
+        <plugin name="gz_ros2_control::GazeboSimROS2ControlPlugin" filename="libgz_ros2_control-system.so">
             <parameters>$(find mobRobURDF_control)/config/steer/gazebo_controller_ackerSteer.yaml</parameters>
         </plugin>

File: src/mobRobURDF_description/urdf/gazebo_files/control/gazebo_ros2_control_4w_diff.xacro (robot description, xacro)
@@ -3,5 +3,5 @@
     <ros2_control name="GazeboSystem" type="system">
         <hardware>
-            <plugin>gazebo_ros2_control/GazeboSystem</plugin>
+            <plugin>gz_ros2_control/GazeboSimSystem</plugin>
         </hardware>
         <joint name="front_left_joint">
@@ -40,5 +40,5 @@
     </ros2_control>
     <gazebo>
-        <plugin name="gazebo_ros2_control" filename="libgazebo_ros2_control.so">
+        <plugin name="gz_ros2_control::GazeboSimROS2ControlPlugin" filename="libgz_ros2_control-system.so">
             <parameters>$(find mobRobURDF_control)/config/drive/gazebo_controller_diffDrive_4wd.yaml</parameters>
         </plugin>

File: src/mobRobURDF_description/urdf/gazebo_files/control/gazebo_ros2_control_4w_mec.xacro (robot description, xacro)
@@ -3,5 +3,5 @@
     <ros2_control name="GazeboSystem" type="system">
         <hardware>
-            <plugin>gazebo_ros2_control/GazeboSystem</plugin>
+            <plugin>gz_ros2_control/GazeboSimSystem</plugin>
         </hardware>
         <joint name="front_left_joint">
@@ -40,5 +40,5 @@
     </ros2_control>
     <gazebo>
-        <plugin name="gazebo_ros2_control" filename="libgazebo_ros2_control.so">
+        <plugin name="gz_ros2_control::GazeboSimROS2ControlPlugin" filename="libgz_ros2_control-system.so">
             <parameters>$(find mobRobURDF_control)/config/drive/gazebo_controller_mecDrive.yaml</parameters>
         </plugin>

File: src/mobRobURDF_description/urdf/gazebo_files/gazebo_properties.xacro (robot description, xacro)
@@ -1,8 +1,356 @@
 <?xml version="1.0"?>
-<robot xmlns:xacro="http://www.ros.org/wiki/xacro">
-    <gazebo reference="chassis">
-        <material>Gazebo/Gray</material>
-        <turnGravityOff>false</turnGravityOff>
-        <visible>true</visible>
+<robot xmlns:xacro="http://ros.org/wiki/xacro">
+  <!-- Macro for Gazebo physical properties -->
+  <xacro:macro name="gazebo_physical_properties" params="controller_type chassis_size wheel_radius wheel_width">
+    <!-- Extract parameters -->
+    <xacro:property name="L" value="${float(chassis_size.split()[0])}"/>
+    <xacro:property name="W" value="${float(chassis_size.split()[1])}"/>
+    <xacro:property name="wheel_radius" value="${float(wheel_radius)}"/>
+    <xacro:property name="wheel_width" value="${float(wheel_width)}"/>
+    <!-- Base link properties (common for all controllers) -->
+    <gazebo reference="base_link">
+      <collision>
+        <surface>
+          <friction>
+            <ode>
+              <mu>0.8</mu>
+              <mu2>0.8</mu2>
+            </ode>
+          </friction>
+          <contact>
+            <kp>1e6</kp>
+            <kd>1.0</kd>
+            <max_vel>0.1</max_vel>
+            <min_depth>0.001</min_depth>
+          </contact>
+          <bounce>
+            <restitution_coefficient>0.0</restitution_coefficient>
+          </bounce>
+        </surface>
+      </collision>
     </gazebo>
+    <!-- diff_2wc: 2-wheeled with caster -->
+    <xacro:if value="${controller_type == 'diff_2wc'}">
+      <!-- Drive wheels -->
+      <xacro:macro name="drive_wheel_properties" params="wheel_link wheel_joint">
+        <gazebo reference="${wheel_link}">
+          <collision>
+            <surface>
+              <friction>
+                <ode>
+                  <mu>1.0</mu>
+                  <mu2>1.0</mu2>
+                </ode>
+              </friction>
+              <contact>
+                <kp>1e6</kp>
+                <kd>1.0</kd>
+                <max_vel>0.1</max_vel>
+                <min_depth>0.001</min_depth>
+              </contact>
+              <bounce>
+                <restitution_coefficient>0.0</restitution_coefficient>
+              </bounce>
+            </surface>
+          </collision>
+        </gazebo>
+        <gazebo reference="${wheel_joint}">
+          <damping>0.1</damping>
+        </gazebo>
+      </xacro:macro>
+      <xacro:drive_wheel_properties wheel_link="left_wheel" wheel_joint="left_joint"/>
+      <xacro:drive_wheel_properties wheel_link="right_wheel" wheel_joint="right_joint"/>
+      <!-- Caster -->
+      <gazebo reference="front_caster">
+        <collision>
+          <surface>
+            <friction>
+              <ode>
+                <mu>0.1</mu>
+                <mu2>0.1</mu2>
+              </ode>
+            </friction>
+            <contact>
+              <kp>1e6</kp>
+              <kd>1.0</kd>
+              <max_vel>0.1</max_vel>
+              <min_depth>0.001</min_depth>
+            </contact>
+            <bounce>
+              <restitution_coefficient>0.0</restitution_coefficient>
+            </bounce>
+          </surface>
+        </collision>
+      </gazebo>
+      <gazebo reference="free-rotating_x_joint">
+        <damping>0.01</damping>
+      </gazebo>
+      <gazebo reference="free-rotating_y_joint">
+        <damping>0.01</damping>
+      </gazebo>
+      <gazebo reference="front_caster_joint">
+        <damping>0.01</damping>
+      </gazebo>
+    </xacro:if>
+    <!-- diff_4w: 4-wheeled differential -->
+    <xacro:if value="${controller_type == 'diff_4w'}">
+      <xacro:macro name="drive_wheel_properties" params="wheel_link wheel_joint">
+        <gazebo reference="${wheel_link}">
+          <collision>
+            <surface>
+              <friction>
+                <ode>
+                  <mu>1.0</mu>
+                  <mu2>1.0</mu2>
+                </ode>
+              </friction>
+              <contact>
+                <kp>1e6</kp>
+                <kd>1.0</kd>
+                <max_vel>0.1</max_vel>
+                <min_depth>0.001</min_depth>
+              </contact>
+              <bounce>
+                <restitution_coefficient>0.0</restitution_coefficient>
+              </bounce>
+            </surface>
+          </collision>
+        </gazebo>
+        <gazebo reference="${wheel_joint}">
+          <damping>0.1</damping>
+        </gazebo>
+      </xacro:macro>
+      <xacro:drive_wheel_properties wheel_link="front_left_wheel" wheel_joint="front_left_joint"/>
+      <xacro:drive_wheel_properties wheel_link="front_right_wheel" wheel_joint="front_right_joint"/>
+      <xacro:drive_wheel_properties wheel_link="rear_left_wheel" wheel_joint="rear_left_joint"/>
+      <xacro:drive_wheel_properties wheel_link="rear_right_wheel" wheel_joint="rear_right_joint"/>
+    </xacro:if>
+    <!-- mecanum: 4-wheeled mecanum -->
+    <xacro:if value="${controller_type == 'mecanum'}">
+      <xacro:macro name="mecanum_wheel_properties" params="wheel_link wheel_joint">
+        <gazebo reference="${wheel_link}">
+          <collision>
+            <surface>
+              <friction>
+                <ode>
+                  <mu>1.2</mu>
+                  <mu2>1.2</mu2>
+                </ode>
+              </friction>
+              <contact>
+                <kp>1e6</kp>
+                <kd>1.0</kd>
+                <max_vel>0.1</max_vel>
+                <min_depth>0.001</min_depth>
+              </contact>
+              <bounce>
+                <restitution_coefficient>0.0</restitution_coefficient>
+              </bounce>
+            </surface>
+          </collision>
+        </gazebo>
+        <gazebo reference="${wheel_joint}">
+          <damping>0.15</damping>
+        </gazebo>
+      </xacro:macro>
+      <xacro:mecanum_wheel_properties wheel_link="front_left_wheel" wheel_joint="front_left_joint"/>
+      <xacro:mecanum_wheel_properties wheel_link="front_right_wheel" wheel_joint="front_right_joint"/>
+      <xacro:mecanum_wheel_properties wheel_link="rear_left_wheel" wheel_joint="rear_left_joint"/>
+      <xacro:mecanum_wheel_properties wheel_link="rear_right_wheel" wheel_joint="rear_right_joint"/>
+    </xacro:if>
+    <!-- tricycle: 3-wheeled tricycle -->
+    <xacro:if value="${controller_type == 'tricycle'}">
+      <!-- Traction wheel -->
+      <gazebo reference="front_wheel">
+        <collision>
+          <surface>
+            <friction>
+              <ode>
+                <mu>1.0</mu>
+                <mu2>1.0</mu2>
+              </ode>
+            </friction>
+            <contact>
+              <kp>1e6</kp>
+              <kd>1.0</kd>
+              <max_vel>0.1</max_vel>
+              <min_depth>0.001</min_depth>
+            </contact>
+            <bounce>
+              <restitution_coefficient>0.0</restitution_coefficient>
+            </bounce>
+          </surface>
+        </collision>
+      </gazebo>
+      <gazebo reference="front_joint">
+        <damping>0.1</damping>
+      </gazebo>
+      <!-- Steering joint -->
+      <gazebo reference="chassis_to_front_steering">
+        <damping>0.01</damping>
+        <friction>0.3</friction>
+      </gazebo>
+      <!-- Rear wheels -->
+      <xacro:macro name="rear_wheel_properties" params="wheel_link wheel_joint">
+        <gazebo reference="${wheel_link}">
+          <collision>
+            <surface>
+              <friction>
+                <ode>
+                  <mu>0.8</mu>
+                  <mu2>0.8</mu2>
+                </ode>
+              </friction>
+              <contact>
+                <kp>1e6</kp>
+                <kd>1.0</kd>
+                <max_vel>0.1</max_vel>
+                <min_depth>0.001</min_depth>
+              </contact>
+              <bounce>
+                <restitution_coefficient>0.0</restitution_coefficient>
+              </bounce>
+            </surface>
+          </collision>
+        </gazebo>
+        <gazebo reference="${wheel_joint}">
+          <damping>0.05</damping>
+        </gazebo>
+      </xacro:macro>
+      <xacro:rear_wheel_properties wheel_link="rear_left_wheel" wheel_joint="rear_left_joint"/>
+      <xacro:rear_wheel_properties wheel_link="rear_right_wheel" wheel_joint="rear_right_joint"/>
+    </xacro:if>
+    <!-- triSteer: 3-wheeled tricycle steering -->
+    <xacro:if value="${controller_type == 'triSteer'}">
+      <!-- Traction wheel -->
+      <gazebo reference="front_wheel">
+        <collision>
+          <surface>
+            <friction>
+              <ode>
+                <mu>1.0</mu>
+                <mu2>1.0</mu2>
+              </ode>
+            </friction>
+            <contact>
+              <kp>1e6</kp>
+              <kd>1.0</kd>
+              <max_vel>0.1</max_vel>
+              <min_depth>0.001</min_depth>
+            </contact>
+            <bounce>
+              <restitution_coefficient>0.0</restitution_coefficient>
+            </bounce>
+          </surface>
+        </collision>
+      </gazebo>
+      <gazebo reference="front_joint">
+        <damping>0.1</damping>
+      </gazebo>
+      <!-- Steering joint -->
+      <gazebo reference="chassis_to_front_steering">
+        <damping>0.02</damping>
+        <friction>0.3</friction>
+      </gazebo>
+      <!-- Rear wheels -->
+      <xacro:macro name="rear_wheel_properties" params="wheel_link wheel_joint">
+        <gazebo reference="${wheel_link}">
+          <collision>
+            <surface>
+              <friction>
+                <ode>
+                  <mu>0.8</mu>
+                  <mu2>0.8</mu2>
+                </ode>
+              </friction>
+              <contact>
+                <kp>1e6</kp>
+                <kd>1.0</kd>
+                <max_vel>0.1</max_vel>
+                <min_depth>0.001</min_depth>
+              </contact>
+              <bounce>
+                <restitution_coefficient>0.0</restitution_coefficient>
+              </bounce>
+            </surface>
+          </collision>
+        </gazebo>
+        <gazebo reference="${wheel_joint}">
+          <damping>0.05</damping>
+        </gazebo>
+      </xacro:macro>
+      <xacro:rear_wheel_properties wheel_link="rear_left_wheel" wheel_joint="rear_left_joint"/>
+      <xacro:rear_wheel_properties wheel_link="rear_right_wheel" wheel_joint="rear_right_joint"/>
+    </xacro:if>
+    <!-- ackermann: 4-wheeled Ackermann -->
+    <xacro:if value="${controller_type == 'ackermann'}">
+      <!-- Traction wheels -->
+      <xacro:macro name="traction_wheel_properties" params="wheel_link wheel_joint">
+        <gazebo reference="${wheel_link}">
+          <collision>
+            <surface>
+              <friction>
+                <ode>
+                  <mu>1.0</mu>
+                  <mu2>1.0</mu2>
+                </ode>
+              </friction>
+              <contact>
+                <kp>1e6</kp>
+                <kd>1.0</kd>
+                <max_vel>0.1</max_vel>
+                <min_depth>0.001</min_depth>
+              </contact>
+              <bounce>
+                <restitution_coefficient>0.0</restitution_coefficient>
+              </bounce>
+            </surface>
+          </collision>
+        </gazebo>
+        <gazebo reference="${wheel_joint}">
+          <damping>0.1</damping>
+        </gazebo>
+      </xacro:macro>
+      <xacro:traction_wheel_properties wheel_link="rear_left_wheel" wheel_joint="rear_left_joint"/>
+      <xacro:traction_wheel_properties wheel_link="rear_right_wheel" wheel_joint="rear_right_joint"/>
+      <!-- Steering joints -->
+      <gazebo reference="chassis_to_front_left_steering">
+        <damping>0.01</damping>
+        <friction>0.3</friction>
+      </gazebo>
+      <gazebo reference="chassis_to_front_right_steering">
+        <damping>0.01</damping>
+        <friction>0.3</friction>
+      </gazebo>
+      <!-- Front wheels -->
+      <xacro:macro name="front_wheel_properties" params="wheel_link wheel_joint">
+        <gazebo reference="${wheel_link}">
+          <collision>
+            <surface>
+              <friction>
+                <ode>
+                  <mu>0.8</mu>
+                  <mu2>0.8</mu2>
+                </ode>
+              </friction>
+              <contact>
+                <kp>1e6</kp>
+                <kd>1.0</kd>
+                <max_vel>0.1</max_vel>
+                <min_depth>0.001</min_depth>
+              </contact>
+              <bounce>
+                <restitution_coefficient>0.0</restitution_coefficient>
+              </bounce>
+            </surface>
+          </collision>
+        </gazebo>
+        <gazebo reference="${wheel_joint}">
+          <damping>0.05</damping>
+        </gazebo>
+      </xacro:macro>
+      <xacro:front_wheel_properties wheel_link="front_left_wheel" wheel_joint="front_left_joint"/>
+      <xacro:front_wheel_properties wheel_link="front_right_wheel" wheel_joint="front_right_joint"/>
+    </xacro:if>
+  </xacro:macro>
 </robot>

File: src/mobRobURDF_description/urdf/gazebo_files/gazebo_sensors.xacro (robot description, xacro)
@@ -3,58 +3,48 @@
   <!-- Gazebo Lidar Plugin -->
   <gazebo reference="lidar">
-    <sensor type="ray" name="lidar_sensor">
-      <pose>0 0 0 0 0 0</pose>
+    <material>Gazebo/Black</material>
+    <sensor name="laser" type="gpu_lidar">
+      <pose> 0 0 0 0 0 0 </pose>
       <visualize>true</visualize>
       <update_rate>10</update_rate>
-      <ray>
+      <lidar>
         <scan>
           <horizontal>
             <samples>360</samples>
-            <resolution>1</resolution>
-            <min_angle>0</min_angle>
-            <max_angle>6.28319</max_angle>
+            <min_angle>-3.14</min_angle>
+            <max_angle>3.14</max_angle>
           </horizontal>
         </scan>
         <range>
-          <min>0.1</min>
-          <max>10</max>
-          <resolution>0.01</resolution>
+          <min>0.3</min>
+          <max>12</max>
         </range>
-      </ray>
-      <plugin name="lidar_plugin" filename="libgazebo_ros_ray_sensor.so">
-        <ros>
-          <namespace>/</namespace>
-          <remapping>~/out:=scan</remapping>
-        </ros>
-        <output_type>sensor_msgs/LaserScan</output_type>
-        <frame_name>lidar</frame_name>
-      </plugin>
+      </lidar>
+        <topic>scan</topic>
+        <gz_frame_id>laser_frame</gz_frame_id>
     </sensor>
   </gazebo>
   <!-- Gazebo Camera Plugin -->
   <gazebo reference="camera">
-    <sensor type="camera" name="camera_sensor">
-      <pose>0 0 0 0 0 0</pose>
+    <material>Gazebo/Black</material>
+    <sensor name="camera" type="camera">
+      <pose> 0 0 0 0 0 0 </pose>
       <visualize>true</visualize>
-      <update_rate>30</update_rate>
+      <update_rate>10</update_rate>
       <camera>
-        <horizontal_fov>1.0472</horizontal_fov>
+        <camera_info_topic>camera/camera_info</camera_info_topic>
+        <horizontal_fov>1.089</horizontal_fov>
         <image>
+          <format>R8G8B8</format>
           <width>640</width>
           <height>480</height>
         </image>
         <clip>
-          <near>0.1</near>
-          <far>100</far>
+          <near>0.05</near>
+          <far>8.0</far>
         </clip>
       </camera>
-      <plugin name="camera_plugin" filename="libgazebo_ros_camera.so">
-        <ros>
-          <namespace>/</namespace>
-          <remapping>~/image_raw:=camera/image_raw</remapping>
-        </ros>
-        <camera_name>camera</camera_name>
-        <frame_name>camera_optical</frame_name> <!-- Use camera_optical frame -->
-      </plugin>
+      <topic>camera/image_raw</topic>
+      <gz_frame_id>camera_link_optical</gz_frame_id>
     </sensor>
   </gazebo>

File: src/mobRobURDF_description/urdf/mobRob.urdf (robot description, URDF)
Before this commit: robot mobRob, 11 links, 10 joints
Joints:
- joint chassis_to_front_left_steering: limit lower=-1.5707963267948966 upper=1.5707963267948966 effort=100 velocity=10 -> lower=-0.7853981633974483 upper=0.7853981633974483 effort=100 velocity=10
- joint chassis_to_front_right_steering: limit lower=-1.5707963267948966 upper=1.5707963267948966 effort=100 velocity=10 -> lower=-0.7853981633974483 upper=0.7853981633974483 effort=100 velocity=10

File: src/mobRobURDF_description/urdf/submodules/2_wheeled_caster/mobRob_2wc_diff.xacro (robot description, xacro)
@@ -1,4 +1,4 @@
 <?xml version="1.0"?>
-<robot xmlns:xacro="http://www.ros.org/wiki/xacro" name="mobRob">
+<robot xmlns:xacro="http://www.ros.org/wiki/xacro">
   <!-- Include Xacro files -->
   <xacro:include filename="$(find mobRobURDF_description)/urdf/submodules/2_wheeled_caster/base.xacro" />
@@ -20,5 +20,10 @@
   <!-- Include Gazebo Xacro files -->
   <xacro:include filename="$(find mobRobURDF_description)/urdf/gazebo_files/control/gazebo_ros2_control_2wc_diff.xacro" />
+  <xacro:include filename="$(find mobRobURDF_description)/urdf/gazebo_files/gazebo_sensors.xacro" />
   <xacro:include filename="$(find mobRobURDF_description)/urdf/gazebo_files/gazebo_properties.xacro" />
-  <xacro:include filename="$(find mobRobURDF_description)/urdf/gazebo_files/gazebo_sensors.xacro" />
+  <xacro:gazebo_physical_properties
+  controller_type="${controller_type}"
+  chassis_size="${chassis_size}"
+  wheel_radius="${wheel_radius}"
+  wheel_width="${wheel_width}"/>
 </robot>
