Commit message: Modified xacro files (for controllers).

File: src/mobRobURDF_description/urdf/submodules/3_wheeled/mobRob_3w_triSteer.xacro (robot description, xacro)
@@ -1,4 +1,4 @@
 <?xml version="1.0"?>
-<robot xmlns:xacro="http://www.ros.org/wiki/xacro" name="mobRob">
+<robot xmlns:xacro="http://www.ros.org/wiki/xacro">
   <!-- Include Xacro files -->
   <xacro:include filename="$(find mobRobURDF_description)/urdf/submodules/3_wheeled/base.xacro" />
@@ -20,5 +20,10 @@
   <!-- Include Gazebo Xacro files -->
   <xacro:include filename="$(find mobRobURDF_description)/urdf/gazebo_files/control/gazebo_ros2_control_3w_triSteer.xacro" />
+  <xacro:include filename="$(find mobRobURDF_description)/urdf/gazebo_files/gazebo_sensors.xacro" />
   <xacro:include filename="$(find mobRobURDF_description)/urdf/gazebo_files/gazebo_properties.xacro" />
-  <xacro:include filename="$(find mobRobURDF_description)/urdf/gazebo_files/gazebo_sensors.xacro" />
+  <xacro:gazebo_physical_properties
+  controller_type="${controller_type}"
+  chassis_size="${chassis_size}"
+  wheel_radius="${wheel_radius}"
+  wheel_width="${wheel_width}"/>
 </robot>

File: src/mobRobURDF_description/urdf/submodules/3_wheeled/mobRob_3w_tricycle.xacro (robot description, xacro)
@@ -1,4 +1,4 @@
 <?xml version="1.0"?>
-<robot xmlns:xacro="http://www.ros.org/wiki/xacro" name="mobRob">
+<robot xmlns:xacro="http://www.ros.org/wiki/xacro">
   <!-- Include Xacro files -->
   <xacro:include filename="$(find mobRobURDF_description)/urdf/submodules/3_wheeled/base.xacro" />
@@ -20,5 +20,10 @@
   <!-- Include Gazebo Xacro files -->
   <xacro:include filename="$(find mobRobURDF_description)/urdf/gazebo_files/control/gazebo_ros2_control_3w_tricycle.xacro" />
+  <xacro:include filename="$(find mobRobURDF_description)/urdf/gazebo_files/gazebo_sensors.xacro" />
   <xacro:include filename="$(find mobRobURDF_description)/urdf/gazebo_files/gazebo_properties.xacro" />
-  <xacro:include filename="$(find mobRobURDF_description)/urdf/gazebo_files/gazebo_sensors.xacro" />
+  <xacro:gazebo_physical_properties
+  controller_type="${controller_type}"
+  chassis_size="${chassis_size}"
+  wheel_radius="${wheel_radius}"
+  wheel_width="${wheel_width}"/>
 </robot>

File: src/mobRobURDF_description/urdf/submodules/4_wheeled/ackermann/mobRob_4w_acker.xacro (robot description, xacro)
@@ -1,4 +1,4 @@
 <?xml version="1.0"?>
-<robot xmlns:xacro="http://www.ros.org/wiki/xacro" name="mobRob">
+<robot xmlns:xacro="http://www.ros.org/wiki/xacro">
   <!-- Include Xacro files -->
   <xacro:include filename="$(find mobRobURDF_description)/urdf/submodules/4_wheeled/ackermann/base.xacro" />
@@ -21,5 +21,10 @@
   <!-- Include Gazebo Xacro files -->
   <xacro:include filename="$(find mobRobURDF_description)/urdf/gazebo_files/control/gazebo_ros2_control_4w_acker.xacro" />
+  <xacro:include filename="$(find mobRobURDF_description)/urdf/gazebo_files/gazebo_sensors.xacro" />
   <xacro:include filename="$(find mobRobURDF_description)/urdf/gazebo_files/gazebo_properties.xacro" />
-  <xacro:include filename="$(find mobRobURDF_description)/urdf/gazebo_files/gazebo_sensors.xacro" />
+  <xacro:gazebo_physical_properties
+  controller_type="${controller_type}"
+  chassis_size="${chassis_size}"
+  wheel_radius="${wheel_radius}"
+  wheel_width="${wheel_width}"/>
 </robot>

File: src/mobRobURDF_description/urdf/submodules/4_wheeled/mobRob_4w_diff.xacro (robot description, xacro)
@@ -1,4 +1,4 @@
 <?xml version="1.0"?>
-<robot xmlns:xacro="http://www.ros.org/wiki/xacro" name="mobRob">
+<robot xmlns:xacro="http://www.ros.org/wiki/xacro">
   <!-- Include Xacro files -->
   <xacro:include filename="$(find mobRobURDF_description)/urdf/submodules/4_wheeled/base.xacro" />
@@ -21,5 +21,10 @@
   <!-- Include Gazebo Xacro files -->
   <xacro:include filename="$(find mobRobURDF_description)/urdf/gazebo_files/control/gazebo_ros2_control_4w_diff.xacro" />
+  <xacro:include filename="$(find mobRobURDF_description)/urdf/gazebo_files/gazebo_sensors.xacro" />
   <xacro:include filename="$(find mobRobURDF_description)/urdf/gazebo_files/gazebo_properties.xacro" />
-  <xacro:include filename="$(find mobRobURDF_description)/urdf/gazebo_files/gazebo_sensors.xacro" />
+  <xacro:gazebo_physical_properties
+  controller_type="${controller_type}"
+  chassis_size="${chassis_size}"
+  wheel_radius="${wheel_radius}"
+  wheel_width="${wheel_width}"/>
 </robot>

File: src/mobRobURDF_description/urdf/submodules/4_wheeled/mobRob_4w_mec.xacro (robot description, xacro)
@@ -1,4 +1,4 @@
 <?xml version="1.0"?>
-<robot xmlns:xacro="http://www.ros.org/wiki/xacro" name="mobRob">
+<robot xmlns:xacro="http://www.ros.org/wiki/xacro">
   <!-- Include Xacro files -->
   <xacro:include filename="$(find mobRobURDF_description)/urdf/submodules/4_wheeled/base.xacro" />
@@ -21,5 +21,10 @@
   <!-- Include Gazebo Xacro files -->
   <xacro:include filename="$(find mobRobURDF_description)/urdf/gazebo_files/control/gazebo_ros2_control_4w_mec.xacro" />
+  <xacro:include filename="$(find mobRobURDF_description)/urdf/gazebo_files/gazebo_sensors.xacro" />
   <xacro:include filename="$(find mobRobURDF_description)/urdf/gazebo_files/gazebo_properties.xacro" />
-  <xacro:include filename="$(find mobRobURDF_description)/urdf/gazebo_files/gazebo_sensors.xacro" />
+  <xacro:gazebo_physical_properties
+  controller_type="${controller_type}"
+  chassis_size="${chassis_size}"
+  wheel_radius="${wheel_radius}"
+  wheel_width="${wheel_width}"/>
 </robot>

Commit message: Added a feature of letting us choose the hardware interface

File: src/mobRobURDF_description/urdf/gazebo_files/control/gazebo_ros2_control_2wc_diff.xacro (robot description, xacro)
@@ -3,5 +3,5 @@
     <ros2_control name="GazeboSystem" type="system">
         <hardware>
-            <plugin>gz_ros2_control/GazeboSimSystem</plugin>
+            <plugin>${hardware_plugin}</plugin>
         </hardware>
         <joint name="left_joint">
@@ -36,8 +36,10 @@
         <!-- - - - - - - - - - - - - - -->
     </ros2_control>
-    <gazebo>
-        <plugin name="gz_ros2_control::GazeboSimROS2ControlPlugin" filename="libgz_ros2_control-system.so">
-            <parameters>$(find mobRobURDF_control)/config/drive/gazebo_controller_diffDrive_2wd_caster.yaml</parameters>
-        </plugin>
-    </gazebo>
+    <xacro:if value="${use_gazebo_sim}">
+        <gazebo>
+            <plugin name="gz_ros2_control::GazeboSimROS2ControlPlugin" filename="libgz_ros2_control-system.so">
+                <parameters>$(find mobRobURDF_control)/config/drive/gazebo_controller_diffDrive_2wd_caster.yaml</parameters>
+            </plugin>
+        </gazebo>
+    </xacro:if>
 </robot>

File: src/mobRobURDF_description/urdf/gazebo_files/control/gazebo_ros2_control_3w_triSteer.xacro (robot description, xacro)
@@ -3,5 +3,5 @@
     <ros2_control name="GazeboSystem" type="system">
         <hardware>
-            <plugin>gz_ros2_control/GazeboSimSystem</plugin>
+            <plugin>${hardware_plugin}</plugin>
         </hardware>
         <joint name="rear_left_joint">
@@ -36,14 +36,16 @@
         <!-- - - - - - - - - - - - - - -->
     </ros2_control>
-    <gazebo>
-        <plugin name="gz_ros2_control::GazeboSimROS2ControlPlugin" filename="libgz_ros2_control-system.so">
-            <parameters>$(find mobRobURDF_control)/config/steer/gazebo_controller_triSteer.yaml</parameters>
-            <ros>
-                <!-- tricycle_steering_controller publishes to ~/tf_odometry and ~/odometry,
-                     not to /tf and /odom. Remap to the standard global topics. -->
-                <remapping>/triSteer_controller/tf_odometry:=/tf</remapping>
-                <remapping>/triSteer_controller/odometry:=/odom</remapping>
-            </ros>
-        </plugin>
-    </gazebo>
+    <xacro:if value="${use_gazebo_sim}">
+        <gazebo>
+            <plugin name="gz_ros2_control::GazeboSimROS2ControlPlugin" filename="libgz_ros2_control-system.so">
+                <parameters>$(find mobRobURDF_control)/config/steer/gazebo_controller_triSteer.yaml</parameters>
+                <ros>
+                    <!-- tricycle_steering_controller publishes to ~/tf_odometry and ~/odometry,
+                         not to /tf and /odom. Remap to the standard global topics. -->
+                    <remapping>/triSteer_controller/tf_odometry:=/tf</remapping>
+                    <remapping>/triSteer_controller/odometry:=/odom</remapping>
+                </ros>
+            </plugin>
+        </gazebo>
+    </xacro:if>
 </robot>

File: src/mobRobURDF_description/urdf/gazebo_files/control/gazebo_ros2_control_3w_tricycle.xacro (robot description, xacro)
@@ -3,5 +3,5 @@
     <ros2_control name="GazeboSystem" type="system">
         <hardware>
-            <plugin>gz_ros2_control/GazeboSimSystem</plugin>
+            <plugin>${hardware_plugin}</plugin>
         </hardware>
         <joint name="front_joint">
@@ -32,8 +32,10 @@
         <!-- - - - - - - - - - - - - - -->
     </ros2_control>
-    <gazebo>
-        <plugin name="gz_ros2_control::GazeboSimROS2ControlPlugin" filename="libgz_ros2_control-system.so">
-            <parameters>$(find mobRobURDF_control)/config/gazebo_controller_tricycle.yaml</parameters>
-        </plugin>
-    </gazebo>
+    <xacro:if value="${use_gazebo_sim}">
+        <gazebo>
+            <plugin name="gz_ros2_control::GazeboSimROS2ControlPlugin" filename="libgz_ros2_control-system.so">
+                <parameters>$(find mobRobURDF_control)/config/gazebo_controller_tricycle.yaml</parameters>
+            </plugin>
+        </gazebo>
+    </xacro:if>
 </robot>

File: src/mobRobURDF_description/urdf/gazebo_files/control/gazebo_ros2_control_4w_acker.xacro (robot description, xacro)
@@ -3,5 +3,5 @@
     <ros2_control name="GazeboSystem" type="system">
         <hardware>
-            <plugin>gz_ros2_control/GazeboSimSystem</plugin>
+            <plugin>${hardware_plugin}</plugin>
         </hardware>
         <joint name="rear_left_joint">
@@ -48,14 +48,16 @@
         <!-- - - - - - - - - - - - - - -->
     </ros2_control>
-    <gazebo>
-        <plugin name="gz_ros2_control::GazeboSimROS2ControlPlugin" filename="libgz_ros2_control-system.so">
-            <parameters>$(find mobRobURDF_control)/config/steer/gazebo_controller_ackerSteer.yaml</parameters>
-            <ros>
-                <!-- ackermann_steering_controller publishes to ~/tf_odometry and ~/odometry,
-                     not to /tf and /odom. Remap to the standard global topics. -->
-                <remapping>/ackerSteer_controller/tf_odometry:=/tf</remapping>
-                <remapping>/ackerSteer_controller/odometry:=/odom</remapping>
-            </ros>
-        </plugin>
-    </gazebo>
+    <xacro:if value="${use_gazebo_sim}">
+        <gazebo>
+            <plugin name="gz_ros2_control::GazeboSimROS2ControlPlugin" filename="libgz_ros2_control-system.so">
+                <parameters>$(find mobRobURDF_control)/config/steer/gazebo_controller_ackerSteer.yaml</parameters>
+                <ros>
+                    <!-- ackermann_steering_controller publishes to ~/tf_odometry and ~/odometry,
+                         not to /tf and /odom. Remap to the standard global topics. -->
+                    <remapping>/ackerSteer_controller/tf_odometry:=/tf</remapping>
+                    <remapping>/ackerSteer_controller/odometry:=/odom</remapping>
+                </ros>
+            </plugin>
+        </gazebo>
+    </xacro:if>
 </robot>

File: src/mobRobURDF_description/urdf/gazebo_files/control/gazebo_ros2_control_4w_diff.xacro (robot description, xacro)
@@ -3,5 +3,5 @@
     <ros2_control name="GazeboSystem" type="system">
         <hardware>
-            <plugin>gz_ros2_control/GazeboSimSystem</plugin>
+            <plugin>${hardware_plugin}</plugin>
         </hardware>
         <joint name="front_left_joint">
@@ -39,8 +39,10 @@
         <!-- - - - - - - - - - - - - - -->
     </ros2_control>
-    <gazebo>
-        <plugin name="gz_ros2_control::GazeboSimROS2ControlPlugin" filename="libgz_ros2_control-system.so">
-            <parameters>$(find mobRobURDF_control)/config/drive/gazebo_controller_diffDrive_4wd.yaml</parameters>
-        </plugin>
-    </gazebo>
+    <xacro:if value="${use_gazebo_sim}">
+        <gazebo>
+            <plugin name="gz_ros2_control::GazeboSimROS2ControlPlugin" filename="libgz_ros2_control-system.so">
+                <parameters>$(find mobRobURDF_control)/config/drive/gazebo_controller_diffDrive_4wd.yaml</parameters>
+            </plugin>
+        </gazebo>
+    </xacro:if>
 </robot>

File: src/mobRobURDF_description/urdf/gazebo_files/control/gazebo_ros2_control_4w_mec.xacro (robot description, xacro)
@@ -3,5 +3,5 @@
     <ros2_control name="GazeboSystem" type="system">
         <hardware>
-            <plugin>gz_ros2_control/GazeboSimSystem</plugin>
+            <plugin>${hardware_plugin}</plugin>
         </hardware>
         <joint name="front_left_joint">
@@ -39,14 +39,16 @@
         <!-- - - - - - - - - - - - - - -->
     </ros2_control>
-    <gazebo>
-        <plugin name="gz_ros2_control::GazeboSimROS2ControlPlugin" filename="libgz_ros2_control-system.so">
-            <parameters>$(find mobRobURDF_control)/config/drive/gazebo_controller_mecDrive.yaml</parameters>
-            <ros>
-                <!-- mecanum_drive_controller publishes to ~/tf_odometry and ~/odometry,
-                     not to /tf and /odom. Remap to the standard global topics. -->
-                <remapping>/mecDrive_controller/tf_odometry:=/tf</remapping>
-                <remapping>/mecDrive_controller/odometry:=/odom</remapping>
-            </ros>
-        </plugin>
-    </gazebo>
+    <xacro:if value="${use_gazebo_sim}">
+        <gazebo>
+            <plugin name="gz_ros2_control::GazeboSimROS2ControlPlugin" filename="libgz_ros2_control-system.so">
+                <parameters>$(find mobRobURDF_control)/config/drive/gazebo_controller_mecDrive.yaml</parameters>
+                <ros>
+                    <!-- mecanum_drive_controller publishes to ~/tf_odometry and ~/odometry,
+                         not to /tf and /odom. Remap to the standard global topics. -->
+                    <remapping>/mecDrive_controller/tf_odometry:=/tf</remapping>
+                    <remapping>/mecDrive_controller/odometry:=/odom</remapping>
+                </ros>
+            </plugin>
+        </gazebo>
+    </xacro:if>
 </robot>

File: src/mobRobURDF_description/urdf/submodules/2_wheeled_caster/mobRob_2wc_diff.xacro (robot description, xacro)
@@ -14,4 +14,7 @@
   <xacro:wheel name="right" radius="${wheel_radius}" width="${wheel_width}" mass="${wheel_mass}" material="${wheel_material}" x="${r_x}" y="${r_y}" z="${r_z}" />
   <xacro:caster name="front_caster" radius="${caster_radius}" mass="${wheel_mass}" material="${wheel_material}" x="${caster_x}" y="${caster_y}" z="${caster_z}" />
+  <!-- Hardware interface (substituted by the wizard; used by the ros2_control xacro below) -->
+  <xacro:property name="hardware_plugin" value="${hardware_plugin}"/>
+  <xacro:property name="use_gazebo_sim" value="${use_gazebo_sim}"/>
   <!-- Include Gazebo Xacro files -->
   <xacro:include filename="$(find mobRobURDF_description)/urdf/gazebo_files/control/gazebo_ros2_control_2wc_diff.xacro" />

File: src/mobRobURDF_description/urdf/submodules/3_wheeled/mobRob_3w_triSteer.xacro (robot description, xacro)
@@ -14,4 +14,7 @@
   <xacro:wheel name="rear_left" radius="${wheel_radius}" width="${wheel_width}" mass="${wheel_mass}" material="${wheel_material}" x="${rl_x}" y="${rl_y}" z="${rl_z}" parent="chassis" />
   <xacro:wheel name="rear_right" radius="${wheel_radius}" width="${wheel_width}" mass="${wheel_mass}" material="${wheel_material}" x="${rr_x}" y="${rr_y}" z="${rr_z}" parent="chassis" />
+  <!-- Hardware interface (substituted by the wizard; used by the ros2_control xacro below) -->
+  <xacro:property name="hardware_plugin" value="${hardware_plugin}"/>
+  <xacro:property name="use_gazebo_sim" value="${use_gazebo_sim}"/>
   <!-- Include Gazebo Xacro files -->
   <xacro:include filename="$(find mobRobURDF_description)/urdf/gazebo_files/control/gazebo_ros2_control_3w_triSteer.xacro" />

File: src/mobRobURDF_description/urdf/submodules/3_wheeled/mobRob_3w_tricycle.xacro (robot description, xacro)
@@ -14,4 +14,7 @@
   <xacro:wheel name="rear_left" radius="${wheel_radius}" width="${wheel_width}" mass="${wheel_mass}" material="${wheel_material}" x="${rl_x}" y="${rl_y}" z="${rl_z}" parent="chassis" />
   <xacro:wheel name="rear_right" radius="${wheel_radius}" width="${wheel_width}" mass="${wheel_mass}" material="${wheel_material}" x="${rr_x}" y="${rr_y}" z="${rr_z}" parent="chassis" />
+  <!-- Hardware interface (substituted by the wizard; used by the ros2_control xacro below) -->
+  <xacro:property name="hardware_plugin" value="${hardware_plugin}"/>
+  <xacro:property name="use_gazebo_sim" value="${use_gazebo_sim}"/>
   <!-- Include Gazebo Xacro files -->
   <xacro:include filename="$(find mobRobURDF_description)/urdf/gazebo_files/control/gazebo_ros2_control_3w_tricycle.xacro" />

File: src/mobRobURDF_description/urdf/submodules/4_wheeled/ackermann/mobRob_4w_acker.xacro (robot description, xacro)
@@ -15,4 +15,7 @@
   <xacro:wheel name="rear_left" radius="${wheel_radius}" width="${wheel_width}" mass="${wheel_mass}" material="${wheel_material}" x="${rl_x}" y="${rl_y}" z="${rl_z}" parent="chassis" />
   <xacro:wheel name="rear_right" radius="${wheel_radius}" width="${wheel_width}" mass="${wheel_mass}" material="${wheel_material}" x="${rr_x}" y="${rr_y}" z="${rr_z}" parent="chassis" />
+  <!-- Hardware interface (substituted by the wizard; used by the ros2_control xacro below) -->
+  <xacro:property name="hardware_plugin" value="${hardware_plugin}"/>
+  <xacro:property name="use_gazebo_sim" value="${use_gazebo_sim}"/>
   <!-- Include Gazebo Xacro files -->
   <xacro:include filename="$(find mobRobURDF_description)/urdf/gazebo_files/control/gazebo_ros2_control_4w_acker.xacro" />

File: src/mobRobURDF_description/urdf/submodules/4_wheeled/mobRob_4w_diff.xacro (robot description, xacro)
@@ -15,4 +15,7 @@
   <xacro:wheel name="rear_left" radius="${wheel_radius}" width="${wheel_width}" mass="${wheel_mass}" material="${wheel_material}" x="${rl_x}" y="${rl_y}" z="${rl_z}" />
   <xacro:wheel name="rear_right" radius="${wheel_radius}" width="${wheel_width}" mass="${wheel_mass}" material="${wheel_material}" x="${rr_x}" y="${rr_y}" z="${rr_z}" />
+  <!-- Hardware interface (substituted by the wizard; used by the ros2_control xacro below) -->
+  <xacro:property name="hardware_plugin" value="${hardware_plugin}"/>
+  <xacro:property name="use_gazebo_sim" value="${use_gazebo_sim}"/>
   <!-- Include Gazebo Xacro files -->
   <xacro:include filename="$(find mobRobURDF_description)/urdf/gazebo_files/control/gazebo_ros2_control_4w_diff.xacro" />

File: src/mobRobURDF_description/urdf/submodules/4_wheeled/mobRob_4w_mec.xacro (robot description, xacro)
@@ -15,4 +15,7 @@
   <xacro:wheel name="rear_left" radius="${wheel_radius}" width="${wheel_width}" mass="${wheel_mass}" material="${wheel_material}" x="${rl_x}" y="${rl_y}" z="${rl_z}" />
   <xacro:wheel name="rear_right" radius="${wheel_radius}" width="${wheel_width}" mass="${wheel_mass}" material="${wheel_material}" x="${rr_x}" y="${rr_y}" z="${rr_z}" />
+  <!-- Hardware interface (substituted by the wizard; used by the ros2_control xacro below) -->
+  <xacro:property name="hardware_plugin" value="${hardware_plugin}"/>
+  <xacro:property name="use_gazebo_sim" value="${use_gazebo_sim}"/>
   <!-- Include Gazebo Xacro files -->
   <xacro:include filename="$(find mobRobURDF_description)/urdf/gazebo_files/control/gazebo_ros2_control_4w_mec.xacro" />
