Commit message: Modifying the 3D-model and real robot model in Rviz

File: src/mobRobURDF_description/urdf/mobRob.urdf (robot description, URDF)
Before this commit: robot mobRob, 9 links, 8 joints
Joints:
- joint base_to_chassis: origin xyz=0 0 0 rpy=0 0 0 -> xyz=0 0 0.15 rpy=0 0 0
- joint camera_joint: origin xyz=0.04 0 0 rpy=0 0 0 -> xyz=0.64 0 0 rpy=0 0 0
- joint front_left_joint: origin xyz=0.6 0.4 -0.15 rpy=0 0 0 -> xyz=0.6 0.46 -0.15 rpy=0 0 0
- joint front_right_joint: origin xyz=0.6 -0.4 -0.15 rpy=0 0 0 -> xyz=0.6 -0.46 -0.15 rpy=0 0 0
- joint lidar_joint: origin xyz=0 0 0.15 rpy=0 0 0 -> xyz=0 0 0.19 rpy=0 0 0
- joint rear_left_joint: origin xyz=-0.6 0.4 -0.15 rpy=0 0 0 -> xyz=-0.6 0.46 -0.15 rpy=0 0 0
- joint rear_right_joint: origin xyz=-0.6 -0.4 -0.15 rpy=0 0 0 -> xyz=-0.6 -0.46 -0.15 rpy=0 0 0

File: src/mobRobURDF_description/urdf/mobRob.xacro (robot description, xacro)
@@ -19,4 +19,4 @@
   <!-- Sensors -->
   <xacro:lidar radius="${lidar_radius}" height="${lidar_height}" mass="${lidar_mass}" material="${lidar_material}" z="${lidar_z}" />
-  <xacro:camera size="${camera_size}" mass="${camera_mass}" material="${camera_material}" />
+  <xacro:camera size="${camera_size}" mass="${camera_mass}" material="${camera_material}" x="${camera_x}" />
 </robot>

File: src/mobRobURDF_description/urdf/submodules/base.xacro (robot description, xacro)
@@ -31,10 +31,10 @@
       </collision>
     </link>
+    <!-- Fixed Joint between base_link and chassis -->
+    <joint name="base_to_chassis" type="fixed">
+      <parent link="base_link" />
+      <child link="chassis" />
+      <origin xyz="0 0 ${h/2}" rpy="0 0 0" />
+    </joint>
   </xacro:macro>
-  <!-- Fixed Joint between base_link and chassis -->
-  <joint name="base_to_chassis" type="fixed">
-    <parent link="base_link" />
-    <child link="chassis" />
-    <origin xyz="0 0 0" rpy="0 0 0" />
-  </joint>
 </robot>

File: src/mobRobURDF_description/urdf/submodules/sensors.xacro (robot description, xacro)
@@ -33,5 +33,5 @@
   </xacro:macro>
   <!-- Camera Macro -->
-  <xacro:macro name="camera" params="size mass material">
+  <xacro:macro name="camera" params="size mass material x">
     <!-- Split the size string into individual components and convert to floats -->
     <xacro:property name="size_list" value="${list(map(float, size.split()))}" />
@@ -64,5 +64,5 @@
       <parent link="chassis" />
       <child link="camera" />
-      <origin xyz="${l / 2} 0 0" rpy="0 0 0" />
+      <origin xyz="${x} 0 0" rpy="0 0 0" />
     </joint>
     <!-- Camera Optical Frame -->

File: src/mobRobURDF_wizard/mobRobURDF_wizard/temp/mobRob.xacro (robot description, xacro)
@@ -1,5 +1,5 @@
 <?xml version="1.0"?>
 <robot xmlns:xacro="http://www.ros.org/wiki/xacro" name="mobRob">
-  <!-- Include other xacro files -->
+  <!-- Include Xacro files -->
   <xacro:include filename="$(find mobRobURDF_description)/urdf/submodules/base.xacro" />
   <xacro:include filename="$(find mobRobURDF_description)/urdf/submodules/wheels.xacro" />
@@ -13,10 +13,10 @@
   <xacro:chassis size="1.2 0.8 0.3" mass="1.0" material="Gray" />
   <!-- Wheels -->
-  <xacro:wheel name="front_left" radius="0.22" width="0.12" mass="0.5" material="Black" x="0.6" y="0.4" z="-0.15" />
-  <xacro:wheel name="front_right" radius="0.22" width="0.12" mass="0.5" material="Black" x="0.6" y="-0.4" z="-0.15" />
-  <xacro:wheel name="rear_left" radius="0.22" width="0.12" mass="0.5" material="Black" x="-0.6" y="0.4" z="-0.15" />
-  <xacro:wheel name="rear_right" radius="0.22" width="0.12" mass="0.5" material="Black" x="-0.6" y="-0.4" z="-0.15" />
+  <xacro:wheel name="front_left" radius="0.22" width="0.12" mass="0.5" material="Black" x="0.6" y="0.46" z="-0.15" />
+  <xacro:wheel name="front_right" radius="0.22" width="0.12" mass="0.5" material="Black" x="0.6" y="-0.46" z="-0.15" />
+  <xacro:wheel name="rear_left" radius="0.22" width="0.12" mass="0.5" material="Black" x="-0.6" y="0.46" z="-0.15" />
+  <xacro:wheel name="rear_right" radius="0.22" width="0.12" mass="0.5" material="Black" x="-0.6" y="-0.46" z="-0.15" />
   <!-- Sensors -->
-  <xacro:lidar radius="0.1" height="0.08" mass="0.2" material="Red" z="0.15" />
-  <xacro:camera size="0.08 0.2 0.08" mass="0.1" material="Blue" />
+  <xacro:lidar radius="0.1" height="0.08" mass="0.2" material="Red" z="0.19" />
+  <xacro:camera size="0.08 0.2 0.08" mass="0.1" material="Blue" x="0.64" />
 </robot>

Commit message: Modified camera rotation using mouse (3-DOF rotation instead of 2-DOF rotation)

File: src/mobRobURDF_description/urdf/mobRob.urdf (robot description, URDF)
Before this commit: robot mobRob, 9 links, 8 joints
Links:
- link camera: mass 0.1 -> 1.2; geometry collision box size=0.05 0.2 0.05; visual box size=0.05 0.2 0.05
- link chassis: mass 1.0 -> 5; geometry collision box size=1.5 0.5 0.1; visual box size=1.5 0.5 0.1
- link front_left_wheel: geometry collision cylinder length=0.05 radius=0.15; visual cylinder length=0.05 radius=0.15
- link front_right_wheel: geometry collision cylinder length=0.05 radius=0.15; visual cylinder length=0.05 radius=0.15
- link lidar: mass 0.2 -> 0.5; geometry collision cylinder length=0.1 radius=0.15; visual cylinder length=0.1 radius=0.15
- link rear_left_wheel: geometry collision cylinder length=0.05 radius=0.15; visual cylinder length=0.05 radius=0.15
- link rear_right_wheel: geometry collision cylinder length=0.05 radius=0.15; visual cylinder length=0.05 radius=0.15
Joints:
- joint base_to_chassis: origin xyz=0 0 0.15 rpy=0 0 0 -> xyz=0 0 0.05 rpy=0 0 0
- joint camera_joint: origin xyz=0.64 0 0 rpy=0 0 0 -> xyz=0.775 0 0 rpy=0 0 0
- joint front_left_joint: origin xyz=0.6 0.46 -0.15 rpy=0 0 0 -> xyz=0.75 0.275 -0.05 rpy=0 0 0
- joint front_right_joint: origin xyz=0.6 -0.46 -0.15 rpy=0 0 0 -> xyz=0.75 -0.275 -0.05 rpy=0 0 0
- joint lidar_joint: origin xyz=0 0 0.19 rpy=0 0 0 -> xyz=0 0 0.1 rpy=0 0 0
- joint rear_left_joint: origin xyz=-0.6 0.46 -0.15 rpy=0 0 0 -> xyz=-0.75 0.275 -0.05 rpy=0 0 0
- joint rear_right_joint: origin xyz=-0.6 -0.46 -0.15 rpy=0 0 0 -> xyz=-0.75 -0.275 -0.05 rpy=0 0 0

File: src/mobRobURDF_wizard/mobRobURDF_wizard/temp/mobRob.xacro (robot description, xacro)
@@ -11,12 +11,12 @@
   <xacro:define_materials/>
   <!-- Define the robot -->
-  <xacro:chassis size="1.2 0.8 0.3" mass="1.0" material="Gray" />
+  <xacro:chassis size="1.5 0.5 0.1" mass="5" material="Red" />
   <!-- Wheels -->
-  <xacro:wheel name="front_left" radius="0.22" width="0.12" mass="0.5" material="Black" x="0.6" y="0.46" z="-0.15" />
-  <xacro:wheel name="front_right" radius="0.22" width="0.12" mass="0.5" material="Black" x="0.6" y="-0.46" z="-0.15" />
-  <xacro:wheel name="rear_left" radius="0.22" width="0.12" mass="0.5" material="Black" x="-0.6" y="0.46" z="-0.15" />
-  <xacro:wheel name="rear_right" radius="0.22" width="0.12" mass="0.5" material="Black" x="-0.6" y="-0.46" z="-0.15" />
+  <xacro:wheel name="front_left" radius="0.15" width="0.05" mass="0.5" material="Green" x="0.75" y="0.275" z="-0.05" />
+  <xacro:wheel name="front_right" radius="0.15" width="0.05" mass="0.5" material="Green" x="0.75" y="-0.275" z="-0.05" />
+  <xacro:wheel name="rear_left" radius="0.15" width="0.05" mass="0.5" material="Green" x="-0.75" y="0.275" z="-0.05" />
+  <xacro:wheel name="rear_right" radius="0.15" width="0.05" mass="0.5" material="Green" x="-0.75" y="-0.275" z="-0.05" />
   <!-- Sensors -->
-  <xacro:lidar radius="0.1" height="0.08" mass="0.2" material="Red" z="0.19" />
-  <xacro:camera size="0.08 0.2 0.08" mass="0.1" material="Blue" x="0.64" />
+  <xacro:lidar radius="0.15" height="0.1" mass="0.5" material="Blue" z="0.1" />
+  <xacro:camera size="0.05 0.2 0.05" mass="1.2" material="Black" x="0.775" />
 </robot>

Commit message: Editing the Wizard window

File: src/mobRobURDF_description/urdf/mobRob.urdf (robot description, URDF)
Before this commit: robot mobRob, 9 links, 8 joints
Links:
- link camera: mass 1.2 -> 0.1; geometry collision box size=0.08 0.2 0.08; visual box size=0.08 0.2 0.08
- link chassis: mass 5 -> 1.0; geometry collision box size=1.2 0.8 0.3; visual box size=1.2 0.8 0.3
- link front_left_wheel: geometry collision cylinder length=0.12 radius=0.22; visual cylinder length=0.12 radius=0.22
- link front_right_wheel: geometry collision cylinder length=0.12 radius=0.22; visual cylinder length=0.12 radius=0.22
- link lidar: mass 0.5 -> 0.2; geometry collision cylinder length=0.2 radius=0.1; visual cylinder length=0.2 radius=0.1
- link rear_left_wheel: geometry collision cylinder length=0.12 radius=0.22; visual cylinder length=0.12 radius=0.22
- link rear_right_wheel: geometry collision cylinder length=0.12 radius=0.22; visual cylinder length=0.12 radius=0.22
Joints:
- joint base_to_chassis: origin xyz=0 0 0.05 rpy=0 0 0 -> xyz=0 0 0.15 rpy=0 0 0
- joint camera_joint: origin xyz=0.775 0 0 rpy=0 0 0 -> xyz=0.64 0 0 rpy=0 0 0
- joint front_left_joint: origin xyz=0.75 0.275 -0.05 rpy=0 0 0 -> xyz=0.6 0.46 -0.15 rpy=0 0 0
- joint front_right_joint: origin xyz=0.75 -0.275 -0.05 rpy=0 0 0 -> xyz=0.6 -0.46 -0.15 rpy=0 0 0
- joint lidar_joint: origin xyz=0 0 0.1 rpy=0 0 0 -> xyz=0 0 0.25 rpy=0 0 0
- joint rear_left_joint: origin xyz=-0.75 0.275 -0.05 rpy=0 0 0 -> xyz=-0.6 0.46 -0.15 rpy=0 0 0
- joint rear_right_joint: origin xyz=-0.75 -0.275 -0.05 rpy=0 0 0 -> xyz=-0.6 -0.46 -0.15 rpy=0 0 0

File: src/mobRobURDF_wizard/mobRobURDF_wizard/classes/temp/mobRob.xacro (robot description, xacro)
@@ -18,5 +18,5 @@
   <xacro:wheel name="rear_right" radius="0.22" width="0.12" mass="0.5" material="Black" x="-0.6" y="-0.46" z="-0.15" />
   <!-- Sensors -->
-  <xacro:lidar radius="0.1" height="0.08" mass="0.2" material="Red" z="0.19" />
+  <xacro:lidar radius="0.1" height="0.2" mass="0.2" material="Red" z="0.25" />
   <xacro:camera size="0.08 0.2 0.08" mass="0.1" material="Blue" x="0.64" />
 </robot>

Commit message: Edited the README.md file

File: src/mobRobURDF_description/urdf/mobRob.urdf (robot description, URDF)
Before this commit: robot mobRob, 9 links, 8 joints
Links:
- link camera: geometry collision box size=0.05 0.1 0.06; visual box size=0.05 0.1 0.06
- link chassis: mass 1.0 -> 5; geometry collision box size=1.0 0.65 0.2; visual box size=1.0 0.65 0.2
- link front_left_wheel: mass 0.5 -> 0.3; geometry collision cylinder length=0.08 radius=0.18; visual cylinder length=0.08 radius=0.18
- link front_right_wheel: mass 0.5 -> 0.3; geometry collision cylinder length=0.08 radius=0.18; visual cylinder length=0.08 radius=0.18
- link lidar: geometry collision cylinder length=0.08 radius=0.09; visual cylinder length=0.08 radius=0.09
- link rear_left_wheel: mass 0.5 -> 0.3; geometry collision cylinder length=0.08 radius=0.18; visual cylinder length=0.08 radius=0.18
- link rear_right_wheel: mass 0.5 -> 0.3; geometry collision cylinder length=0.08 radius=0.18; visual cylinder length=0.08 radius=0.18
Joints:
- joint base_to_chassis: origin xyz=0 0 0.15 rpy=0 0 0 -> xyz=0 0 0.1 rpy=0 0 0
- joint camera_joint: origin xyz=0.64 0 0 rpy=0 0 0 -> xyz=0.525 0 0 rpy=0 0 0
- joint front_left_joint: origin xyz=0.6 0.46 -0.15 rpy=0 0 0 -> xyz=0.5 0.365 -0.1 rpy=0 0 0
- joint front_right_joint: origin xyz=0.6 -0.46 -0.15 rpy=0 0 0 -> xyz=0.5 -0.365 -0.1 rpy=0 0 0
- joint lidar_joint: origin xyz=0 0 0.25 rpy=0 0 0 -> xyz=0 0 0.14 rpy=0 0 0
- joint rear_left_joint: origin xyz=-0.6 0.46 -0.15 rpy=0 0 0 -> xyz=-0.5 0.365 -0.1 rpy=0 0 0
- joint rear_right_joint: origin xyz=-0.6 -0.46 -0.15 rpy=0 0 0 -> xyz=-0.5 -0.365 -0.1 rpy=0 0 0

File: src/mobRobURDF_wizard/mobRobURDF_wizard/classes/temp/mobRob.xacro (robot description, xacro)
@@ -11,12 +11,12 @@
   <xacro:define_materials/>
   <!-- Define the robot -->
-  <xacro:chassis size="1.2 0.8 0.3" mass="1.0" material="Gray" />
+  <xacro:chassis size="1 0.65 0.2" mass="5" material="Gray" />
   <!-- Wheels -->
-  <xacro:wheel name="front_left" radius="0.22" width="0.12" mass="0.5" material="Black" x="0.6" y="0.46" z="-0.15" />
-  <xacro:wheel name="front_right" radius="0.22" width="0.12" mass="0.5" material="Black" x="0.6" y="-0.46" z="-0.15" />
-  <xacro:wheel name="rear_left" radius="0.22" width="0.12" mass="0.5" material="Black" x="-0.6" y="0.46" z="-0.15" />
-  <xacro:wheel name="rear_right" radius="0.22" width="0.12" mass="0.5" material="Black" x="-0.6" y="-0.46" z="-0.15" />
+  <xacro:wheel name="front_left" radius="0.18" width="0.08" mass="0.3" material="Black" x="0.5" y="0.365" z="-0.1" />
+  <xacro:wheel name="front_right" radius="0.18" width="0.08" mass="0.3" material="Black" x="0.5" y="-0.365" z="-0.1" />
+  <xacro:wheel name="rear_left" radius="0.18" width="0.08" mass="0.3" material="Black" x="-0.5" y="0.365" z="-0.1" />
+  <xacro:wheel name="rear_right" radius="0.18" width="0.08" mass="0.3" material="Black" x="-0.5" y="-0.365" z="-0.1" />
   <!-- Sensors -->
-  <xacro:lidar radius="0.1" height="0.2" mass="0.2" material="Red" z="0.25" />
-  <xacro:camera size="0.08 0.2 0.08" mass="0.1" material="Blue" x="0.64" />
+  <xacro:lidar radius="0.09" height="0.08" mass="0.2" material="Red" z="0.14" />
+  <xacro:camera size="0.05 0.1 0.06" mass="0.1" material="Blue" x="0.525" />
 </robot>

Commit message: Adding more pages to wizard. Also, 3_wheeled and 2_wheeled_caster robot models

File: src/mobRobURDF_description/urdf/mobRob.urdf (robot description, URDF)
Before this commit: robot mobRob, 9 links, 8 joints
Links:
- link camera: mass 0.1 -> 0.3; geometry collision box size=0.05 0.1 0.05; visual box size=0.05 0.1 0.05
- link chassis: geometry collision box size=1.0 0.6 0.2; visual box size=1.0 0.6 0.2
- link front_left_wheel: mass 0.3 -> 0.5; geometry collision cylinder length=0.08 radius=0.2; visual cylinder length=0.08 radius=0.2
- link front_right_wheel: mass 0.3 -> 0.5; geometry collision cylinder length=0.08 radius=0.2; visual cylinder length=0.08 radius=0.2
- link lidar: mass 0.2 -> 0.4; geometry collision cylinder length=0.12 radius=0.12; visual cylinder length=0.12 radius=0.12
- link rear_left_wheel: mass 0.3 -> 0.5; geometry collision cylinder length=0.08 radius=0.2; visual cylinder length=0.08 radius=0.2
- link rear_right_wheel: mass 0.3 -> 0.5; geometry collision cylinder length=0.08 radius=0.2; visual cylinder length=0.08 radius=0.2
Joints:
- joint front_left_joint: origin xyz=0.5 0.365 -0.1 rpy=0 0 0 -> xyz=0.5 0.33999999999999997 -0.1 rpy=0 0 0
- joint front_right_joint: origin xyz=0.5 -0.365 -0.1 rpy=0 0 0 -> xyz=0.5 -0.33999999999999997 -0.1 rpy=0 0 0
- joint lidar_joint: origin xyz=0 0 0.14 rpy=0 0 0 -> xyz=0 0 0.16 rpy=0 0 0
- joint rear_left_joint: origin xyz=-0.5 0.365 -0.1 rpy=0 0 0 -> xyz=-0.5 0.33999999999999997 -0.1 rpy=0 0 0
- joint rear_right_joint: origin xyz=-0.5 -0.365 -0.1 rpy=0 0 0 -> xyz=-0.5 -0.33999999999999997 -0.1 rpy=0 0 0

Commit message: Modified codebase

File: src/mobRobURDF_description/urdf/mobRob.urdf (robot description, URDF)
Before this commit: robot mobRob, 8 links, 7 joints
Links:
- removed link front_caster_wheel
- removed link left_wheel
- removed link right_wheel
- added link front_steering_link, mass 0.001
- added link front_wheel, mass 0.5; collision cylinder length=0.12 radius=0.22; visual cylinder length=0.12 radius=0.22
- added link rear_left_wheel, mass 0.5; collision cylinder length=0.12 radius=0.22; visual cylinder length=0.12 radius=0.22
- added link rear_right_wheel, mass 0.5; collision cylinder length=0.12 radius=0.22; visual cylinder length=0.12 radius=0.22
- link chassis: geometry collision box size=1.0 0.5 0.2; visual box size=1.0 0.5 0.2
Joints:
- removed joint front_caster_joint
- removed joint left_joint
- removed joint right_joint
- added joint chassis_to_front_steering: type revolute, parent chassis, child front_steering_link, origin xyz=0.5 0 -0.1 rpy=0 0 0, axis 0 0 1, limit lower=-1.5707963267948966 upper=1.5707963267948966 effort=100 velocity=10
- added joint front_joint: type continuous, parent front_steering_link, child front_wheel, origin xyz=0 0 0 rpy=0 0 0, axis 0 1 0
- added joint rear_left_joint: type continuous, parent chassis, child rear_left_wheel, origin xyz=-0.5 0.31 -0.1 rpy=0 0 0, axis 0 1 0
- added joint rear_right_joint: type continuous, parent chassis, child rear_right_wheel, origin xyz=-0.5 -0.31 -0.1 rpy=0 0 0, axis 0 1 0
- joint base_to_chassis: origin xyz=0 0 0.15 rpy=0 0 0 -> xyz=0 0 0.1 rpy=0 0 0
- joint camera_joint: origin xyz=0.64 0 0 rpy=0 0 0 -> xyz=0.54 0 0 rpy=0 0 0
- joint lidar_joint: origin xyz=0 0 0.19 rpy=0 0 0 -> xyz=0 0 0.14 rpy=0 0 0

Commit message: Enhancement in the view

File: src/mobRobURDF_description/urdf/mobRob.urdf (robot description, URDF)
Before this commit: robot mobRob, 9 links, 8 joints
Links:
- link chassis: geometry collision box size=1.2 0.8 0.3; visual box size=1.2 0.8 0.3
- link lidar: geometry collision cylinder length=0.2 radius=0.1; visual cylinder length=0.2 radius=0.1
Joints:
- joint base_to_chassis: origin xyz=0 0 0.1 rpy=0 0 0 -> xyz=0 0 0.15 rpy=0 0 0
- joint camera_joint: origin xyz=0.54 0 0 rpy=0 0 0 -> xyz=0.64 0 0 rpy=0 0 0
- joint chassis_to_front_steering: origin xyz=0.5 0 -0.1 rpy=0 0 0 -> xyz=0.6 0 -0.15 rpy=0 0 0
- joint lidar_joint: origin xyz=0 0 0.14 rpy=0 0 0 -> xyz=0 0 0.25 rpy=0 0 0
- joint rear_left_joint: origin xyz=-0.5 0.31 -0.1 rpy=0 0 0 -> xyz=-0.6 0.46 -0.15 rpy=0 0 0
- joint rear_right_joint: origin xyz=-0.5 -0.31 -0.1 rpy=0 0 0 -> xyz=-0.6 -0.46 -0.15 rpy=0 0 0

Commit message: Adjustments for saving

File: src/mobRobURDF_description/urdf/mobRob.urdf (robot description, URDF)
Before this commit: robot mobRob, 9 links, 8 joints
Links:
- link camera: geometry collision box size=0.3 0.3 0.3; visual box size=0.3 0.3 0.3
Joints:
- joint camera_joint: origin xyz=0.64 0 0 rpy=0 0 0 -> xyz=0.75 0 0 rpy=0 0 0

Commit message: Fixed xacro files

File: src/mobRobURDF_description/urdf/mobRob.urdf (robot description, URDF)
Before this commit: robot mobRob, 9 links, 8 joints
Links:
- link camera: geometry collision box size=0.08 0.2 0.08; visual box size=0.08 0.2 0.08
- link front_wheel: geometry collision cylinder length=0.12 radius=0.2; visual cylinder length=0.12 radius=0.2
- link rear_left_wheel: geometry collision cylinder length=0.12 radius=0.2; visual cylinder length=0.12 radius=0.2
- link rear_right_wheel: geometry collision cylinder length=0.12 radius=0.2; visual cylinder length=0.12 radius=0.2
Joints:
- joint camera_joint: origin xyz=0.75 0 0 rpy=0 0 0 -> xyz=0.64 0 0.10999999999999999 rpy=0 0 0
- joint rear_left_joint: origin xyz=-0.6 0.46 -0.15 rpy=0 0 0 -> xyz=-0.4666666666666667 0.46 -0.15 rpy=0 0 0
- joint rear_right_joint: origin xyz=-0.6 -0.46 -0.15 rpy=0 0 0 -> xyz=-0.4666666666666667 -0.46 -0.15 rpy=0 0 0

File: src/mobRobURDF_description/urdf/submodules/2_wheeled_caster/mobRob.xacro (robot description, xacro)
@@ -15,5 +15,5 @@
   <xacro:wheel name="left" radius="${wheel_radius}" width="${wheel_width}" mass="${wheel_mass}" material="${wheel_material}" x="${l_x}" y="${l_y}" z="${l_z}" />
   <xacro:wheel name="right" radius="${wheel_radius}" width="${wheel_width}" mass="${wheel_mass}" material="${wheel_material}" x="${r_x}" y="${r_y}" z="${r_z}" />
-  <xacro:caster name="front_caster" radius="${wheel_radius}" mass="${wheel_mass}" material="${wheel_material}" x="${caster_x}" y="${caster_y}" z="${caster_z}" />
+  <xacro:caster name="front_caster" radius="${caster_radius}" mass="${wheel_mass}" material="${wheel_material}" x="${caster_x}" y="${caster_y}" z="${caster_z}" />
   <!-- Sensors -->
   <xacro:lidar radius="${lidar_radius}" height="${lidar_height}" mass="${lidar_mass}" material="${lidar_material}" z="${lidar_z}" />

File: src/mobRobURDF_description/urdf/submodules/3_wheeled/mobRob.xacro (robot description, xacro)
@@ -18,4 +18,4 @@
   <!-- Sensors -->
   <xacro:lidar radius="${lidar_radius}" height="${lidar_height}" mass="${lidar_mass}" material="${lidar_material}" z="${lidar_z}" />
-  <xacro:camera size="${camera_size}" mass="${camera_mass}" material="${camera_material}" x="${camera_x}" />
+  <xacro:camera size="${camera_size}" mass="${camera_mass}" material="${camera_material}" x="${camera_x}" z="${camera_z}" />
 </robot>

File: src/mobRobURDF_description/urdf/submodules/3_wheeled/sensors.xacro (robot description, xacro)
@@ -33,5 +33,5 @@
   </xacro:macro>
   <!-- Camera Macro -->
-  <xacro:macro name="camera" params="size mass material x">
+  <xacro:macro name="camera" params="size mass material x z">
     <!-- Split the size string into individual components and convert to floats -->
     <xacro:property name="size_list" value="${list(map(float, size.split()))}" />
@@ -64,5 +64,5 @@
       <parent link="chassis" />
       <child link="camera" />
-      <origin xyz="${x} 0 0" rpy="0 0 0" />
+      <origin xyz="${x} 0 ${z}" rpy="0 0 0" />
     </joint>
     <!-- Camera Optical Frame -->

Commit message: Edited navigation in nav bar

File: src/mobRobURDF_description/urdf/mobRob.urdf (robot description, URDF)
Before this commit: robot mobRob, 9 links, 8 joints
Links:
- removed link front_steering_link
- removed link front_wheel
- added link front_left_wheel, mass 0.5; collision cylinder length=0.12 radius=0.22; visual cylinder length=0.12 radius=0.22
- added link front_right_wheel, mass 0.5; collision cylinder length=0.12 radius=0.22; visual cylinder length=0.12 radius=0.22
- link rear_left_wheel: geometry collision cylinder length=0.12 radius=0.22; visual cylinder length=0.12 radius=0.22
- link rear_right_wheel: geometry collision cylinder length=0.12 radius=0.22; visual cylinder length=0.12 radius=0.22
Joints:
- removed joint chassis_to_front_steering
- removed joint front_joint
- added joint front_left_joint: type continuous, parent chassis, child front_left_wheel, origin xyz=0.4533333333333333 0.46 -0.15 rpy=0 0 0, axis 0 1 0
- added joint front_right_joint: type continuous, parent chassis, child front_right_wheel, origin xyz=0.4533333333333333 -0.46 -0.15 rpy=0 0 0, axis 0 1 0
- joint camera_joint: origin xyz=0.64 0 0.10999999999999999 rpy=0 0 0 -> xyz=0.64 0 0 rpy=0 0 0
- joint rear_left_joint: origin xyz=-0.4666666666666667 0.46 -0.15 rpy=0 0 0 -> xyz=-0.4533333333333333 0.46 -0.15 rpy=0 0 0
- joint rear_right_joint: origin xyz=-0.4666666666666667 -0.46 -0.15 rpy=0 0 0 -> xyz=-0.4533333333333333 -0.46 -0.15 rpy=0 0 0
