Commit message: Organized files

File: src/mobRobURDF_description/urdf/mobRob.urdf (robot description, URDF)
Before this commit: robot mobRob, 9 links, 8 joints
Links:
- removed link front_left_wheel
- removed link front_right_wheel
- removed link rear_left_wheel
- removed link rear_right_wheel
- added link front_caster_wheel, mass 0.5; collision sphere radius=0.22; visual sphere radius=0.22
- added link left_wheel, mass 0.5; collision cylinder length=0.12 radius=0.22; visual cylinder length=0.12 radius=0.22
- added link right_wheel, mass 0.5; collision cylinder length=0.12 radius=0.22; visual cylinder length=0.12 radius=0.22
Joints:
- removed joint front_left_joint
- removed joint front_right_joint
- removed joint rear_left_joint
- removed joint rear_right_joint
- added joint front_caster_joint: type fixed, parent chassis, child front_caster_wheel, origin xyz=0.38 0 -0.15 rpy=0 0 0
- added joint left_joint: type continuous, parent chassis, child left_wheel, origin xyz=-0.3 0.46 -0.15 rpy=0 0 0, axis 0 1 0
- added joint right_joint: type continuous, parent chassis, child right_wheel, origin xyz=-0.3 -0.46 -0.15 rpy=0 0 0, axis 0 1 0

Commit message: Edited images and finalized the work

File: src/mobRobURDF_description/urdf/mobRob.urdf (robot description, URDF)
Before this commit: robot mobRob, 8 links, 7 joints
Links:
- removed link front_caster_wheel
- removed link left_wheel
- removed link right_wheel
- added link front_left_wheel, mass 0.5; collision cylinder length=0.12 radius=0.22; visual cylinder length=0.12 radius=0.22
- added link front_right_wheel, mass 0.5; collision cylinder length=0.12 radius=0.22; visual cylinder length=0.12 radius=0.22
- added link rear_left_wheel, mass 0.5; collision cylinder length=0.12 radius=0.22; visual cylinder length=0.12 radius=0.22
- added link rear_right_wheel, mass 0.5; collision cylinder length=0.12 radius=0.22; visual cylinder length=0.12 radius=0.22
Joints:
- removed joint front_caster_joint
- removed joint left_joint
- removed joint right_joint
- added joint front_left_joint: type continuous, parent chassis, child front_left_wheel, origin xyz=0.4533333333333333 0.46 -0.15 rpy=0 0 0, axis 0 1 0
- added joint front_right_joint: type continuous, parent chassis, child front_right_wheel, origin xyz=0.4533333333333333 -0.46 -0.15 rpy=0 0 0, axis 0 1 0
- added joint rear_left_joint: type continuous, parent chassis, child rear_left_wheel, origin xyz=-0.4533333333333333 0.46 -0.15 rpy=0 0 0, axis 0 1 0
- added joint rear_right_joint: type continuous, parent chassis, child rear_right_wheel, origin xyz=-0.4533333333333333 -0.46 -0.15 rpy=0 0 0, axis 0 1 0

Commit message: Test commit

File: src/mobRobURDF_description/urdf/mobRob.urdf (robot description, URDF)
Before this commit: robot mobRob, 9 links, 8 joints
Links:
- removed link front_left_wheel
- removed link front_right_wheel
- added link front_steering_link, mass 0.001
- added link front_wheel, mass 0.5; collision cylinder length=0.12 radius=0.2; visual cylinder length=0.12 radius=0.2
- link rear_left_wheel: geometry collision cylinder length=0.12 radius=0.2; visual cylinder length=0.12 radius=0.2
- link rear_right_wheel: geometry collision cylinder length=0.12 radius=0.2; visual cylinder length=0.12 radius=0.2
Joints:
- removed joint front_left_joint
- removed joint front_right_joint
- added joint chassis_to_front_steering: type revolute, parent chassis, child front_steering_link, origin xyz=0.6 0 -0.15 rpy=0 0 0, axis 0 0 1, limit lower=-1.5707963267948966 upper=1.5707963267948966 effort=100 velocity=10
- added joint front_joint: type continuous, parent front_steering_link, child front_wheel, origin xyz=0 0 0 rpy=0 0 0, axis 0 1 0
- joint camera_joint: origin xyz=0.64 0 0 rpy=0 0 0 -> xyz=0.64 0 0.10999999999999999 rpy=0 0 0
- joint rear_left_joint: origin xyz=-0.4533333333333333 0.46 -0.15 rpy=0 0 0 -> xyz=-0.4666666666666667 0.46 -0.15 rpy=0 0 0
- joint rear_right_joint: origin xyz=-0.4533333333333333 -0.46 -0.15 rpy=0 0 0 -> xyz=-0.4666666666666667 -0.46 -0.15 rpy=0 0 0

Commit message: Edited .gitignore file

File: src/mobRobURDF_description/urdf/mobRob.urdf (robot description, URDF)
Before this commit: robot mobRob, 9 links, 8 joints
Links:
- removed link front_steering_link
- removed link front_wheel
- removed link rear_left_wheel
- removed link rear_right_wheel
- added link front_caster_wheel, mass 0.5; collision sphere radius=0.22; visual sphere radius=0.22
- added link left_wheel, mass 0.5; collision cylinder length=0.12 radius=0.22; visual cylinder length=0.12 radius=0.22
- added link right_wheel, mass 0.5; collision cylinder length=0.12 radius=0.22; visual cylinder length=0.12 radius=0.22
Joints:
- removed joint chassis_to_front_steering
- removed joint front_joint
- removed joint rear_left_joint
- removed joint rear_right_joint
- added joint front_caster_joint: type fixed, parent chassis, child front_caster_wheel, origin xyz=0.38 0 -0.15 rpy=0 0 0
- added joint left_joint: type continuous, parent chassis, child left_wheel, origin xyz=-0.3 0.46 -0.15 rpy=0 0 0, axis 0 1 0
- added joint right_joint: type continuous, parent chassis, child right_wheel, origin xyz=-0.3 -0.46 -0.15 rpy=0 0 0, axis 0 1 0
- joint camera_joint: origin xyz=0.64 0 0.10999999999999999 rpy=0 0 0 -> xyz=0.64 0 0 rpy=0 0 0

Commit message: Enhanced 2_wheeled_caster robot type (3-DOF caster)

File: src/mobRobURDF_description/urdf/mobRob.urdf (robot description, URDF)
Before this commit: robot mobRob, 8 links, 7 joints
Links:
- added link free-rotating_x_link, mass 0.001
- added link free-rotating_y_link, mass 0.001
Joints:
- added joint free-rotating_x_joint: type continuous, parent chassis, child free-rotating_x_link, origin xyz=0.38 0 -0.15 rpy=0 0 0, axis 1 0 0
- added joint free-rotating_y_joint: type continuous, parent free-rotating_x_link, child free-rotating_y_link, origin xyz=0 0 0 rpy=0 0 0, axis 0 1 0
- joint front_caster_joint: axis (none) -> 0 0 1; origin xyz=0.38 0 -0.15 rpy=0 0 0 -> xyz=0 0 0 rpy=0 0 0; parent chassis -> free-rotating_y_link; type fixed -> continuous

File: src/mobRobURDF_description/urdf/submodules/2_wheeled_caster/base.xacro (robot description, xacro)
@@ -11,4 +11,5 @@
     <xacro:property name="w" value="${size_list[1]}" />
     <xacro:property name="h" value="${size_list[2]}" />
+    <!-- Chassis Link -->
     <link name="chassis">
       <inertial>

File: src/mobRobURDF_description/urdf/submodules/2_wheeled_caster/wheels.xacro (robot description, xacro)
@@ -39,5 +39,5 @@
         <mass value="${mass}" />
         <origin xyz="0 0 0" rpy="0 0 0" />
-        <!-- Use the sphere_inertia macro from inertial_macros.xacro (assumed to exist) -->
+        <!-- Use the sphere_inertia macro from inertial_macros.xacro -->
         <xacro:sphere_inertia mass="${mass}" r="${radius}" />
       </inertial>
@@ -56,8 +56,39 @@
       </collision>
     </link>
-    <joint name="${name}_joint" type="fixed">
+    <joint name="${name}_joint" type="continuous">
+      <parent link="free-rotating_y_link" />
+      <child link="${name}_wheel" />
+      <origin xyz="0 0 0" rpy="0 0 0" />
+      <axis xyz="0 0 1" />
+    </joint>
+    <!-- Front free-rotating Link (around y) for 2-Wheeled Robot -->
+    <link name="free-rotating_y_link">
+      <!-- No mass or geometry needed -->
+      <inertial>
+        <mass value="0.001" /> <!-- Minimal mass to avoid simulation issues -->
+        <origin xyz="0 0 0" rpy="0 0 0" />
+        <inertia ixx="1e-6" ixy="0" ixz="0" iyy="1e-6" iyz="0" izz="1e-6" />
+      </inertial>
+    </link>
+    <joint name="free-rotating_y_joint" type="continuous">
+      <parent link="free-rotating_x_link" />
+      <child link="free-rotating_y_link" />
+      <origin xyz="0 0 0" rpy="0 0 0" />
+      <axis xyz="0 1 0" />
+    </joint>
+    <!-- Front free-rotating Link (around x) for 2-Wheeled Robot -->
+    <link name="free-rotating_x_link">
+      <!-- No mass or geometry needed -->
+      <inertial>
+        <mass value="0.001" /> <!-- Minimal mass to avoid simulation issues -->
+        <origin xyz="0 0 0" rpy="0 0 0" />
+        <inertia ixx="1e-6" ixy="0" ixz="0" iyy="1e-6" iyz="0" izz="1e-6" />
+      </inertial>
+    </link>
+    <joint name="free-rotating_x_joint" type="continuous">
       <parent link="chassis" />
-      <child link="${name}_wheel" />
+      <child link="free-rotating_x_link" />
       <origin xyz="${x} ${y} ${z}" rpy="0 0 0" />
+      <axis xyz="1 0 0" />
     </joint>
   </xacro:macro>

Commit message: Added ackermann-specific urdf files (xacros)

File: src/mobRobURDF_description/urdf/mobRob.urdf (robot description, URDF)
Before this commit: robot mobRob, 10 links, 9 joints
Links:
- removed link free-rotating_x_link
- removed link free-rotating_y_link
- removed link front_caster_wheel
- removed link left_wheel
- removed link right_wheel
- added link front_left_steering_link, mass 0.001
- added link front_left_wheel, mass 0.5; collision cylinder length=0.12 radius=0.22; visual cylinder length=0.12 radius=0.22
- added link front_right_steering_link, mass 0.001
- added link front_right_wheel, mass 0.5; collision cylinder length=0.12 radius=0.22; visual cylinder length=0.12 radius=0.22
- added link rear_left_wheel, mass 0.5; collision cylinder length=0.12 radius=0.22; visual cylinder length=0.12 radius=0.22
- added link rear_right_wheel, mass 0.5; collision cylinder length=0.12 radius=0.22; visual cylinder length=0.12 radius=0.22
Joints:
- removed joint free-rotating_x_joint
- removed joint free-rotating_y_joint
- removed joint front_caster_joint
- removed joint left_joint
- removed joint right_joint
- added joint chassis_to_front_left_steering: type revolute, parent chassis, child front_left_steering_link, origin xyz=0.4533333333333333 0.46 -0.15 rpy=0 0 0, axis 0 0 1, limit lower=-1.5707963267948966 upper=1.5707963267948966 effort=100 velocity=10
- added joint chassis_to_front_right_steering: type revolute, parent chassis, child front_right_steering_link, origin xyz=0.4533333333333333 -0.46 -0.15 rpy=0 0 0, axis 0 0 1, limit lower=-1.5707963267948966 upper=1.5707963267948966 effort=100 velocity=10
- added joint front_left_joint: type continuous, parent front_left_steering_link, child front_left_wheel, origin xyz=0 0 0 rpy=0 0 0, axis 0 1 0
- added joint front_right_joint: type continuous, parent front_right_steering_link, child front_right_wheel, origin xyz=0 0 0 rpy=0 0 0, axis 0 1 0
- added joint rear_left_joint: type continuous, parent chassis, child rear_left_wheel, origin xyz=-0.4533333333333333 0.46 -0.15 rpy=0 0 0, axis 0 1 0
- added joint rear_right_joint: type continuous, parent chassis, child rear_right_wheel, origin xyz=-0.4533333333333333 -0.46 -0.15 rpy=0 0 0, axis 0 1 0

Commit message: Edited buttons of the ControlConfigurationPage.

File: src/mobRobURDF_description/urdf/mobRob.urdf (robot description, URDF)
Before this commit: robot None, 11 links, 10 joints
Links:
- removed link front_left_steering_link
- removed link front_left_wheel
- removed link front_right_steering_link
- removed link front_right_wheel
- removed link rear_left_wheel
- removed link rear_right_wheel
- added link free-rotating_x_link, mass 0.001
- added link free-rotating_y_link, mass 0.001
- added link front_caster_wheel, mass 0.5; collision sphere radius=0.22; visual sphere radius=0.22
- added link left_wheel, mass 0.5; collision cylinder length=0.12 radius=0.22; visual cylinder length=0.12 radius=0.22
- added link right_wheel, mass 0.5; collision cylinder length=0.12 radius=0.22; visual cylinder length=0.12 radius=0.22
Joints:
- removed joint chassis_to_front_left_steering
- removed joint chassis_to_front_right_steering
- removed joint front_left_joint
- removed joint front_right_joint
- removed joint rear_left_joint
- removed joint rear_right_joint
- added joint free-rotating_x_joint: type continuous, parent chassis, child free-rotating_x_link, origin xyz=0.38 0 -0.15 rpy=0 0 0, axis 1 0 0
- added joint free-rotating_y_joint: type continuous, parent free-rotating_x_link, child free-rotating_y_link, origin xyz=0 0 0 rpy=0 0 0, axis 0 1 0
- added joint front_caster_joint: type continuous, parent free-rotating_y_link, child front_caster_wheel, origin xyz=0 0 0 rpy=0 0 0, axis 0 0 1
- added joint left_joint: type continuous, parent chassis, child left_wheel, origin xyz=-0.3 0.46 -0.15 rpy=0 0 0, axis 0 1 0
- added joint right_joint: type continuous, parent chassis, child right_wheel, origin xyz=-0.3 -0.46 -0.15 rpy=0 0 0, axis 0 1 0

File: src/mobRobURDF_description/urdf/mobRob.urdf.xacro (robot description, xacro)
@@ -16,19 +16,17 @@
   <xacro:property name="wheel_mass" value="0.5"/>
   <xacro:property name="wheel_material" value="Black"/>
-  <xacro:property name="fl_x" value="0.4533333333333333"/>
-  <xacro:property name="fl_y" value="0.46"/>
-  <xacro:property name="fl_z" value="-0.15"/>
-  <xacro:property name="fr_x" value="0.4533333333333333"/>
-  <xacro:property name="fr_y" value="-0.46"/>
-  <xacro:property name="fr_z" value="-0.15"/>
-  <xacro:property name="rl_x" value="-0.4533333333333333"/>
-  <xacro:property name="rl_y" value="0.46"/>
-  <xacro:property name="rl_z" value="-0.15"/>
-  <xacro:property name="rr_x" value="-0.4533333333333333"/>
-  <xacro:property name="rr_y" value="-0.46"/>
-  <xacro:property name="rr_z" value="-0.15"/>
+  <xacro:property name="caster_radius" value="0.22"/>
+  <xacro:property name="l_x" value="-0.3"/>
+  <xacro:property name="l_y" value="0.46"/>
+  <xacro:property name="l_z" value="-0.15"/>
+  <xacro:property name="r_x" value="-0.3"/>
+  <xacro:property name="r_y" value="-0.46"/>
+  <xacro:property name="r_z" value="-0.15"/>
+  <xacro:property name="caster_x" value="0.38"/>
+  <xacro:property name="caster_y" value="0"/>
+  <xacro:property name="caster_z" value="-0.15"/>
   <xacro:property name="lidar_z" value="0.19"/>
   <xacro:property name="camera_x" value="0.64"/>
-  <xacro:property name="controller_type" value="ackermann"/>
-  <xacro:include filename="$(find mobRobURDF_description)/urdf/submodules/4_wheeled/ackermann/mobRob_4w_acker.xacro"/>
+  <xacro:property name="controller_type" value="diff_2wc"/>
+  <xacro:include filename="$(find mobRobURDF_description)/urdf/submodules/2_wheeled_caster/mobRob_2wc_diff.xacro"/>
 </robot>

Commit message: Modified the UI (more beautiful, more responsive)

File: src/mobRobURDF_description/urdf/mobRob.urdf (robot description, URDF)
Before this commit: robot None, 10 links, 9 joints
Links:
- removed link free-rotating_x_link
- removed link free-rotating_y_link
- removed link front_caster_wheel
- removed link left_wheel
- removed link right_wheel
- added link front_left_wheel, mass 3; collision cylinder length=0.3 radius=0.5; visual cylinder length=0.3 radius=0.5
- added link front_right_wheel, mass 3; collision cylinder length=0.3 radius=0.5; visual cylinder length=0.3 radius=0.5
- added link rear_left_wheel, mass 3; collision cylinder length=0.3 radius=0.5; visual cylinder length=0.3 radius=0.5
- added link rear_right_wheel, mass 3; collision cylinder length=0.3 radius=0.5; visual cylinder length=0.3 radius=0.5
- link camera: mass 0.1 -> 1; geometry collision box size=0.2 0.2 0.1; visual box size=0.2 0.2 0.1
- link chassis: mass 1.0 -> 10; geometry collision box size=1.0 2.0 1.0; visual box size=1.0 2.0 1.0
- link lidar: mass 0.2 -> 2; geometry collision cylinder length=0.4 radius=0.3; visual cylinder length=0.4 radius=0.3
Joints:
- removed joint free-rotating_x_joint
- removed joint free-rotating_y_joint
- removed joint front_caster_joint
- removed joint left_joint
- removed joint right_joint
- added joint front_left_joint: type continuous, parent chassis, child front_left_wheel, origin xyz=0.16666666666666669 1.15 -0.5 rpy=0 0 0, axis 0 1 0
- added joint front_right_joint: type continuous, parent chassis, child front_right_wheel, origin xyz=0.16666666666666669 -1.15 -0.5 rpy=0 0 0, axis 0 1 0
- added joint rear_left_joint: type continuous, parent chassis, child rear_left_wheel, origin xyz=-0.16666666666666669 1.15 -0.5 rpy=0 0 0, axis 0 1 0
- added joint rear_right_joint: type continuous, parent chassis, child rear_right_wheel, origin xyz=-0.16666666666666669 -1.15 -0.5 rpy=0 0 0, axis 0 1 0
- joint base_to_chassis: origin xyz=0 0 0.15 rpy=0 0 0 -> xyz=0 0 0.5 rpy=0 0 0
- joint camera_joint: origin xyz=0.64 0 0 rpy=0 0 0 -> xyz=0.6 0 0 rpy=0 0 0
- joint lidar_joint: origin xyz=0 0 0.19 rpy=0 0 0 -> xyz=0 0 0.7 rpy=0 0 0

File: src/mobRobURDF_description/urdf/mobRob.urdf.xacro (robot description, xacro)
@@ -2,31 +2,33 @@
 <robot name="mobRob" xmlns:xacro="http://ros.org/wiki/xacro">
   <!-- Xacro parameters -->
-  <xacro:property name="chassis_size" value="1.2 0.8 0.3"/>
-  <xacro:property name="chassis_mass" value="1.0"/>
-  <xacro:property name="chassis_material" value="Gray"/>
-  <xacro:property name="lidar_radius" value="0.1"/>
-  <xacro:property name="lidar_height" value="0.08"/>
-  <xacro:property name="lidar_mass" value="0.2"/>
-  <xacro:property name="lidar_material" value="Red"/>
-  <xacro:property name="camera_size" value="0.08 0.2 0.08"/>
-  <xacro:property name="camera_mass" value="0.1"/>
-  <xacro:property name="camera_material" value="Blue"/>
-  <xacro:property name="wheel_radius" value="0.22"/>
-  <xacro:property name="wheel_width" value="0.12"/>
-  <xacro:property name="wheel_mass" value="0.5"/>
-  <xacro:property name="wheel_material" value="Black"/>
-  <xacro:property name="caster_radius" value="0.22"/>
-  <xacro:property name="l_x" value="-0.3"/>
-  <xacro:property name="l_y" value="0.46"/>
-  <xacro:property name="l_z" value="-0.15"/>
-  <xacro:property name="r_x" value="-0.3"/>
-  <xacro:property name="r_y" value="-0.46"/>
-  <xacro:property name="r_z" value="-0.15"/>
-  <xacro:property name="caster_x" value="0.38"/>
-  <xacro:property name="caster_y" value="0"/>
-  <xacro:property name="caster_z" value="-0.15"/>
-  <xacro:property name="lidar_z" value="0.19"/>
-  <xacro:property name="camera_x" value="0.64"/>
-  <xacro:property name="controller_type" value="diff_2wc"/>
-  <xacro:include filename="$(find mobRobURDF_description)/urdf/submodules/2_wheeled_caster/mobRob_2wc_diff.xacro"/>
+  <xacro:property name="chassis_size" value="1 2 1"/>
+  <xacro:property name="chassis_mass" value="10"/>
+  <xacro:property name="chassis_material" value="Red"/>
+  <xacro:property name="lidar_radius" value="0.3"/>
+  <xacro:property name="lidar_height" value="0.4"/>
+  <xacro:property name="lidar_mass" value="2"/>
+  <xacro:property name="lidar_material" value="Black"/>
+  <xacro:property name="camera_size" value="0.2 0.2 0.1"/>
+  <xacro:property name="camera_mass" value="1"/>
+  <xacro:property name="camera_material" value="Green"/>
+  <xacro:property name="wheel_radius" value="0.5"/>
+  <xacro:property name="wheel_width" value="0.3"/>
+  <xacro:property name="wheel_mass" value="3"/>
+  <xacro:property name="wheel_material" value="Blue"/>
+  <xacro:property name="fl_x" value="0.16666666666666669"/>
+  <xacro:property name="fl_y" value="1.15"/>
+  <xacro:property name="fl_z" value="-0.5"/>
+  <xacro:property name="fr_x" value="0.16666666666666669"/>
+  <xacro:property name="fr_y" value="-1.15"/>
+  <xacro:property name="fr_z" value="-0.5"/>
+  <xacro:property name="rl_x" value="-0.16666666666666669"/>
+  <xacro:property name="rl_y" value="1.15"/>
+  <xacro:property name="rl_z" value="-0.5"/>
+  <xacro:property name="rr_x" value="-0.16666666666666669"/>
+  <xacro:property name="rr_y" value="-1.15"/>
+  <xacro:property name="rr_z" value="-0.5"/>
+  <xacro:property name="lidar_z" value="0.7"/>
+  <xacro:property name="camera_x" value="0.6"/>
+  <xacro:property name="controller_type" value="mecanum"/>
+  <xacro:include filename="$(find mobRobURDF_description)/urdf/submodules/4_wheeled/mobRob_4w_mec.xacro"/>
 </robot>

Commit message: Separated the URDF editor (added its own page)

File: src/mobRobURDF_description/urdf/mobRob.urdf (robot description, URDF)
Before this commit: robot mobRob, 9 links, 8 joints
Joints:
- joint camera_1_joint: origin xyz=0.64 0.0 0.0 rpy=0.0 0.0 0.0 -> xyz=0.0 0.0 0.0 rpy=0.0 0.0 0.0
- joint lidar_1_joint: origin xyz=0.0 0.0 0.19 rpy=0.0 0.0 0.0 -> xyz=0.0 0.0 0.3 rpy=0.0 0.0 0.0

Commit message: Updated the Future Features page

File: src/mobRobURDF_description/urdf/mobRob.urdf (robot description, URDF)
Before this commit: robot mobRob, 9 links, 8 joints
Joints:
- joint camera_1_joint: origin xyz=0.0 0.0 0.0 rpy=0.0 0.0 0.0 -> xyz=0.64 0.0 0.0 rpy=0.0 0.0 0.0
- joint lidar_1_joint: origin xyz=0.0 0.0 0.3 rpy=0.0 0.0 0.0 -> xyz=0.0 0.0 0.19 rpy=0.0 0.0 0.0

Commit message: Added the TeleoperationPage

File: src/mobRobURDF_description/urdf/mobRob.urdf (robot description, URDF)
Before this commit: robot mobRob, 9 links, 8 joints
Links:
- removed link front_left_wheel
- removed link front_right_wheel
- added link front_steering_link, mass 0.001
- added link front_wheel, mass 0.5; collision cylinder length=0.12 radius=0.22; visual cylinder length=0.12 radius=0.22
Joints:
- removed joint front_left_joint
- removed joint front_right_joint
- added joint chassis_to_front_steering: type revolute, parent chassis, child front_steering_link, origin xyz=0.6 0 -0.15 rpy=0 0 0, axis 0 0 1, limit lower=-1.5707963267948966 upper=1.5707963267948966 effort=100 velocity=10
- added joint front_joint: type continuous, parent front_steering_link, child front_wheel, origin xyz=0 0 0 rpy=0 0 0, axis 0 1 0

File: src/mobRobURDF_description/urdf/mobRob.urdf.xacro (robot description, xacro)
@@ -9,10 +9,7 @@
   <xacro:property name="wheel_mass" value="0.5"/>
   <xacro:property name="wheel_material" value="Black"/>
-  <xacro:property name="fl_x" value="0.4533333333333333"/>
-  <xacro:property name="fl_y" value="0.46"/>
-  <xacro:property name="fl_z" value="-0.15"/>
-  <xacro:property name="fr_x" value="0.4533333333333333"/>
-  <xacro:property name="fr_y" value="-0.46"/>
-  <xacro:property name="fr_z" value="-0.15"/>
+  <xacro:property name="front_x" value="0.6"/>
+  <xacro:property name="front_y" value="0"/>
+  <xacro:property name="front_z" value="-0.15"/>
   <xacro:property name="rl_x" value="-0.4533333333333333"/>
   <xacro:property name="rl_y" value="0.46"/>
@@ -21,6 +18,6 @@
   <xacro:property name="rr_y" value="-0.46"/>
   <xacro:property name="rr_z" value="-0.15"/>
-  <xacro:property name="controller_type" value="mecanum"/>
-  <xacro:include filename="$(find mobRobURDF_description)/urdf/submodules/4_wheeled/mobRob_4w_mec.xacro"/>
+  <xacro:property name="controller_type" value="triSteer"/>
+  <xacro:include filename="$(find mobRobURDF_description)/urdf/submodules/3_wheeled/mobRob_3w_triSteer.xacro"/>
   <xacro:include filename="$(find mobRobURDF_description)/urdf/user_sensors.xacro"/>
 </robot>
