Commit message: Added a start page (for starting fresh, or loading a saved session)

File: src/mobRobURDF_description/urdf/mobRob.urdf (robot description, URDF)
Before this commit: robot mobRob, 9 links, 8 joints
Links:
- added link camera_2, mass 0.1; collision box size=0.08 0.08 0.06; visual box size=0.08 0.08 0.06
- added link camera_2_optical
- added link lidar_2, mass 0.1; collision cylinder length=0.08 radius=0.1; visual cylinder length=0.08 radius=0.1
Joints:
- added joint camera_2_joint: type fixed, parent chassis, child camera_2, origin xyz=0.0 0.5 0.0 rpy=0.0 0.0 0.0
- added joint camera_2_optical_joint: type fixed, parent camera_2, child camera_2_optical, origin xyz=0 0 0 rpy=-1.5707963 0 -1.5707963
- added joint lidar_2_joint: type fixed, parent chassis, child lidar_2, origin xyz=0.0 0.2 0.3 rpy=0.0 0.0 0.0

File: src/mobRobURDF_description/urdf/mobRob.urdf.xacro (robot description, xacro)
@@ -18,6 +18,6 @@
   <xacro:property name="rr_y" value="-0.46"/>
   <xacro:property name="rr_z" value="-0.15"/>
-  <xacro:property name="controller_type" value="tricycle"/>
-  <xacro:include filename="$(find mobRobURDF_description)/urdf/submodules/3_wheeled/mobRob_3w_tricycle.xacro"/>
+  <xacro:property name="controller_type" value="triSteer"/>
+  <xacro:include filename="$(find mobRobURDF_description)/urdf/submodules/3_wheeled/mobRob_3w_triSteer.xacro"/>
   <xacro:include filename="$(find mobRobURDF_description)/urdf/user_sensors.xacro"/>
 </robot>
