Commit message: Modified some issues in the FutureFeaturesPage

File: src/mobRobURDF_description/urdf/mobRob.urdf.xacro (robot description, xacro)
@@ -21,6 +21,6 @@
   <xacro:property name="rr_y" value="-0.46"/>
   <xacro:property name="rr_z" value="-0.15"/>
-  <xacro:property name="controller_type" value="diff_4w"/>
-  <xacro:include filename="$(find mobRobURDF_description)/urdf/submodules/4_wheeled/mobRob_4w_diff.xacro"/>
+  <xacro:property name="controller_type" value="mecanum"/>
+  <xacro:include filename="$(find mobRobURDF_description)/urdf/submodules/4_wheeled/mobRob_4w_mec.xacro"/>
   <xacro:include filename="$(find mobRobURDF_description)/urdf/user_sensors.xacro"/>
 </robot>

Commit message: Moved the Start Simulation button (and modfied some issues in URDF)

File: src/mobRobURDF_description/urdf/mobRob.urdf.xacro (robot description, xacro)
@@ -18,6 +18,6 @@
   <xacro:property name="rr_y" value="-0.46"/>
   <xacro:property name="rr_z" value="-0.15"/>
-  <xacro:property name="controller_type" value="triSteer"/>
-  <xacro:include filename="$(find mobRobURDF_description)/urdf/submodules/3_wheeled/mobRob_3w_triSteer.xacro"/>
+  <xacro:property name="controller_type" value="tricycle"/>
+  <xacro:include filename="$(find mobRobURDF_description)/urdf/submodules/3_wheeled/mobRob_3w_tricycle.xacro"/>
   <xacro:include filename="$(find mobRobURDF_description)/urdf/user_sensors.xacro"/>
 </robot>

Commit message: Added units to all the text boxes

File: src/mobRobURDF_description/urdf/mobRob.urdf.xacro (robot description, xacro)
@@ -21,6 +21,8 @@
   <xacro:property name="rr_y" value="-0.46"/>
   <xacro:property name="rr_z" value="-0.15"/>
-  <xacro:property name="controller_type" value="mecanum"/>
-  <xacro:include filename="$(find mobRobURDF_description)/urdf/submodules/4_wheeled/mobRob_4w_mec.xacro"/>
+  <xacro:property name="controller_type" value="diff_4w"/>
+  <xacro:property name="hardware_plugin" value="mock_components/GenericSystem"/>
+  <xacro:property name="use_gazebo_sim" value="0"/>
+  <xacro:include filename="$(find mobRobURDF_description)/urdf/submodules/4_wheeled/mobRob_4w_diff.xacro"/>
   <xacro:include filename="$(find mobRobURDF_description)/urdf/user_sensors.xacro"/>
 </robot>

File: src/mobRobURDF_description/urdf/submodules/2_wheeled_caster/mobRob_2wc_diff.xacro (robot description, xacro)
@@ -14,7 +14,4 @@
   <xacro:wheel name="right" radius="${wheel_radius}" width="${wheel_width}" mass="${wheel_mass}" material="${wheel_material}" x="${r_x}" y="${r_y}" z="${r_z}" />
   <xacro:caster name="front_caster" radius="${caster_radius}" mass="${wheel_mass}" material="${wheel_material}" x="${caster_x}" y="${caster_y}" z="${caster_z}" />
-  <!-- Hardware interface (substituted by the wizard; used by the ros2_control xacro below) -->
-  <xacro:property name="hardware_plugin" value="${hardware_plugin}"/>
-  <xacro:property name="use_gazebo_sim" value="${use_gazebo_sim}"/>
   <!-- Include Gazebo Xacro files -->
   <xacro:include filename="$(find mobRobURDF_description)/urdf/gazebo_files/control/gazebo_ros2_control_2wc_diff.xacro" />

File: src/mobRobURDF_description/urdf/submodules/3_wheeled/mobRob_3w_triSteer.xacro (robot description, xacro)
@@ -14,7 +14,4 @@
   <xacro:wheel name="rear_left" radius="${wheel_radius}" width="${wheel_width}" mass="${wheel_mass}" material="${wheel_material}" x="${rl_x}" y="${rl_y}" z="${rl_z}" parent="chassis" />
   <xacro:wheel name="rear_right" radius="${wheel_radius}" width="${wheel_width}" mass="${wheel_mass}" material="${wheel_material}" x="${rr_x}" y="${rr_y}" z="${rr_z}" parent="chassis" />
-  <!-- Hardware interface (substituted by the wizard; used by the ros2_control xacro below) -->
-  <xacro:property name="hardware_plugin" value="${hardware_plugin}"/>
-  <xacro:property name="use_gazebo_sim" value="${use_gazebo_sim}"/>
   <!-- Include Gazebo Xacro files -->
   <xacro:include filename="$(find mobRobURDF_description)/urdf/gazebo_files/control/gazebo_ros2_control_3w_triSteer.xacro" />

File: src/mobRobURDF_description/urdf/submodules/3_wheeled/mobRob_3w_tricycle.xacro (robot description, xacro)
@@ -14,7 +14,4 @@
   <xacro:wheel name="rear_left" radius="${wheel_radius}" width="${wheel_width}" mass="${wheel_mass}" material="${wheel_material}" x="${rl_x}" y="${rl_y}" z="${rl_z}" parent="chassis" />
   <xacro:wheel name="rear_right" radius="${wheel_radius}" width="${wheel_width}" mass="${wheel_mass}" material="${wheel_material}" x="${rr_x}" y="${rr_y}" z="${rr_z}" parent="chassis" />
-  <!-- Hardware interface (substituted by the wizard; used by the ros2_control xacro below) -->
-  <xacro:property name="hardware_plugin" value="${hardware_plugin}"/>
-  <xacro:property name="use_gazebo_sim" value="${use_gazebo_sim}"/>
   <!-- Include Gazebo Xacro files -->
   <xacro:include filename="$(find mobRobURDF_description)/urdf/gazebo_files/control/gazebo_ros2_control_3w_tricycle.xacro" />

File: src/mobRobURDF_description/urdf/submodules/4_wheeled/ackermann/mobRob_4w_acker.xacro (robot description, xacro)
@@ -15,7 +15,4 @@
   <xacro:wheel name="rear_left" radius="${wheel_radius}" width="${wheel_width}" mass="${wheel_mass}" material="${wheel_material}" x="${rl_x}" y="${rl_y}" z="${rl_z}" parent="chassis" />
   <xacro:wheel name="rear_right" radius="${wheel_radius}" width="${wheel_width}" mass="${wheel_mass}" material="${wheel_material}" x="${rr_x}" y="${rr_y}" z="${rr_z}" parent="chassis" />
-  <!-- Hardware interface (substituted by the wizard; used by the ros2_control xacro below) -->
-  <xacro:property name="hardware_plugin" value="${hardware_plugin}"/>
-  <xacro:property name="use_gazebo_sim" value="${use_gazebo_sim}"/>
   <!-- Include Gazebo Xacro files -->
   <xacro:include filename="$(find mobRobURDF_description)/urdf/gazebo_files/control/gazebo_ros2_control_4w_acker.xacro" />

File: src/mobRobURDF_description/urdf/submodules/4_wheeled/mobRob_4w_diff.xacro (robot description, xacro)
@@ -15,7 +15,4 @@
   <xacro:wheel name="rear_left" radius="${wheel_radius}" width="${wheel_width}" mass="${wheel_mass}" material="${wheel_material}" x="${rl_x}" y="${rl_y}" z="${rl_z}" />
   <xacro:wheel name="rear_right" radius="${wheel_radius}" width="${wheel_width}" mass="${wheel_mass}" material="${wheel_material}" x="${rr_x}" y="${rr_y}" z="${rr_z}" />
-  <!-- Hardware interface (substituted by the wizard; used by the ros2_control xacro below) -->
-  <xacro:property name="hardware_plugin" value="${hardware_plugin}"/>
-  <xacro:property name="use_gazebo_sim" value="${use_gazebo_sim}"/>
   <!-- Include Gazebo Xacro files -->
   <xacro:include filename="$(find mobRobURDF_description)/urdf/gazebo_files/control/gazebo_ros2_control_4w_diff.xacro" />

File: src/mobRobURDF_description/urdf/submodules/4_wheeled/mobRob_4w_mec.xacro (robot description, xacro)
@@ -15,7 +15,4 @@
   <xacro:wheel name="rear_left" radius="${wheel_radius}" width="${wheel_width}" mass="${wheel_mass}" material="${wheel_material}" x="${rl_x}" y="${rl_y}" z="${rl_z}" />
   <xacro:wheel name="rear_right" radius="${wheel_radius}" width="${wheel_width}" mass="${wheel_mass}" material="${wheel_material}" x="${rr_x}" y="${rr_y}" z="${rr_z}" />
-  <!-- Hardware interface (substituted by the wizard; used by the ros2_control xacro below) -->
-  <xacro:property name="hardware_plugin" value="${hardware_plugin}"/>
-  <xacro:property name="use_gazebo_sim" value="${use_gazebo_sim}"/>
   <!-- Include Gazebo Xacro files -->
   <xacro:include filename="$(find mobRobURDF_description)/urdf/gazebo_files/control/gazebo_ros2_control_4w_mec.xacro" />

Commit message: Fixed final bugs and modified the README

File: src/mobRobURDF_description/urdf/mobRob.urdf.xacro (robot description, xacro)
@@ -21,8 +21,8 @@
   <xacro:property name="rr_y" value="-0.46"/>
   <xacro:property name="rr_z" value="-0.15"/>
-  <xacro:property name="controller_type" value="mecanum"/>
+  <xacro:property name="controller_type" value="ackermann"/>
   <xacro:property name="hardware_plugin" value="gz_ros2_control/GazeboSimSystem"/>
   <xacro:property name="use_gazebo_sim" value="1"/>
-  <xacro:include filename="$(find mobRobURDF_description)/urdf/submodules/4_wheeled/mobRob_4w_mec.xacro"/>
+  <xacro:include filename="$(find mobRobURDF_description)/urdf/submodules/4_wheeled/ackermann/mobRob_4w_acker.xacro"/>
   <xacro:include filename="$(find mobRobURDF_description)/urdf/user_sensors.xacro"/>
 </robot>

Commit message: Added top-bar (as info) for all the pages

File: src/mobRobURDF_description/urdf/mobRob.urdf.xacro (robot description, xacro)
@@ -21,8 +21,8 @@
   <xacro:property name="rr_y" value="-0.46"/>
   <xacro:property name="rr_z" value="-0.15"/>
-  <xacro:property name="controller_type" value="ackermann"/>
+  <xacro:property name="controller_type" value="mecanum"/>
   <xacro:property name="hardware_plugin" value="gz_ros2_control/GazeboSimSystem"/>
   <xacro:property name="use_gazebo_sim" value="1"/>
-  <xacro:include filename="$(find mobRobURDF_description)/urdf/submodules/4_wheeled/ackermann/mobRob_4w_acker.xacro"/>
+  <xacro:include filename="$(find mobRobURDF_description)/urdf/submodules/4_wheeled/mobRob_4w_mec.xacro"/>
   <xacro:include filename="$(find mobRobURDF_description)/urdf/user_sensors.xacro"/>
 </robot>

Commit message: Fixed the issue with cmd_vel_timeout of tricycle kinematics

File: src/mobRobURDF_description/urdf/mobRob.urdf.xacro (robot description, xacro)
@@ -9,18 +9,17 @@
   <xacro:property name="wheel_mass" value="0.5"/>
   <xacro:property name="wheel_material" value="Black"/>
-  <xacro:property name="caster_radius" value="0.22"/>
-  <xacro:property name="l_x" value="-0.3"/>
-  <xacro:property name="l_y" value="0.46"/>
-  <xacro:property name="l_z" value="-0.15"/>
-  <xacro:property name="r_x" value="-0.3"/>
-  <xacro:property name="r_y" value="-0.46"/>
-  <xacro:property name="r_z" value="-0.15"/>
-  <xacro:property name="caster_x" value="0.38"/>
-  <xacro:property name="caster_y" value="0"/>
-  <xacro:property name="caster_z" value="-0.15"/>
-  <xacro:property name="controller_type" value="diff_2wc"/>
+  <xacro:property name="front_x" value="0.6"/>
+  <xacro:property name="front_y" value="0"/>
+  <xacro:property name="front_z" value="-0.15"/>
+  <xacro:property name="rl_x" value="-0.4533333333333333"/>
+  <xacro:property name="rl_y" value="0.46"/>
+  <xacro:property name="rl_z" value="-0.15"/>
+  <xacro:property name="rr_x" value="-0.4533333333333333"/>
+  <xacro:property name="rr_y" value="-0.46"/>
+  <xacro:property name="rr_z" value="-0.15"/>
+  <xacro:property name="controller_type" value="triSteer"/>
   <xacro:property name="hardware_plugin" value="gz_ros2_control/GazeboSimSystem"/>
   <xacro:property name="use_gazebo_sim" value="1"/>
-  <xacro:include filename="$(find mobRobURDF_description)/urdf/submodules/2_wheeled_caster/mobRob_2wc_diff.xacro"/>
+  <xacro:include filename="$(find mobRobURDF_description)/urdf/submodules/3_wheeled/mobRob_3w_triSteer.xacro"/>
   <xacro:include filename="$(find mobRobURDF_description)/urdf/user_sensors.xacro"/>
 </robot>

Commit message: Modified max_acceleration and max_deceleration (based on wheel_radius)

File: src/mobRobURDF_description/urdf/mobRob.urdf.xacro (robot description, xacro)
@@ -9,7 +9,10 @@
   <xacro:property name="wheel_mass" value="0.5"/>
   <xacro:property name="wheel_material" value="Black"/>
-  <xacro:property name="front_x" value="0.6"/>
-  <xacro:property name="front_y" value="0"/>
-  <xacro:property name="front_z" value="-0.15"/>
+  <xacro:property name="fl_x" value="0.4533333333333333"/>
+  <xacro:property name="fl_y" value="0.46"/>
+  <xacro:property name="fl_z" value="-0.15"/>
+  <xacro:property name="fr_x" value="0.4533333333333333"/>
+  <xacro:property name="fr_y" value="-0.46"/>
+  <xacro:property name="fr_z" value="-0.15"/>
   <xacro:property name="rl_x" value="-0.4533333333333333"/>
   <xacro:property name="rl_y" value="0.46"/>
@@ -18,8 +21,8 @@
   <xacro:property name="rr_y" value="-0.46"/>
   <xacro:property name="rr_z" value="-0.15"/>
-  <xacro:property name="controller_type" value="triSteer"/>
+  <xacro:property name="controller_type" value="mecanum"/>
   <xacro:property name="hardware_plugin" value="gz_ros2_control/GazeboSimSystem"/>
   <xacro:property name="use_gazebo_sim" value="1"/>
-  <xacro:include filename="$(find mobRobURDF_description)/urdf/submodules/3_wheeled/mobRob_3w_triSteer.xacro"/>
+  <xacro:include filename="$(find mobRobURDF_description)/urdf/submodules/4_wheeled/mobRob_4w_mec.xacro"/>
   <xacro:include filename="$(find mobRobURDF_description)/urdf/user_sensors.xacro"/>
 </robot>

Commit message: Modified the default parameters for sensors and chassis and wheels

File: src/mobRobURDF_description/urdf/mobRob.urdf.xacro (robot description, xacro)
@@ -4,25 +4,23 @@
   <xacro:property name="chassis_size" value="1.2 0.8 0.3"/>
   <xacro:property name="chassis_mass" value="1.0"/>
-  <xacro:property name="chassis_material" value="Gray"/>
+  <xacro:property name="chassis_material" value="Brown"/>
   <xacro:property name="wheel_radius" value="0.22"/>
   <xacro:property name="wheel_width" value="0.12"/>
   <xacro:property name="wheel_mass" value="0.5"/>
-  <xacro:property name="wheel_material" value="Black"/>
-  <xacro:property name="fl_x" value="0.4533333333333333"/>
-  <xacro:property name="fl_y" value="0.46"/>
-  <xacro:property name="fl_z" value="-0.15"/>
-  <xacro:property name="fr_x" value="0.4533333333333333"/>
-  <xacro:property name="fr_y" value="-0.46"/>
-  <xacro:property name="fr_z" value="-0.15"/>
-  <xacro:property name="rl_x" value="-0.4533333333333333"/>
-  <xacro:property name="rl_y" value="0.46"/>
-  <xacro:property name="rl_z" value="-0.15"/>
-  <xacro:property name="rr_x" value="-0.4533333333333333"/>
-  <xacro:property name="rr_y" value="-0.46"/>
-  <xacro:property name="rr_z" value="-0.15"/>
-  <xacro:property name="controller_type" value="mecanum"/>
+  <xacro:property name="wheel_material" value="Dark Gray"/>
+  <xacro:property name="caster_radius" value="0.22"/>
+  <xacro:property name="l_x" value="-0.3"/>
+  <xacro:property name="l_y" value="0.46"/>
+  <xacro:property name="l_z" value="-0.15"/>
+  <xacro:property name="r_x" value="-0.3"/>
+  <xacro:property name="r_y" value="-0.46"/>
+  <xacro:property name="r_z" value="-0.15"/>
+  <xacro:property name="caster_x" value="0.38"/>
+  <xacro:property name="caster_y" value="0"/>
+  <xacro:property name="caster_z" value="-0.15"/>
+  <xacro:property name="controller_type" value="diff_2wc"/>
   <xacro:property name="hardware_plugin" value="gz_ros2_control/GazeboSimSystem"/>
   <xacro:property name="use_gazebo_sim" value="1"/>
-  <xacro:include filename="$(find mobRobURDF_description)/urdf/submodules/4_wheeled/mobRob_4w_mec.xacro"/>
+  <xacro:include filename="$(find mobRobURDF_description)/urdf/submodules/2_wheeled_caster/mobRob_2wc_diff.xacro"/>
   <xacro:include filename="$(find mobRobURDF_description)/urdf/user_sensors.xacro"/>
 </robot>

Commit message: Modified initial rpy of the sensors

File: src/mobRobURDF_description/urdf/mobRob.urdf.xacro (robot description, xacro)
@@ -9,18 +9,20 @@
   <xacro:property name="wheel_mass" value="0.5"/>
   <xacro:property name="wheel_material" value="Dark Gray"/>
-  <xacro:property name="caster_radius" value="0.22"/>
-  <xacro:property name="l_x" value="-0.3"/>
-  <xacro:property name="l_y" value="0.46"/>
-  <xacro:property name="l_z" value="-0.15"/>
-  <xacro:property name="r_x" value="-0.3"/>
-  <xacro:property name="r_y" value="-0.46"/>
-  <xacro:property name="r_z" value="-0.15"/>
-  <xacro:property name="caster_x" value="0.38"/>
-  <xacro:property name="caster_y" value="0"/>
-  <xacro:property name="caster_z" value="-0.15"/>
-  <xacro:property name="controller_type" value="diff_2wc"/>
+  <xacro:property name="fl_x" value="0.4533333333333333"/>
+  <xacro:property name="fl_y" value="0.46"/>
+  <xacro:property name="fl_z" value="-0.15"/>
+  <xacro:property name="fr_x" value="0.4533333333333333"/>
+  <xacro:property name="fr_y" value="-0.46"/>
+  <xacro:property name="fr_z" value="-0.15"/>
+  <xacro:property name="rl_x" value="-0.4533333333333333"/>
+  <xacro:property name="rl_y" value="0.46"/>
+  <xacro:property name="rl_z" value="-0.15"/>
+  <xacro:property name="rr_x" value="-0.4533333333333333"/>
+  <xacro:property name="rr_y" value="-0.46"/>
+  <xacro:property name="rr_z" value="-0.15"/>
+  <xacro:property name="controller_type" value="diff_4w"/>
   <xacro:property name="hardware_plugin" value="gz_ros2_control/GazeboSimSystem"/>
   <xacro:property name="use_gazebo_sim" value="1"/>
-  <xacro:include filename="$(find mobRobURDF_description)/urdf/submodules/2_wheeled_caster/mobRob_2wc_diff.xacro"/>
+  <xacro:include filename="$(find mobRobURDF_description)/urdf/submodules/4_wheeled/mobRob_4w_diff.xacro"/>
   <xacro:include filename="$(find mobRobURDF_description)/urdf/user_sensors.xacro"/>
 </robot>

Commit message: Modified README

File: src/mobRobURDF_description/urdf/mobRob.urdf.xacro (robot description, xacro)
@@ -9,10 +9,7 @@
   <xacro:property name="wheel_mass" value="0.5"/>
   <xacro:property name="wheel_material" value="Dark Gray"/>
-  <xacro:property name="fl_x" value="0.4533333333333333"/>
-  <xacro:property name="fl_y" value="0.46"/>
-  <xacro:property name="fl_z" value="-0.15"/>
-  <xacro:property name="fr_x" value="0.4533333333333333"/>
-  <xacro:property name="fr_y" value="-0.46"/>
-  <xacro:property name="fr_z" value="-0.15"/>
+  <xacro:property name="front_x" value="0.6"/>
+  <xacro:property name="front_y" value="0"/>
+  <xacro:property name="front_z" value="-0.15"/>
   <xacro:property name="rl_x" value="-0.4533333333333333"/>
   <xacro:property name="rl_y" value="0.46"/>
@@ -21,8 +18,8 @@
   <xacro:property name="rr_y" value="-0.46"/>
   <xacro:property name="rr_z" value="-0.15"/>
-  <xacro:property name="controller_type" value="ackermann"/>
+  <xacro:property name="controller_type" value="tricycle"/>
   <xacro:property name="hardware_plugin" value="gz_ros2_control/GazeboSimSystem"/>
   <xacro:property name="use_gazebo_sim" value="1"/>
-  <xacro:include filename="$(find mobRobURDF_description)/urdf/submodules/4_wheeled/ackermann/mobRob_4w_acker.xacro"/>
+  <xacro:include filename="$(find mobRobURDF_description)/urdf/submodules/3_wheeled/mobRob_3w_tricycle.xacro"/>
   <xacro:include filename="$(find mobRobURDF_description)/urdf/user_sensors.xacro"/>
 </robot>

Commit message: Small fix to the readme file

File: src/mobRobURDF_description/urdf/mobRob.urdf.xacro (robot description, xacro)
@@ -21,8 +21,8 @@
   <xacro:property name="rr_y" value="-0.46"/>
   <xacro:property name="rr_z" value="-0.15"/>
-  <xacro:property name="controller_type" value="diff_4w"/>
+  <xacro:property name="controller_type" value="ackermann"/>
   <xacro:property name="hardware_plugin" value="gz_ros2_control/GazeboSimSystem"/>
   <xacro:property name="use_gazebo_sim" value="1"/>
-  <xacro:include filename="$(find mobRobURDF_description)/urdf/submodules/4_wheeled/mobRob_4w_diff.xacro"/>
+  <xacro:include filename="$(find mobRobURDF_description)/urdf/submodules/4_wheeled/ackermann/mobRob_4w_acker.xacro"/>
   <xacro:include filename="$(find mobRobURDF_description)/urdf/user_sensors.xacro"/>
 </robot>
