Commit message: Modified the controllers

File: src/mobRobURDF_description/urdf/gazebo_files/gazebo_properties.xacro (robot description, xacro)
@@ -8,5 +8,5 @@
     <xacro:property name="wheel_radius" value="${float(wheel_radius)}"/>
     <xacro:property name="wheel_width" value="${float(wheel_width)}"/>
-    <!-- Base link properties (common for all controllers) -->
+    <!-- Base link (never touches ground, no friction needed) -->
     <gazebo reference="base_link">
       <collision>
@@ -14,38 +14,32 @@
           <friction>
             <ode>
-              <mu>0.8</mu>
-              <mu2>0.8</mu2>
+              <mu>0.0</mu>
+              <mu2>0.0</mu2>
             </ode>
           </friction>
-          <contact>
-            <kp>1e6</kp>
-            <kd>1.0</kd>
-            <max_vel>0.1</max_vel>
-            <min_depth>0.001</min_depth>
-          </contact>
-          <bounce>
-            <restitution_coefficient>0.0</restitution_coefficient>
-          </bounce>
         </surface>
       </collision>
     </gazebo>
-    <!-- diff_2wc: 2-wheeled with caster -->
+    <!-- ================================================================
+         diff_2wc: 2-wheeled differential with caster
+         ================================================================ -->
     <xacro:if value="${controller_type == 'diff_2wc'}">
-      <!-- Drive wheels -->
-      <xacro:macro name="drive_wheel_properties" params="wheel_link wheel_joint">
-        <gazebo reference="${wheel_link}">
-          <collision>
-            <surface>
-              <friction>
-                <ode>
-                  <mu>1.0</mu>
-                  <mu2>1.0</mu2>
-                </ode>
-              </friction>
-              <contact>
-                <kp>1e6</kp>
-                <kd>1.0</kd>
-                <max_vel>0.1</max_vel>
-                <min_depth>0.001</min_depth>
+      <xacro:macro name="drive_wheel_2wc" params="wheel_link wheel_joint">
+        <gazebo reference="${wheel_link}">
+          <collision>
+            <surface>
+              <friction>
+                <ode>
+                  <mu>1.0</mu>
+                  <mu2>1.0</mu2>
+                </ode>
+              </friction>
+              <contact>
+                <ode>
+                  <kp>1000000.0</kp>
+                  <kd>100.0</kd>
+                  <max_vel>0.1</max_vel>
+                  <min_depth>0.001</min_depth>
+                </ode>
               </contact>
               <bounce>
@@ -59,7 +53,7 @@
         </gazebo>
       </xacro:macro>
-      <xacro:drive_wheel_properties wheel_link="left_wheel" wheel_joint="left_joint"/>
-      <xacro:drive_wheel_properties wheel_link="right_wheel" wheel_joint="right_joint"/>
-      <!-- Caster (link name is "<caster_name>_wheel", i.e. front_caster_wheel) -->
+      <xacro:drive_wheel_2wc wheel_link="left_wheel"  wheel_joint="left_joint"/>
+      <xacro:drive_wheel_2wc wheel_link="right_wheel" wheel_joint="right_joint"/>
+      <!-- Caster: very low friction so it swivels freely -->
       <gazebo reference="front_caster_wheel">
         <collision>
@@ -67,13 +61,127 @@
             <friction>
               <ode>
-                <mu>0.1</mu>
-                <mu2>0.1</mu2>
+                <mu>0.01</mu>
+                <mu2>0.01</mu2>
               </ode>
             </friction>
             <contact>
-              <kp>1e6</kp>
-              <kd>1.0</kd>
-              <max_vel>0.1</max_vel>
-              <min_depth>0.001</min_depth>
+              <ode>
+                <kp>1000000.0</kp>
+                <kd>100.0</kd>
+                <max_vel>0.1</max_vel>
+                <min_depth>0.001</min_depth>
+              </ode>
+            </contact>
+          </surface>
+        </collision>
+      </gazebo>
+      <gazebo reference="free-rotating_x_joint">
+        <damping>0.01</damping>
+      </gazebo>
+      <gazebo reference="free-rotating_y_joint">
+        <damping>0.01</damping>
+      </gazebo>
+      <gazebo reference="front_caster_joint">
+        <damping>0.01</damping>
+      </gazebo>
+    </xacro:if>
+    <!-- ================================================================
+         diff_4w: 4-wheeled skid-steering differential
+         Skid-steer kinematics require anisotropic friction:
+           fdir1=1 0 0  → μ  applies to rolling direction (high)
+                        → μ2 applies to lateral direction (lower, allows skid-turn)
+         ================================================================ -->
+    <xacro:if value="${controller_type == 'diff_4w'}">
+      <xacro:macro name="skid_wheel" params="wheel_link wheel_joint">
+        <gazebo reference="${wheel_link}">
+          <collision>
+            <surface>
+              <friction>
+                <ode>
+                  <mu>1.5</mu>
+                  <mu2>0.3</mu2>
+                  <fdir1>1 0 0</fdir1>
+                </ode>
+              </friction>
+              <contact>
+                <ode>
+                  <kp>1000000.0</kp>
+                  <kd>100.0</kd>
+                  <max_vel>0.1</max_vel>
+                  <min_depth>0.001</min_depth>
+                </ode>
+              </contact>
+              <bounce>
+                <restitution_coefficient>0.0</restitution_coefficient>
+              </bounce>
+            </surface>
+          </collision>
+        </gazebo>
+        <gazebo reference="${wheel_joint}">
+          <damping>0.1</damping>
+        </gazebo>
+      </xacro:macro>
+      <xacro:skid_wheel wheel_link="front_left_wheel"  wheel_joint="front_left_joint"/>
+      <xacro:skid_wheel wheel_link="front_right_wheel" wheel_joint="front_right_joint"/>
+      <xacro:skid_wheel wheel_link="rear_left_wheel"   wheel_joint="rear_left_joint"/>
+      <xacro:skid_wheel wheel_link="rear_right_wheel"  wheel_joint="rear_right_joint"/>
+    </xacro:if>
+    <!-- ================================================================
+         mecanum: 4-wheeled mecanum drive
+         ================================================================ -->
+    <xacro:if value="${controller_type == 'mecanum'}">
+      <xacro:macro name="mecanum_wheel" params="wheel_link wheel_joint">
+        <gazebo reference="${wheel_link}">
+          <collision>
+            <surface>
+              <friction>
+                <ode>
+                  <mu>1.2</mu>
+                  <mu2>1.2</mu2>
+                </ode>
+              </friction>
+              <contact>
+                <ode>
+                  <kp>1000000.0</kp>
+                  <kd>100.0</kd>
+                  <max_vel>0.1</max_vel>
+                  <min_depth>0.001</min_depth>
+                </ode>
+              </contact>
+              <bounce>
+                <restitution_coefficient>0.0</restitution_coefficient>
+              </bounce>
+            </surface>
+          </collision>
+        </gazebo>
+        <gazebo reference="${wheel_joint}">
+          <damping>0.15</damping>
+        </gazebo>
+      </xacro:macro>
+      <xacro:mecanum_wheel wheel_link="front_left_wheel"  wheel_joint="front_left_joint"/>
+      <xacro:mecanum_wheel wheel_link="front_right_wheel" wheel_joint="front_right_joint"/>
+      <xacro:mecanum_wheel wheel_link="rear_left_wheel"   wheel_joint="rear_left_joint"/>
+      <xacro:mecanum_wheel wheel_link="rear_right_wheel"  wheel_joint="rear_right_joint"/>
+    </xacro:if>
+    <!-- ================================================================
+         tricycle: 3-wheeled tricycle (front wheel drives + steers)
+         ================================================================ -->
+    <xacro:if value="${controller_type == 'tricycle'}">
+      <gazebo reference="front_wheel">
+        <collision>
+          <surface>
+            <friction>
+              <ode>
+                <mu>1.0</mu>
+                <mu2>1.0</mu2>
+              </ode>
+            </friction>
+            <contact>
+              <ode>
+                <kp>1000000.0</kp>
+                <kd>100.0</kd>
+                <max_vel>0.1</max_vel>
+                <min_depth>0.001</min_depth>
+              </ode>
             </contact>
             <bounce>
@@ -83,83 +191,46 @@
         </collision>
       </gazebo>
-      <gazebo reference="free-rotating_x_joint">
-        <damping>0.01</damping>
-      </gazebo>
-      <gazebo reference="free-rotating_y_joint">
-        <damping>0.01</damping>
-      </gazebo>
-      <gazebo reference="front_caster_joint">
-        <damping>0.01</damping>
-      </gazebo>
-    </xacro:if>
-    <!-- diff_4w: 4-wheeled differential -->
-    <xacro:if value="${controller_type == 'diff_4w'}">
-      <xacro:macro name="drive_wheel_properties" params="wheel_link wheel_joint">
-        <gazebo reference="${wheel_link}">
-          <collision>
-            <surface>
-              <friction>
-                <ode>
-                  <mu>1.0</mu>
-                  <mu2>1.0</mu2>
-                </ode>
-              </friction>
-              <contact>
-                <kp>1e6</kp>
-                <kd>1.0</kd>
-                <max_vel>0.1</max_vel>
-                <min_depth>0.001</min_depth>
-              </contact>
-              <bounce>
-                <restitution_coefficient>0.0</restitution_coefficient>
-              </bounce>
-            </surface>
-          </collision>
-        </gazebo>
-        <gazebo reference="${wheel_joint}">
-          <damping>0.1</damping>
-        </gazebo>
-      </xacro:macro>
-      <xacro:drive_wheel_properties wheel_link="front_left_wheel" wheel_joint="front_left_joint"/>
-      <xacro:drive_wheel_properties wheel_link="front_right_wheel" wheel_joint="front_right_joint"/>
-      <xacro:drive_wheel_properties wheel_link="rear_left_wheel" wheel_joint="rear_left_joint"/>
-      <xacro:drive_wheel_properties wheel_link="rear_right_wheel" wheel_joint="rear_right_joint"/>
-    </xacro:if>
-    <!-- mecanum: 4-wheeled mecanum -->
-    <xacro:if value="${controller_type == 'mecanum'}">
-      <xacro:macro name="mecanum_wheel_properties" params="wheel_link wheel_joint">
-        <gazebo reference="${wheel_link}">
-          <collision>
-            <surface>
-              <friction>
-                <ode>
-                  <mu>1.2</mu>
-                  <mu2>1.2</mu2>
-                </ode>
-              </friction>
-              <contact>
-                <kp>1e6</kp>
-                <kd>1.0</kd>
-                <max_vel>0.1</max_vel>
-                <min_depth>0.001</min_depth>
-              </contact>
-              <bounce>
-                <restitution_coefficient>0.0</restitution_coefficient>
-              </bounce>
-            </surface>
-          </collision>
-        </gazebo>
-        <gazebo reference="${wheel_joint}">
-          <damping>0.15</damping>
-        </gazebo>
-      </xacro:macro>
-      <xacro:mecanum_wheel_properties wheel_link="front_left_wheel" wheel_joint="front_left_joint"/>
-      <xacro:mecanum_wheel_properties wheel_link="front_right_wheel" wheel_joint="front_right_joint"/>
-      <xacro:mecanum_wheel_properties wheel_link="rear_left_wheel" wheel_joint="rear_left_joint"/>
-      <xacro:mecanum_wheel_properties wheel_link="rear_right_wheel" wheel_joint="rear_right_joint"/>
-    </xacro:if>
-    <!-- tricycle: 3-wheeled tricycle -->
-    <xacro:if value="${controller_type == 'tricycle'}">
-      <!-- Traction wheel -->
+      <gazebo reference="front_joint">
+        <damping>0.1</damping>
+      </gazebo>
+      <gazebo reference="chassis_to_front_steering">
+        <damping>0.01</damping>
+        <friction>0.3</friction>
+      </gazebo>
+      <xacro:macro name="tricycle_rear_wheel" params="wheel_link wheel_joint">
+        <gazebo reference="${wheel_link}">
+          <collision>
+            <surface>
+              <friction>
+                <ode>
+                  <mu>1.0</mu>
+                  <mu2>1.0</mu2>
+                </ode>
+              </friction>
+              <contact>
+                <ode>
+                  <kp>1000000.0</kp>
+                  <kd>100.0</kd>
+                  <max_vel>0.1</max_vel>
+                  <min_depth>0.001</min_depth>
+                </ode>
+              </contact>
+              <bounce>
+                <restitution_coefficient>0.0</restitution_coefficient>
+              </bounce>
+            </surface>
+          </collision>
+        </gazebo>
+        <gazebo reference="${wheel_joint}">
+          <damping>0.05</damping>
+        </gazebo>
+      </xacro:macro>
+      <xacro:tricycle_rear_wheel wheel_link="rear_left_wheel"  wheel_joint="rear_left_joint"/>
+      <xacro:tricycle_rear_wheel wheel_link="rear_right_wheel" wheel_joint="rear_right_joint"/>
+    </xacro:if>
+    <!-- ================================================================
+         triSteer: 3-wheeled tricycle steering
+         ================================================================ -->
+    <xacro:if value="${controller_type == 'triSteer'}">
       <gazebo reference="front_wheel">
         <collision>
@@ -172,8 +243,10 @@
             </friction>
             <contact>
-              <kp>1e6</kp>
-              <kd>1.0</kd>
-              <max_vel>0.1</max_vel>
-              <min_depth>0.001</min_depth>
+              <ode>
+                <kp>1000000.0</kp>
+                <kd>100.0</kd>
+                <max_vel>0.1</max_vel>
+                <min_depth>0.001</min_depth>
+              </ode>
             </contact>
             <bounce>
@@ -186,87 +259,25 @@
         <damping>0.1</damping>
       </gazebo>
-      <!-- Steering joint -->
-      <gazebo reference="chassis_to_front_steering">
-        <damping>0.01</damping>
-        <friction>0.3</friction>
-      </gazebo>
-      <!-- Rear wheels -->
-      <xacro:macro name="rear_wheel_properties" params="wheel_link wheel_joint">
-        <gazebo reference="${wheel_link}">
-          <collision>
-            <surface>
-              <friction>
-                <ode>
-                  <mu>1.0</mu>
-                  <mu2>1.0</mu2>
-                </ode>
-              </friction>
-              <contact>
-                <kp>1e6</kp>
-                <kd>1.0</kd>
-                <max_vel>0.1</max_vel>
-                <min_depth>0.001</min_depth>
-              </contact>
-              <bounce>
-                <restitution_coefficient>0.0</restitution_coefficient>
-              </bounce>
-            </surface>
-          </collision>
-        </gazebo>
-        <gazebo reference="${wheel_joint}">
-          <damping>0.05</damping>
-        </gazebo>
-      </xacro:macro>
-      <xacro:rear_wheel_properties wheel_link="rear_left_wheel" wheel_joint="rear_left_joint"/>
-      <xacro:rear_wheel_properties wheel_link="rear_right_wheel" wheel_joint="rear_right_joint"/>
-    </xacro:if>
-    <!-- triSteer: 3-wheeled tricycle steering -->
-    <xacro:if value="${controller_type == 'triSteer'}">
-      <!-- Traction wheel -->
-      <gazebo reference="front_wheel">
-        <collision>
-          <surface>
-            <friction>
-              <ode>
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
File: src/mobRobURDF_description/urdf/mobRob.urdf (robot description, URDF)
Before this commit: robot None, 9 links, 8 joints
Links:
- removed link front_left_wheel
- removed link front_right_wheel
- removed link rear_left_wheel
- removed link rear_right_wheel
- added link free-rotating_x_link, mass 0.001
- added link free-rotating_y_link, mass 0.001
- added link front_caster_wheel, mass 0.5; collision sphere radius=0.22; visual sphere radius=0.22
- added link left_wheel, mass 0.5; collision cylinder length=0.12 radius=0.22; visual cylinder length=0.12 radius=0.22
- added link right_wheel, mass 0.5; collision cylinder length=0.12 radius=0.22; visual cylinder length=0.12 radius=0.22
- link camera: mass 1 -> 0.1; geometry collision box size=0.08 0.2 0.08; visual box size=0.08 0.2 0.08
- link chassis: mass 10 -> 1.0; geometry collision box size=1.2 0.8 0.3; visual box size=1.2 0.8 0.3
- link lidar: mass 2 -> 0.2; geometry collision cylinder length=0.08 radius=0.1; visual cylinder length=0.08 radius=0.1
Joints:
- removed joint front_left_joint
- removed joint front_right_joint
- removed joint rear_left_joint
- removed joint rear_right_joint
- added joint free-rotating_x_joint: type continuous, parent chassis, child free-rotating_x_link, origin xyz=0.38 0 -0.15 rpy=0 0 0, axis 1 0 0
- added joint free-rotating_y_joint: type continuous, parent free-rotating_x_link, child free-rotating_y_link, origin xyz=0 0 0 rpy=0 0 0, axis 0 1 0
- added joint front_caster_joint: type continuous, parent free-rotating_y_link, child front_caster_wheel, origin xyz=0 0 0 rpy=0 0 0, axis 0 0 1
- added joint left_joint: type continuous, parent chassis, child left_wheel, origin xyz=-0.3 0.46 -0.15 rpy=0 0 0, axis 0 1 0
- added joint right_joint: type continuous, parent chassis, child right_wheel, origin xyz=-0.3 -0.46 -0.15 rpy=0 0 0, axis 0 1 0
- joint base_to_chassis: origin xyz=0 0 0.5 rpy=0 0 0 -> xyz=0 0 0.15 rpy=0 0 0
- joint camera_joint: origin xyz=0.6 0 0 rpy=0 0 0 -> xyz=0.64 0 0 rpy=0 0 0
- joint lidar_joint: origin xyz=0 0 0.7 rpy=0 0 0 -> xyz=0 0 0.19 rpy=0 0 0

File: src/mobRobURDF_description/urdf/mobRob.urdf.xacro (robot description, xacro)
@@ -2,33 +2,31 @@
 <robot name="mobRob" xmlns:xacro="http://ros.org/wiki/xacro">
   <!-- Xacro parameters -->
-  <xacro:property name="chassis_size" value="1 2 1"/>
-  <xacro:property name="chassis_mass" value="10"/>
-  <xacro:property name="chassis_material" value="Red"/>
-  <xacro:property name="lidar_radius" value="0.3"/>
-  <xacro:property name="lidar_height" value="0.4"/>
-  <xacro:property name="lidar_mass" value="2"/>
-  <xacro:property name="lidar_material" value="Black"/>
-  <xacro:property name="camera_size" value="0.2 0.2 0.1"/>
-  <xacro:property name="camera_mass" value="1"/>
-  <xacro:property name="camera_material" value="Green"/>
-  <xacro:property name="wheel_radius" value="0.5"/>
-  <xacro:property name="wheel_width" value="0.3"/>
-  <xacro:property name="wheel_mass" value="3"/>
-  <xacro:property name="wheel_material" value="Blue"/>
-  <xacro:property name="fl_x" value="0.16666666666666669"/>
-  <xacro:property name="fl_y" value="1.15"/>
-  <xacro:property name="fl_z" value="-0.5"/>
-  <xacro:property name="fr_x" value="0.16666666666666669"/>
-  <xacro:property name="fr_y" value="-1.15"/>
-  <xacro:property name="fr_z" value="-0.5"/>
-  <xacro:property name="rl_x" value="-0.16666666666666669"/>
-  <xacro:property name="rl_y" value="1.15"/>
-  <xacro:property name="rl_z" value="-0.5"/>
-  <xacro:property name="rr_x" value="-0.16666666666666669"/>
-  <xacro:property name="rr_y" value="-1.15"/>
-  <xacro:property name="rr_z" value="-0.5"/>
-  <xacro:property name="lidar_z" value="0.7"/>
-  <xacro:property name="camera_x" value="0.6"/>
-  <xacro:property name="controller_type" value="mecanum"/>
-  <xacro:include filename="$(find mobRobURDF_description)/urdf/submodules/4_wheeled/mobRob_4w_mec.xacro"/>
+  <xacro:property name="chassis_size" value="1.2 0.8 0.3"/>
+  <xacro:property name="chassis_mass" value="1.0"/>
+  <xacro:property name="chassis_material" value="Gray"/>
+  <xacro:property name="lidar_radius" value="0.1"/>
+  <xacro:property name="lidar_height" value="0.08"/>
+  <xacro:property name="lidar_mass" value="0.2"/>
+  <xacro:property name="lidar_material" value="Red"/>
+  <xacro:property name="camera_size" value="0.08 0.2 0.08"/>
+  <xacro:property name="camera_mass" value="0.1"/>
+  <xacro:property name="camera_material" value="Blue"/>
+  <xacro:property name="wheel_radius" value="0.22"/>
+  <xacro:property name="wheel_width" value="0.12"/>
+  <xacro:property name="wheel_mass" value="0.5"/>
+  <xacro:property name="wheel_material" value="Black"/>
+  <xacro:property name="caster_radius" value="0.22"/>
+  <xacro:property name="l_x" value="-0.3"/>
+  <xacro:property name="l_y" value="0.46"/>
+  <xacro:property name="l_z" value="-0.15"/>
+  <xacro:property name="r_x" value="-0.3"/>
+  <xacro:property name="r_y" value="-0.46"/>
+  <xacro:property name="r_z" value="-0.15"/>
+  <xacro:property name="caster_x" value="0.38"/>
+  <xacro:property name="caster_y" value="0"/>
+  <xacro:property name="caster_z" value="-0.15"/>
+  <xacro:property name="lidar_z" value="0.19"/>
+  <xacro:property name="camera_x" value="0.64"/>
+  <xacro:property name="controller_type" value="diff_2wc"/>
+  <xacro:include filename="$(find mobRobURDF_description)/urdf/submodules/2_wheeled_caster/mobRob_2wc_diff.xacro"/>
 </robot>

File: src/mobRobURDF_description/urdf/submodules/2_wheeled_caster/mobRob_2wc_diff.xacro (robot description, xacro)
@@ -27,3 +27,10 @@
   wheel_radius="${wheel_radius}"
   wheel_width="${wheel_width}"/>
+  <xacro:include filename="$(find mobRobURDF_description)/urdf/gazebo_files/gazebo_colors.xacro" />
+  <xacro:gazebo_visual_colors
+  controller_type="${controller_type}"
+  chassis_material="${chassis_material}"
+  wheel_material="${wheel_material}"
+  lidar_material="${lidar_material}"
+  camera_material="${camera_material}"/>
 </robot>

File: src/mobRobURDF_description/urdf/submodules/3_wheeled/mobRob_3w_triSteer.xacro (robot description, xacro)
@@ -27,3 +27,10 @@
   wheel_radius="${wheel_radius}"
   wheel_width="${wheel_width}"/>
+  <xacro:include filename="$(find mobRobURDF_description)/urdf/gazebo_files/gazebo_colors.xacro" />
+  <xacro:gazebo_visual_colors
+  controller_type="${controller_type}"
+  chassis_material="${chassis_material}"
+  wheel_material="${wheel_material}"
+  lidar_material="${lidar_material}"
+  camera_material="${camera_material}"/>
 </robot>

File: src/mobRobURDF_description/urdf/submodules/3_wheeled/mobRob_3w_tricycle.xacro (robot description, xacro)
@@ -27,3 +27,10 @@
   wheel_radius="${wheel_radius}"
   wheel_width="${wheel_width}"/>
+  <xacro:include filename="$(find mobRobURDF_description)/urdf/gazebo_files/gazebo_colors.xacro" />
+  <xacro:gazebo_visual_colors
+  controller_type="${controller_type}"
+  chassis_material="${chassis_material}"
+  wheel_material="${wheel_material}"
+  lidar_material="${lidar_material}"
+  camera_material="${camera_material}"/>
 </robot>

File: src/mobRobURDF_description/urdf/submodules/4_wheeled/ackermann/mobRob_4w_acker.xacro (robot description, xacro)
@@ -28,3 +28,10 @@
   wheel_radius="${wheel_radius}"
   wheel_width="${wheel_width}"/>
+  <xacro:include filename="$(find mobRobURDF_description)/urdf/gazebo_files/gazebo_colors.xacro" />
+  <xacro:gazebo_visual_colors
+  controller_type="${controller_type}"
+  chassis_material="${chassis_material}"
+  wheel_material="${wheel_material}"
+  lidar_material="${lidar_material}"
+  camera_material="${camera_material}"/>
 </robot>
