Commit message: Modified the controllers

File: src/mobRobURDF_description/urdf/submodules/4_wheeled/mobRob_4w_diff.xacro (robot description, xacro)
@@ -28,3 +28,10 @@
   wheel_radius="${wheel_radius}"
   wheel_width="${wheel_width}"/>
+  <xacro:include filename="$(find mobRobURDF_description)/urdf/gazebo_files/gazebo_colors.xacro" />
+  <xacro:gazebo_visual_colors
+  controller_type="${controller_type}"
+  chassis_material="${chassis_material}"
+  wheel_material="${wheel_material}"
+  lidar_material="${lidar_material}"
+  camera_material="${camera_material}"/>
 </robot>

File: src/mobRobURDF_description/urdf/submodules/4_wheeled/mobRob_4w_mec.xacro (robot description, xacro)
@@ -28,3 +28,10 @@
   wheel_radius="${wheel_radius}"
   wheel_width="${wheel_width}"/>
+  <xacro:include filename="$(find mobRobURDF_description)/urdf/gazebo_files/gazebo_colors.xacro" />
+  <xacro:gazebo_visual_colors
+  controller_type="${controller_type}"
+  chassis_material="${chassis_material}"
+  wheel_material="${wheel_material}"
+  lidar_material="${lidar_material}"
+  camera_material="${camera_material}"/>
 </robot>

Commit message: Fixed the issue with mecanum drive + increased frequency of TeleoperationPage

File: src/mobRobURDF_description/urdf/gazebo_files/gazebo_properties.xacro (robot description, xacro)
@@ -129,38 +129,77 @@
     <!-- ================================================================
          mecanum: 4-wheeled mecanum drive
+         Mecanum rollers are at ±45° — simulate with anisotropic friction:
+           fdir1 = high-friction direction (perpendicular to roller axis)
+           mu    = high (1.0)  — grips in fdir1 direction
+           mu2   = very low (0.01) — roller slips freely along the other axis
+         X-pattern roller layout (matching mecanum_drive_controller kinematics):
+           FL + RR: roller axis "1 1 0"  → fdir1 = "1 -1 0"
+           FR + RL: roller axis "1 -1 0" → fdir1 = "1 1 0"
          ================================================================ -->
     <xacro:if value="${controller_type == 'mecanum'}">
-      <xacro:macro name="mecanum_wheel" params="wheel_link wheel_joint">
-        <gazebo reference="${wheel_link}">
-          <collision>
-            <surface>
-              <friction>
-                <ode>
-                  <mu>1.2</mu>
-                  <mu2>1.2</mu2>
-                </ode>
-              </friction>
-              <contact>
-                <ode>
-                  <kp>1000000.0</kp>
-                  <kd>100.0</kd>
-                  <max_vel>0.1</max_vel>
-                  <min_depth>0.001</min_depth>
-                </ode>
-              </contact>
-              <bounce>
-                <restitution_coefficient>0.0</restitution_coefficient>
-              </bounce>
-            </surface>
-          </collision>
-        </gazebo>
-        <gazebo reference="${wheel_joint}">
-          <damping>0.15</damping>
-        </gazebo>
-      </xacro:macro>
-      <xacro:mecanum_wheel wheel_link="front_left_wheel"  wheel_joint="front_left_joint"/>
-      <xacro:mecanum_wheel wheel_link="front_right_wheel" wheel_joint="front_right_joint"/>
-      <xacro:mecanum_wheel wheel_link="rear_left_wheel"   wheel_joint="rear_left_joint"/>
-      <xacro:mecanum_wheel wheel_link="rear_right_wheel"  wheel_joint="rear_right_joint"/>
+      <!-- FL and RR: rollers at +45°, fdir1 perpendicular = "1 -1 0" -->
+      <xacro:macro name="mecanum_wheel_pos45" params="wheel_link wheel_joint">
+        <gazebo reference="${wheel_link}">
+          <collision>
+            <surface>
+              <friction>
+                <ode>
+                  <mu>1.0</mu>
+                  <mu2>0.01</mu2>
+                  <fdir1>1 -1 0</fdir1>
+                </ode>
+              </friction>
+              <contact>
+                <ode>
+                  <kp>1000000.0</kp>
+                  <kd>100.0</kd>
+                  <max_vel>0.1</max_vel>
+                  <min_depth>0.001</min_depth>
+                </ode>
+              </contact>
+              <bounce>
+                <restitution_coefficient>0.0</restitution_coefficient>
+              </bounce>
+            </surface>
+          </collision>
+        </gazebo>
+        <gazebo reference="${wheel_joint}">
+          <damping>0.05</damping>
+        </gazebo>
+      </xacro:macro>
+      <!-- FR and RL: rollers at -45°, fdir1 perpendicular = "1 1 0" -->
+      <xacro:macro name="mecanum_wheel_neg45" params="wheel_link wheel_joint">
+        <gazebo reference="${wheel_link}">
+          <collision>
+            <surface>
+              <friction>
+                <ode>
+                  <mu>1.0</mu>
+                  <mu2>0.01</mu2>
+                  <fdir1>1 1 0</fdir1>
+                </ode>
+              </friction>
+              <contact>
+                <ode>
+                  <kp>1000000.0</kp>
+                  <kd>100.0</kd>
+                  <max_vel>0.1</max_vel>
+                  <min_depth>0.001</min_depth>
+                </ode>
+              </contact>
+              <bounce>
+                <restitution_coefficient>0.0</restitution_coefficient>
+              </bounce>
+            </surface>
+          </collision>
+        </gazebo>
+        <gazebo reference="${wheel_joint}">
+          <damping>0.05</damping>
+        </gazebo>
+      </xacro:macro>
+      <xacro:mecanum_wheel_pos45 wheel_link="front_left_wheel"  wheel_joint="front_left_joint"/>
+      <xacro:mecanum_wheel_neg45 wheel_link="front_right_wheel" wheel_joint="front_right_joint"/>
+      <xacro:mecanum_wheel_neg45 wheel_link="rear_left_wheel"   wheel_joint="rear_left_joint"/>
+      <xacro:mecanum_wheel_pos45 wheel_link="rear_right_wheel"  wheel_joint="rear_right_joint"/>
     </xacro:if>
     <!-- ================================================================

File: src/mobRobURDF_description/urdf/mobRob.urdf (robot description, URDF)
Before this commit: robot mobRob, 11 links, 10 joints
Links:
- removed link front_left_steering_link
- removed link front_right_steering_link
Joints:
- removed joint chassis_to_front_left_steering
- removed joint chassis_to_front_right_steering
- joint front_left_joint: origin xyz=0 0 0 rpy=0 0 0 -> xyz=0.4533333333333333 0.46 -0.15 rpy=0 0 0; parent front_left_steering_link -> chassis
- joint front_right_joint: origin xyz=0 0 0 rpy=0 0 0 -> xyz=0.4533333333333333 -0.46 -0.15 rpy=0 0 0; parent front_right_steering_link -> chassis

File: src/mobRobURDF_description/urdf/mobRob.urdf.xacro (robot description, xacro)
@@ -21,6 +21,6 @@
   <xacro:property name="rr_y" value="-0.46"/>
   <xacro:property name="rr_z" value="-0.15"/>
-  <xacro:property name="controller_type" value="ackermann"/>
-  <xacro:include filename="$(find mobRobURDF_description)/urdf/submodules/4_wheeled/ackermann/mobRob_4w_acker.xacro"/>
+  <xacro:property name="controller_type" value="mecanum"/>
+  <xacro:include filename="$(find mobRobURDF_description)/urdf/submodules/4_wheeled/mobRob_4w_mec.xacro"/>
   <xacro:include filename="$(find mobRobURDF_description)/urdf/user_sensors.xacro"/>
 </robot>

Commit message: Fixed the issue with mecanum kinematics completely

File: src/mobRobURDF_description/urdf/gazebo_files/gazebo_properties.xacro (robot description, xacro)
@@ -1,4 +1,4 @@
 <?xml version="1.0"?>
-<robot xmlns:xacro="http://ros.org/wiki/xacro">
+<robot xmlns:xacro="http://ros.org/wiki/xacro" xmlns:gz="http://gazebosim.org/schema">
   <!-- Macro for Gazebo physical properties -->
   <xacro:macro name="gazebo_physical_properties" params="controller_type chassis_size wheel_radius wheel_width">
@@ -138,5 +138,7 @@
          ================================================================ -->
     <xacro:if value="${controller_type == 'mecanum'}">
-      <!-- FL and RR: rollers at +45°, fdir1 perpendicular = "1 -1 0" -->
+      <!-- FL and RR: rollers at +45°, grip direction fdir1 = "1 -1 0".
+           fdir1 MUST be expressed in the (non-spinning) base_link frame, otherwise
+           it rotates with the wheel and strafing becomes erratic. -->
       <xacro:macro name="mecanum_wheel_pos45" params="wheel_link wheel_joint">
         <gazebo reference="${wheel_link}">
@@ -146,6 +148,6 @@
                 <ode>
                   <mu>1.0</mu>
-                  <mu2>0.01</mu2>
-                  <fdir1>1 -1 0</fdir1>
+                  <mu2>0.0</mu2>
+                  <fdir1 gz:expressed_in="base_link">1 -1 0</fdir1>
                 </ode>
               </friction>
@@ -168,5 +170,7 @@
         </gazebo>
       </xacro:macro>
-      <!-- FR and RL: rollers at -45°, fdir1 perpendicular = "1 1 0" -->
+      <!-- FR and RL: rollers at -45°, grip direction fdir1 = "1 1 0".
+           fdir1 MUST be expressed in the (non-spinning) base_link frame, otherwise
+           it rotates with the wheel and strafing becomes erratic. -->
       <xacro:macro name="mecanum_wheel_neg45" params="wheel_link wheel_joint">
         <gazebo reference="${wheel_link}">
@@ -176,6 +180,6 @@
                 <ode>
                   <mu>1.0</mu>
-                  <mu2>0.01</mu2>
-                  <fdir1>1 1 0</fdir1>
+                  <mu2>0.0</mu2>
+                  <fdir1 gz:expressed_in="base_link">1 1 0</fdir1>
                 </ode>
               </friction>

File: src/mobRobURDF_description/urdf/mobRob.urdf (robot description, URDF)
Before this commit: robot mobRob, 9 links, 8 joints
Links:
- link front_left_wheel: geometry collision sphere radius=0.22; visual cylinder length=0.12 radius=0.22
- link front_right_wheel: geometry collision sphere radius=0.22; visual cylinder length=0.12 radius=0.22
- link rear_left_wheel: geometry collision sphere radius=0.22; visual cylinder length=0.12 radius=0.22
- link rear_right_wheel: geometry collision sphere radius=0.22; visual cylinder length=0.12 radius=0.22

File: src/mobRobURDF_description/urdf/mobRob.urdf.xacro (robot description, xacro)
@@ -1,4 +1,4 @@
 <?xml version="1.0" ?>
-<robot name="mobRob" xmlns:xacro="http://ros.org/wiki/xacro">
+<robot name="mobRob" xmlns:xacro="http://ros.org/wiki/xacro" xmlns:gz="http://gazebosim.org/schema">
   <!-- Xacro parameters -->
   <xacro:property name="chassis_size" value="1.2 0.8 0.3"/>
@@ -21,8 +21,8 @@
   <xacro:property name="rr_y" value="-0.46"/>
   <xacro:property name="rr_z" value="-0.15"/>
-  <xacro:property name="controller_type" value="diff_4w"/>
-  <xacro:property name="hardware_plugin" value="mock_components/GenericSystem"/>
-  <xacro:property name="use_gazebo_sim" value="0"/>
-  <xacro:include filename="$(find mobRobURDF_description)/urdf/submodules/4_wheeled/mobRob_4w_diff.xacro"/>
+  <xacro:property name="controller_type" value="mecanum"/>
+  <xacro:property name="hardware_plugin" value="gz_ros2_control/GazeboSimSystem"/>
+  <xacro:property name="use_gazebo_sim" value="1"/>
+  <xacro:include filename="$(find mobRobURDF_description)/urdf/submodules/4_wheeled/mobRob_4w_mec.xacro"/>
   <xacro:include filename="$(find mobRobURDF_description)/urdf/user_sensors.xacro"/>
 </robot>

File: src/mobRobURDF_description/urdf/submodules/4_wheeled/mobRob_4w_mec.xacro (robot description, xacro)
@@ -10,9 +10,9 @@
   <!-- Define the robot -->
   <xacro:chassis size="${chassis_size}" mass="${chassis_mass}" material="${chassis_material}" />
-  <!-- Wheels -->
-  <xacro:wheel name="front_left" radius="${wheel_radius}" width="${wheel_width}" mass="${wheel_mass}" material="${wheel_material}" x="${fl_x}" y="${fl_y}" z="${fl_z}" />
-  <xacro:wheel name="front_right" radius="${wheel_radius}" width="${wheel_width}" mass="${wheel_mass}" material="${wheel_material}" x="${fr_x}" y="${fr_y}" z="${fr_z}" />
-  <xacro:wheel name="rear_left" radius="${wheel_radius}" width="${wheel_width}" mass="${wheel_mass}" material="${wheel_material}" x="${rl_x}" y="${rl_y}" z="${rl_z}" />
-  <xacro:wheel name="rear_right" radius="${wheel_radius}" width="${wheel_width}" mass="${wheel_mass}" material="${wheel_material}" x="${rr_x}" y="${rr_y}" z="${rr_z}" />
+  <!-- Wheels — sphere collision for reliable mecanum strafing (visual stays a cylinder) -->
+  <xacro:wheel name="front_left" radius="${wheel_radius}" width="${wheel_width}" mass="${wheel_mass}" material="${wheel_material}" x="${fl_x}" y="${fl_y}" z="${fl_z}" collision_geom="sphere" />
+  <xacro:wheel name="front_right" radius="${wheel_radius}" width="${wheel_width}" mass="${wheel_mass}" material="${wheel_material}" x="${fr_x}" y="${fr_y}" z="${fr_z}" collision_geom="sphere" />
+  <xacro:wheel name="rear_left" radius="${wheel_radius}" width="${wheel_width}" mass="${wheel_mass}" material="${wheel_material}" x="${rl_x}" y="${rl_y}" z="${rl_z}" collision_geom="sphere" />
+  <xacro:wheel name="rear_right" radius="${wheel_radius}" width="${wheel_width}" mass="${wheel_mass}" material="${wheel_material}" x="${rr_x}" y="${rr_y}" z="${rr_z}" collision_geom="sphere" />
   <!-- Include Gazebo Xacro files -->
   <xacro:include filename="$(find mobRobURDF_description)/urdf/gazebo_files/control/gazebo_ros2_control_4w_mec.xacro" />

File: src/mobRobURDF_description/urdf/submodules/4_wheeled/wheels.xacro (robot description, xacro)
@@ -4,5 +4,9 @@
   <xacro:include filename="$(find mobRobURDF_description)/urdf/macros/inertial_macros.xacro" />
   <!-- Wheel Macro -->
-  <xacro:macro name="wheel" params="name radius width mass material x y z">
+  <!-- collision_geom: "cylinder" (default) or "sphere". A spherical collision
+       gives a single stable contact point, which the mecanum friction model
+       (anisotropic fdir1) needs to strafe reliably. The visual stays a cylinder
+       so the wheel still looks normal. -->
+  <xacro:macro name="wheel" params="name radius width mass material x y z collision_geom:=cylinder">
     <link name="${name}_wheel">
       <inertial>
@@ -22,5 +26,10 @@
         <origin xyz="0 0 0" rpy="${pi/2} 0 0" />
         <geometry>
-          <cylinder radius="${radius}" length="${width}" />
+          <xacro:if value="${collision_geom == 'sphere'}">
+            <sphere radius="${radius}" />
+          </xacro:if>
+          <xacro:unless value="${collision_geom == 'sphere'}">
+            <cylinder radius="${radius}" length="${width}" />
+          </xacro:unless>
         </geometry>
       </collision>
