Commit message: Added multi-sensor usage and customizable sensors

File: src/mobRobURDF_description/urdf/gazebo_files/gazebo_colors.xacro (robot description, xacro)
@@ -22,11 +22,9 @@
     </gazebo>
   </xacro:macro>
-  <!-- Apply colors to every visual link, selecting wheel names by controller_type. -->
+  <!-- Apply colors to chassis and wheels. Sensor colors are now handled by
+       user_sensors.xacro which is generated per-session by the wizard. -->
   <xacro:macro name="gazebo_visual_colors"
-               params="controller_type chassis_material wheel_material lidar_material camera_material">
-    <!-- Chassis and sensors are the same across all robot types. -->
+               params="controller_type chassis_material wheel_material">
     <xacro:gz_link_color link_name="chassis" color="${chassis_material}"/>
-    <xacro:gz_link_color link_name="lidar"   color="${lidar_material}"/>
-    <xacro:gz_link_color link_name="camera"  color="${camera_material}"/>
     <!-- 4-wheeled robots: diff_4w, mecanum, ackermann -->
     <xacro:if value="${controller_type in ('diff_4w', 'mecanum', 'ackermann')}">

File: src/mobRobURDF_description/urdf/mobRob.urdf (robot description, URDF)
Before this commit: robot None, 10 links, 9 joints
Links:
- removed link camera
- removed link camera_optical
- removed link free-rotating_x_link
- removed link free-rotating_y_link
- removed link front_caster_wheel
- removed link left_wheel
- removed link lidar
- removed link right_wheel
- added link camera_1, mass 0.1; collision box size=0.08 0.08 0.06; visual box size=0.08 0.08 0.06
- added link camera_1_optical
- added link front_left_wheel, mass 0.5; collision cylinder length=0.12 radius=0.22; visual cylinder length=0.12 radius=0.22
- added link front_right_wheel, mass 0.5; collision cylinder length=0.12 radius=0.22; visual cylinder length=0.12 radius=0.22
- added link lidar_1, mass 0.1; collision cylinder length=0.08 radius=0.1; visual cylinder length=0.08 radius=0.1
- added link rear_left_wheel, mass 0.5; collision cylinder length=0.12 radius=0.22; visual cylinder length=0.12 radius=0.22
- added link rear_right_wheel, mass 0.5; collision cylinder length=0.12 radius=0.22; visual cylinder length=0.12 radius=0.22
Joints:
- removed joint camera_joint
- removed joint camera_optical_joint
- removed joint free-rotating_x_joint
- removed joint free-rotating_y_joint
- removed joint front_caster_joint
- removed joint left_joint
- removed joint lidar_joint
- removed joint right_joint
- added joint camera_1_joint: type fixed, parent chassis, child camera_1, origin xyz=0.64 0.0 0.0 rpy=0.0 0.0 0.0
- added joint camera_1_optical_joint: type fixed, parent camera_1, child camera_1_optical, origin xyz=0 0 0 rpy=-1.5707963 0 -1.5707963
- added joint front_left_joint: type continuous, parent chassis, child front_left_wheel, origin xyz=0.4533333333333333 0.46 -0.15 rpy=0 0 0, axis 0 1 0
- added joint front_right_joint: type continuous, parent chassis, child front_right_wheel, origin xyz=0.4533333333333333 -0.46 -0.15 rpy=0 0 0, axis 0 1 0
- added joint lidar_1_joint: type fixed, parent chassis, child lidar_1, origin xyz=0.0 0.0 0.19 rpy=0.0 0.0 0.0
- added joint rear_left_joint: type continuous, parent chassis, child rear_left_wheel, origin xyz=-0.4533333333333333 0.46 -0.15 rpy=0 0 0, axis 0 1 0
- added joint rear_right_joint: type continuous, parent chassis, child rear_right_wheel, origin xyz=-0.4533333333333333 -0.46 -0.15 rpy=0 0 0, axis 0 1 0

File: src/mobRobURDF_description/urdf/mobRob.urdf.xacro (robot description, xacro)
@@ -5,28 +5,22 @@
   <xacro:property name="chassis_mass" value="1.0"/>
   <xacro:property name="chassis_material" value="Gray"/>
-  <xacro:property name="lidar_radius" value="0.1"/>
-  <xacro:property name="lidar_height" value="0.08"/>
-  <xacro:property name="lidar_mass" value="0.2"/>
-  <xacro:property name="lidar_material" value="Red"/>
-  <xacro:property name="camera_size" value="0.08 0.2 0.08"/>
-  <xacro:property name="camera_mass" value="0.1"/>
-  <xacro:property name="camera_material" value="Blue"/>
   <xacro:property name="wheel_radius" value="0.22"/>
   <xacro:property name="wheel_width" value="0.12"/>
   <xacro:property name="wheel_mass" value="0.5"/>
   <xacro:property name="wheel_material" value="Black"/>
-  <xacro:property name="caster_radius" value="0.22"/>
-  <xacro:property name="l_x" value="-0.3"/>
-  <xacro:property name="l_y" value="0.46"/>
-  <xacro:property name="l_z" value="-0.15"/>
-  <xacro:property name="r_x" value="-0.3"/>
-  <xacro:property name="r_y" value="-0.46"/>
-  <xacro:property name="r_z" value="-0.15"/>
-  <xacro:property name="caster_x" value="0.38"/>
-  <xacro:property name="caster_y" value="0"/>
-  <xacro:property name="caster_z" value="-0.15"/>
-  <xacro:property name="lidar_z" value="0.19"/>
-  <xacro:property name="camera_x" value="0.64"/>
-  <xacro:property name="controller_type" value="diff_2wc"/>
-  <xacro:include filename="$(find mobRobURDF_description)/urdf/submodules/2_wheeled_caster/mobRob_2wc_diff.xacro"/>
+  <xacro:property name="fl_x" value="0.4533333333333333"/>
+  <xacro:property name="fl_y" value="0.46"/>
+  <xacro:property name="fl_z" value="-0.15"/>
+  <xacro:property name="fr_x" value="0.4533333333333333"/>
+  <xacro:property name="fr_y" value="-0.46"/>
+  <xacro:property name="fr_z" value="-0.15"/>
+  <xacro:property name="rl_x" value="-0.4533333333333333"/>
+  <xacro:property name="rl_y" value="0.46"/>
+  <xacro:property name="rl_z" value="-0.15"/>
+  <xacro:property name="rr_x" value="-0.4533333333333333"/>
+  <xacro:property name="rr_y" value="-0.46"/>
+  <xacro:property name="rr_z" value="-0.15"/>
+  <xacro:property name="controller_type" value="diff_4w"/>
+  <xacro:include filename="$(find mobRobURDF_description)/urdf/submodules/4_wheeled/mobRob_4w_diff.xacro"/>
+  <xacro:include filename="$(find mobRobURDF_description)/urdf/user_sensors.xacro"/>
 </robot>

File: src/mobRobURDF_description/urdf/submodules/2_wheeled_caster/mobRob_2wc_diff.xacro (robot description, xacro)
@@ -4,5 +4,4 @@
   <xacro:include filename="$(find mobRobURDF_description)/urdf/submodules/2_wheeled_caster/base.xacro" />
   <xacro:include filename="$(find mobRobURDF_description)/urdf/submodules/2_wheeled_caster/wheels.xacro" />
-  <xacro:include filename="$(find mobRobURDF_description)/urdf/submodules/2_wheeled_caster/sensors.xacro" />
   <xacro:include filename="$(find mobRobURDF_description)/urdf/macros/inertial_macros.xacro" />
   <xacro:include filename="$(find mobRobURDF_description)/urdf/macros/material_macros.xacro" />
@@ -15,10 +14,6 @@
   <xacro:wheel name="right" radius="${wheel_radius}" width="${wheel_width}" mass="${wheel_mass}" material="${wheel_material}" x="${r_x}" y="${r_y}" z="${r_z}" />
   <xacro:caster name="front_caster" radius="${caster_radius}" mass="${wheel_mass}" material="${wheel_material}" x="${caster_x}" y="${caster_y}" z="${caster_z}" />
-  <!-- Sensors -->
-  <xacro:lidar radius="${lidar_radius}" height="${lidar_height}" mass="${lidar_mass}" material="${lidar_material}" z="${lidar_z}" />
-  <xacro:camera size="${camera_size}" mass="${camera_mass}" material="${camera_material}" x="${camera_x}" />
   <!-- Include Gazebo Xacro files -->
   <xacro:include filename="$(find mobRobURDF_description)/urdf/gazebo_files/control/gazebo_ros2_control_2wc_diff.xacro" />
-  <xacro:include filename="$(find mobRobURDF_description)/urdf/gazebo_files/gazebo_sensors.xacro" />
   <xacro:include filename="$(find mobRobURDF_description)/urdf/gazebo_files/gazebo_properties.xacro" />
   <xacro:gazebo_physical_properties
@@ -31,6 +26,4 @@
   controller_type="${controller_type}"
   chassis_material="${chassis_material}"
-  wheel_material="${wheel_material}"
-  lidar_material="${lidar_material}"
-  camera_material="${camera_material}"/>
+  wheel_material="${wheel_material}"/>
 </robot>

File: src/mobRobURDF_description/urdf/submodules/3_wheeled/mobRob_3w_triSteer.xacro (robot description, xacro)
@@ -4,5 +4,4 @@
   <xacro:include filename="$(find mobRobURDF_description)/urdf/submodules/3_wheeled/base.xacro" />
   <xacro:include filename="$(find mobRobURDF_description)/urdf/submodules/3_wheeled/wheels.xacro" />
-  <xacro:include filename="$(find mobRobURDF_description)/urdf/submodules/3_wheeled/sensors.xacro" />
   <xacro:include filename="$(find mobRobURDF_description)/urdf/macros/inertial_macros.xacro" />
   <xacro:include filename="$(find mobRobURDF_description)/urdf/macros/material_macros.xacro" />
@@ -15,10 +14,6 @@
   <xacro:wheel name="rear_left" radius="${wheel_radius}" width="${wheel_width}" mass="${wheel_mass}" material="${wheel_material}" x="${rl_x}" y="${rl_y}" z="${rl_z}" parent="chassis" />
   <xacro:wheel name="rear_right" radius="${wheel_radius}" width="${wheel_width}" mass="${wheel_mass}" material="${wheel_material}" x="${rr_x}" y="${rr_y}" z="${rr_z}" parent="chassis" />
-  <!-- Sensors -->
-  <xacro:lidar radius="${lidar_radius}" height="${lidar_height}" mass="${lidar_mass}" material="${lidar_material}" z="${lidar_z}" />
-  <xacro:camera size="${camera_size}" mass="${camera_mass}" material="${camera_material}" x="${camera_x}" z="${camera_z}" />
   <!-- Include Gazebo Xacro files -->
   <xacro:include filename="$(find mobRobURDF_description)/urdf/gazebo_files/control/gazebo_ros2_control_3w_triSteer.xacro" />
-  <xacro:include filename="$(find mobRobURDF_description)/urdf/gazebo_files/gazebo_sensors.xacro" />
   <xacro:include filename="$(find mobRobURDF_description)/urdf/gazebo_files/gazebo_properties.xacro" />
   <xacro:gazebo_physical_properties
@@ -31,6 +26,4 @@
   controller_type="${controller_type}"
   chassis_material="${chassis_material}"
-  wheel_material="${wheel_material}"
-  lidar_material="${lidar_material}"
-  camera_material="${camera_material}"/>
+  wheel_material="${wheel_material}"/>
 </robot>

File: src/mobRobURDF_description/urdf/submodules/3_wheeled/mobRob_3w_tricycle.xacro (robot description, xacro)
@@ -4,5 +4,4 @@
   <xacro:include filename="$(find mobRobURDF_description)/urdf/submodules/3_wheeled/base.xacro" />
   <xacro:include filename="$(find mobRobURDF_description)/urdf/submodules/3_wheeled/wheels.xacro" />
-  <xacro:include filename="$(find mobRobURDF_description)/urdf/submodules/3_wheeled/sensors.xacro" />
   <xacro:include filename="$(find mobRobURDF_description)/urdf/macros/inertial_macros.xacro" />
   <xacro:include filename="$(find mobRobURDF_description)/urdf/macros/material_macros.xacro" />
@@ -15,10 +14,6 @@
   <xacro:wheel name="rear_left" radius="${wheel_radius}" width="${wheel_width}" mass="${wheel_mass}" material="${wheel_material}" x="${rl_x}" y="${rl_y}" z="${rl_z}" parent="chassis" />
   <xacro:wheel name="rear_right" radius="${wheel_radius}" width="${wheel_width}" mass="${wheel_mass}" material="${wheel_material}" x="${rr_x}" y="${rr_y}" z="${rr_z}" parent="chassis" />
-  <!-- Sensors -->
-  <xacro:lidar radius="${lidar_radius}" height="${lidar_height}" mass="${lidar_mass}" material="${lidar_material}" z="${lidar_z}" />
-  <xacro:camera size="${camera_size}" mass="${camera_mass}" material="${camera_material}" x="${camera_x}" z="${camera_z}" />
   <!-- Include Gazebo Xacro files -->
   <xacro:include filename="$(find mobRobURDF_description)/urdf/gazebo_files/control/gazebo_ros2_control_3w_tricycle.xacro" />
-  <xacro:include filename="$(find mobRobURDF_description)/urdf/gazebo_files/gazebo_sensors.xacro" />
   <xacro:include filename="$(find mobRobURDF_description)/urdf/gazebo_files/gazebo_properties.xacro" />
   <xacro:gazebo_physical_properties
@@ -31,6 +26,4 @@
   controller_type="${controller_type}"
   chassis_material="${chassis_material}"
-  wheel_material="${wheel_material}"
-  lidar_material="${lidar_material}"
-  camera_material="${camera_material}"/>
+  wheel_material="${wheel_material}"/>
 </robot>

File: src/mobRobURDF_description/urdf/submodules/4_wheeled/ackermann/mobRob_4w_acker.xacro (robot description, xacro)
@@ -4,5 +4,4 @@
   <xacro:include filename="$(find mobRobURDF_description)/urdf/submodules/4_wheeled/ackermann/base.xacro" />
   <xacro:include filename="$(find mobRobURDF_description)/urdf/submodules/4_wheeled/ackermann/wheels.xacro" />
-  <xacro:include filename="$(find mobRobURDF_description)/urdf/submodules/4_wheeled/ackermann/sensors.xacro" />
   <xacro:include filename="$(find mobRobURDF_description)/urdf/macros/inertial_macros.xacro" />
   <xacro:include filename="$(find mobRobURDF_description)/urdf/macros/material_macros.xacro" />
@@ -16,10 +15,6 @@
   <xacro:wheel name="rear_left" radius="${wheel_radius}" width="${wheel_width}" mass="${wheel_mass}" material="${wheel_material}" x="${rl_x}" y="${rl_y}" z="${rl_z}" parent="chassis" />
   <xacro:wheel name="rear_right" radius="${wheel_radius}" width="${wheel_width}" mass="${wheel_mass}" material="${wheel_material}" x="${rr_x}" y="${rr_y}" z="${rr_z}" parent="chassis" />
-  <!-- Sensors -->
-  <xacro:lidar radius="${lidar_radius}" height="${lidar_height}" mass="${lidar_mass}" material="${lidar_material}" z="${lidar_z}" />
-  <xacro:camera size="${camera_size}" mass="${camera_mass}" material="${camera_material}" x="${camera_x}" />
   <!-- Include Gazebo Xacro files -->
   <xacro:include filename="$(find mobRobURDF_description)/urdf/gazebo_files/control/gazebo_ros2_control_4w_acker.xacro" />
-  <xacro:include filename="$(find mobRobURDF_description)/urdf/gazebo_files/gazebo_sensors.xacro" />
   <xacro:include filename="$(find mobRobURDF_description)/urdf/gazebo_files/gazebo_properties.xacro" />
   <xacro:gazebo_physical_properties
@@ -32,6 +27,4 @@
   controller_type="${controller_type}"
   chassis_material="${chassis_material}"
-  wheel_material="${wheel_material}"
-  lidar_material="${lidar_material}"
-  camera_material="${camera_material}"/>
+  wheel_material="${wheel_material}"/>
 </robot>

File: src/mobRobURDF_description/urdf/submodules/4_wheeled/mobRob_4w_diff.xacro (robot description, xacro)
@@ -4,5 +4,4 @@
   <xacro:include filename="$(find mobRobURDF_description)/urdf/submodules/4_wheeled/base.xacro" />
   <xacro:include filename="$(find mobRobURDF_description)/urdf/submodules/4_wheeled/wheels.xacro" />
-  <xacro:include filename="$(find mobRobURDF_description)/urdf/submodules/4_wheeled/sensors.xacro" />
   <xacro:include filename="$(find mobRobURDF_description)/urdf/macros/inertial_macros.xacro" />
   <xacro:include filename="$(find mobRobURDF_description)/urdf/macros/material_macros.xacro" />
@@ -16,10 +15,6 @@
   <xacro:wheel name="rear_left" radius="${wheel_radius}" width="${wheel_width}" mass="${wheel_mass}" material="${wheel_material}" x="${rl_x}" y="${rl_y}" z="${rl_z}" />
   <xacro:wheel name="rear_right" radius="${wheel_radius}" width="${wheel_width}" mass="${wheel_mass}" material="${wheel_material}" x="${rr_x}" y="${rr_y}" z="${rr_z}" />
-  <!-- Sensors -->
-  <xacro:lidar radius="${lidar_radius}" height="${lidar_height}" mass="${lidar_mass}" material="${lidar_material}" z="${lidar_z}" />
-  <xacro:camera size="${camera_size}" mass="${camera_mass}" material="${camera_material}" x="${camera_x}" />
   <!-- Include Gazebo Xacro files -->
   <xacro:include filename="$(find mobRobURDF_description)/urdf/gazebo_files/control/gazebo_ros2_control_4w_diff.xacro" />
-  <xacro:include filename="$(find mobRobURDF_description)/urdf/gazebo_files/gazebo_sensors.xacro" />
   <xacro:include filename="$(find mobRobURDF_description)/urdf/gazebo_files/gazebo_properties.xacro" />
   <xacro:gazebo_physical_properties
@@ -32,6 +27,4 @@
   controller_type="${controller_type}"
   chassis_material="${chassis_material}"
-  wheel_material="${wheel_material}"
-  lidar_material="${lidar_material}"
-  camera_material="${camera_material}"/>
+  wheel_material="${wheel_material}"/>
 </robot>

File: src/mobRobURDF_description/urdf/submodules/4_wheeled/mobRob_4w_mec.xacro (robot description, xacro)
@@ -4,5 +4,4 @@
   <xacro:include filename="$(find mobRobURDF_description)/urdf/submodules/4_wheeled/base.xacro" />
   <xacro:include filename="$(find mobRobURDF_description)/urdf/submodules/4_wheeled/wheels.xacro" />
-  <xacro:include filename="$(find mobRobURDF_description)/urdf/submodules/4_wheeled/sensors.xacro" />
   <xacro:include filename="$(find mobRobURDF_description)/urdf/macros/inertial_macros.xacro" />
   <xacro:include filename="$(find mobRobURDF_description)/urdf/macros/material_macros.xacro" />
@@ -16,10 +15,6 @@
   <xacro:wheel name="rear_left" radius="${wheel_radius}" width="${wheel_width}" mass="${wheel_mass}" material="${wheel_material}" x="${rl_x}" y="${rl_y}" z="${rl_z}" />
   <xacro:wheel name="rear_right" radius="${wheel_radius}" width="${wheel_width}" mass="${wheel_mass}" material="${wheel_material}" x="${rr_x}" y="${rr_y}" z="${rr_z}" />
-  <!-- Sensors -->
-  <xacro:lidar radius="${lidar_radius}" height="${lidar_height}" mass="${lidar_mass}" material="${lidar_material}" z="${lidar_z}" />
-  <xacro:camera size="${camera_size}" mass="${camera_mass}" material="${camera_material}" x="${camera_x}" />
   <!-- Include Gazebo Xacro files -->
   <xacro:include filename="$(find mobRobURDF_description)/urdf/gazebo_files/control/gazebo_ros2_control_4w_mec.xacro" />
-  <xacro:include filename="$(find mobRobURDF_description)/urdf/gazebo_files/gazebo_sensors.xacro" />
   <xacro:include filename="$(find mobRobURDF_description)/urdf/gazebo_files/gazebo_properties.xacro" />
   <xacro:gazebo_physical_properties
@@ -32,6 +27,4 @@
   controller_type="${controller_type}"
   chassis_material="${chassis_material}"
-  wheel_material="${wheel_material}"
-  lidar_material="${lidar_material}"
-  camera_material="${camera_material}"/>
+  wheel_material="${wheel_material}"/>
 </robot>
