Commit message: Changed chassis to base_link and base_link to base_footprint

File: src/mobRobURDF_description/urdf/gazebo_files/gazebo_colors.xacro (robot description, xacro)
@@ -26,5 +26,5 @@
   <xacro:macro name="gazebo_visual_colors"
                params="controller_type chassis_material wheel_material">
-    <xacro:gz_link_color link_name="chassis" color="${chassis_material}"/>
+    <xacro:gz_link_color link_name="base_link" color="${chassis_material}"/>
     <!-- 4-wheeled robots: diff_4w, mecanum, ackermann -->
     <xacro:if value="${controller_type in ('diff_4w', 'mecanum', 'ackermann')}">

File: src/mobRobURDF_description/urdf/gazebo_files/gazebo_properties.xacro (robot description, xacro)
@@ -8,6 +8,6 @@
     <xacro:property name="wheel_radius" value="${float(wheel_radius)}"/>
     <xacro:property name="wheel_width" value="${float(wheel_width)}"/>
-    <!-- Base link (never touches ground, no friction needed) -->
-    <gazebo reference="base_link">
+    <!-- Base footprint (massless ground-projection frame, never touches ground, no friction needed) -->
+    <gazebo reference="base_footprint">
       <collision>
         <surface>
@@ -31,6 +31,6 @@
               <friction>
                 <ode>
-                  <mu>1.0</mu>
-                  <mu2>1.0</mu2>
+                  <mu>3.0</mu>
+                  <mu2>3.0</mu2>
                 </ode>
               </friction>
@@ -99,6 +99,6 @@
               <friction>
                 <ode>
-                  <mu>1.5</mu>
-                  <mu2>0.3</mu2>
+                  <mu>3.0</mu>
+                  <mu2>0.5</mu2>
                   <fdir1>1 0 0</fdir1>
                 </ode>
@@ -131,6 +131,8 @@
          Mecanum rollers are at ±45° — simulate with anisotropic friction:
            fdir1 = high-friction direction (perpendicular to roller axis)
-           mu    = high (1.0)  — grips in fdir1 direction
-           mu2   = very low (0.01) — roller slips freely along the other axis
+           mu    = 1.0  — grips in fdir1 direction (do NOT crank this up:
+                          the anisotropic mecanum contact is numerically
+                          delicate and high mu makes forward/back drift & slide)
+           mu2   = 0.0 — roller slips freely along the other axis
          X-pattern roller layout (matching mecanum_drive_controller kinematics):
            FL + RR: roller axis "1 1 0"  → fdir1 = "1 -1 0"
@@ -139,5 +141,5 @@
     <xacro:if value="${controller_type == 'mecanum'}">
       <!-- FL and RR: rollers at +45°, grip direction fdir1 = "1 -1 0".
-           fdir1 MUST be expressed in the (non-spinning) base_link frame, otherwise
+           fdir1 MUST be expressed in the (non-spinning) base_footprint frame, otherwise
            it rotates with the wheel and strafing becomes erratic. -->
       <xacro:macro name="mecanum_wheel_pos45" params="wheel_link wheel_joint">
@@ -149,5 +151,5 @@
                   <mu>1.0</mu>
                   <mu2>0.0</mu2>
-                  <fdir1 gz:expressed_in="base_link">1 -1 0</fdir1>
+                  <fdir1 gz:expressed_in="base_footprint">1 -1 0</fdir1>
                 </ode>
               </friction>
@@ -171,5 +173,5 @@
       </xacro:macro>
       <!-- FR and RL: rollers at -45°, grip direction fdir1 = "1 1 0".
-           fdir1 MUST be expressed in the (non-spinning) base_link frame, otherwise
+           fdir1 MUST be expressed in the (non-spinning) base_footprint frame, otherwise
            it rotates with the wheel and strafing becomes erratic. -->
       <xacro:macro name="mecanum_wheel_neg45" params="wheel_link wheel_joint">
@@ -181,5 +183,5 @@
                   <mu>1.0</mu>
                   <mu2>0.0</mu2>
-                  <fdir1 gz:expressed_in="base_link">1 1 0</fdir1>
+                  <fdir1 gz:expressed_in="base_footprint">1 1 0</fdir1>
                 </ode>
               </friction>
@@ -216,6 +218,6 @@
             <friction>
               <ode>
-                <mu>1.0</mu>
-                <mu2>1.0</mu2>
+                <mu>3.0</mu>
+                <mu2>3.0</mu2>
               </ode>
             </friction>
@@ -247,6 +249,6 @@
               <friction>
                 <ode>
-                  <mu>1.0</mu>
-                  <mu2>1.0</mu2>
+                  <mu>3.0</mu>
+                  <mu2>3.0</mu2>
                 </ode>
               </friction>
@@ -281,6 +283,6 @@
             <friction>
               <ode>
-                <mu>1.0</mu>
-                <mu2>1.0</mu2>
+                <mu>3.0</mu>
+                <mu2>3.0</mu2>
               </ode>
             </friction>
@@ -312,6 +314,6 @@
               <friction>
                 <ode>
-                  <mu>1.0</mu>
-                  <mu2>1.0</mu2>
+                  <mu>3.0</mu>
+                  <mu2>3.0</mu2>
                 </ode>
               </friction>
@@ -347,6 +349,6 @@
               <friction>
                 <ode>
-                  <mu>1.0</mu>
-                  <mu2>1.0</mu2>
+                  <mu>3.0</mu>
+                  <mu2>3.0</mu2>
                 </ode>
               </friction>
@@ -385,6 +387,6 @@
               <friction>
                 <ode>
-                  <mu>1.0</mu>
-                  <mu2>1.0</mu2>
+                  <mu>3.0</mu>
+                  <mu2>3.0</mu2>
                 </ode>
               </friction>

File: src/mobRobURDF_description/urdf/mobRob.urdf.xacro (robot description, xacro)
@@ -21,8 +21,8 @@
   <xacro:property name="rr_y" value="-0.46"/>
   <xacro:property name="rr_z" value="-0.15"/>
-  <xacro:property name="controller_type" value="diff_4w"/>
+  <xacro:property name="controller_type" value="mecanum"/>
   <xacro:property name="hardware_plugin" value="gz_ros2_control/GazeboSimSystem"/>
   <xacro:property name="use_gazebo_sim" value="1"/>
-  <xacro:include filename="$(find mobRobURDF_description)/urdf/submodules/4_wheeled/mobRob_4w_diff.xacro"/>
+  <xacro:include filename="$(find mobRobURDF_description)/urdf/submodules/4_wheeled/mobRob_4w_mec.xacro"/>
   <xacro:include filename="$(find mobRobURDF_description)/urdf/user_sensors.xacro"/>
 </robot>

File: src/mobRobURDF_description/urdf/submodules/2_wheeled_caster/base.xacro (robot description, xacro)
@@ -3,14 +3,14 @@
   <!-- Include the inertial_macros.xacro file -->
   <xacro:include filename="$(find mobRobURDF_description)/urdf/macros/inertial_macros.xacro" />
-  <!-- Base Link -->
-  <link name="base_link"></link>
+  <!-- Base Footprint (ground-projected origin; massless, sits where the wheels touch the ground) -->
+  <link name="base_footprint"></link>
   <!-- Chassis Macro -->
-  <xacro:macro name="chassis" params="size mass material">
+  <xacro:macro name="chassis" params="size mass material wheel_radius">
     <xacro:property name="size_list" value="${list(map(float, size.split()))}" />
     <xacro:property name="l" value="${size_list[0]}" />
     <xacro:property name="w" value="${size_list[1]}" />
     <xacro:property name="h" value="${size_list[2]}" />
-    <!-- Chassis Link -->
-    <link name="chassis">
+    <!-- Base Link (physical robot body / chassis) -->
+    <link name="base_link">
       <inertial>
         <mass value="${mass}" />
@@ -32,9 +32,11 @@
       </collision>
     </link>
-    <!-- Fixed Joint between base_link and chassis -->
-    <joint name="base_to_chassis" type="fixed">
-      <parent link="base_link" />
-      <child link="chassis" />
-      <origin xyz="0 0 ${h/2}" rpy="0 0 0" />
+    <!-- Fixed Joint between base_footprint and base_link.
+         Raised by h/2 + wheel_radius so base_footprint lands exactly at the
+         ground contact point (wheel centres sit at z = wheel_radius). -->
+    <joint name="base_footprint_to_base_link" type="fixed">
+      <parent link="base_footprint" />
+      <child link="base_link" />
+      <origin xyz="0 0 ${h/2 + float(wheel_radius)}" rpy="0 0 0" />
     </joint>
   </xacro:macro>

File: src/mobRobURDF_description/urdf/submodules/2_wheeled_caster/mobRob_2wc_diff.xacro (robot description, xacro)
@@ -9,5 +9,5 @@
   <xacro:define_materials/>
   <!-- Define the robot -->
-  <xacro:chassis size="${chassis_size}" mass="${chassis_mass}" material="${chassis_material}" />
+  <xacro:chassis size="${chassis_size}" mass="${chassis_mass}" material="${chassis_material}" wheel_radius="${wheel_radius}" />
   <!-- Wheels -->
   <xacro:wheel name="left" radius="${wheel_radius}" width="${wheel_width}" mass="${wheel_mass}" material="${wheel_material}" x="${l_x}" y="${l_y}" z="${l_z}" />

File: src/mobRobURDF_description/urdf/submodules/2_wheeled_caster/sensors.xacro (robot description, xacro)
@@ -27,5 +27,5 @@
     </link>
     <joint name="lidar_joint" type="fixed">
-      <parent link="chassis" />
+      <parent link="base_link" />
       <child link="lidar" />
       <origin xyz="0 0 ${z}" rpy="0 0 0" />
@@ -62,5 +62,5 @@
     </link>
     <joint name="camera_joint" type="fixed">
-      <parent link="chassis" />
+      <parent link="base_link" />
       <child link="camera" />
       <origin xyz="${x} 0 0" rpy="0 0 0" />

File: src/mobRobURDF_description/urdf/submodules/2_wheeled_caster/wheels.xacro (robot description, xacro)
@@ -27,5 +27,5 @@
     </link>
     <joint name="${name}_joint" type="continuous">
-      <parent link="chassis" />
+      <parent link="base_link" />
       <child link="${name}_wheel" />
       <origin xyz="${x} ${y} ${z}" rpy="0 0 0" />
@@ -87,5 +87,5 @@
     </link>
     <joint name="free-rotating_x_joint" type="continuous">
-      <parent link="chassis" />
+      <parent link="base_link" />
       <child link="free-rotating_x_link" />
       <origin xyz="${x} ${y} ${z}" rpy="0 0 0" />

File: src/mobRobURDF_description/urdf/submodules/3_wheeled/base.xacro (robot description, xacro)
@@ -3,14 +3,14 @@
   <!-- Include the inertial_macros.xacro file -->
   <xacro:include filename="$(find mobRobURDF_description)/urdf/macros/inertial_macros.xacro" />
-  <!-- Base Link -->
-  <link name="base_link"></link>
+  <!-- Base Footprint (ground-projected origin; massless, sits where the wheels touch the ground) -->
+  <link name="base_footprint"></link>
   <!-- Chassis Macro -->
-  <xacro:macro name="chassis" params="size mass material">
+  <xacro:macro name="chassis" params="size mass material wheel_radius">
     <xacro:property name="size_list" value="${list(map(float, size.split()))}" />
     <xacro:property name="l" value="${size_list[0]}" />
     <xacro:property name="w" value="${size_list[1]}" />
     <xacro:property name="h" value="${size_list[2]}" />
-    <!-- Chassis Link -->
-    <link name="chassis">
+    <!-- Base Link (physical robot body / chassis) -->
+    <link name="base_link">
       <inertial>
         <mass value="${mass}" />
@@ -32,9 +32,11 @@
       </collision>
     </link>
-    <!-- Fixed Joint between base_link and chassis -->
-    <joint name="base_to_chassis" type="fixed">
-      <parent link="base_link" />
-      <child link="chassis" />
-      <origin xyz="0 0 ${h/2}" rpy="0 0 0" />
+    <!-- Fixed Joint between base_footprint and base_link.
+         Raised by h/2 + wheel_radius so base_footprint lands exactly at the
+         ground contact point (wheel centres sit at z = wheel_radius). -->
+    <joint name="base_footprint_to_base_link" type="fixed">
+      <parent link="base_footprint" />
+      <child link="base_link" />
+      <origin xyz="0 0 ${h/2 + float(wheel_radius)}" rpy="0 0 0" />
     </joint>
     <!-- Front Steering Link for 3-Wheeled Robot -->
@@ -49,5 +51,5 @@
     <!-- Revolute Joint for Steering (z-axis rotation) -->
     <joint name="chassis_to_front_steering" type="revolute">
-      <parent link="chassis" />
+      <parent link="base_link" />
       <child link="front_steering_link" />
       <origin xyz="${l/2} 0 ${-h/2}" rpy="0 0 0" /> <!-- Position at front wheel base -->

File: src/mobRobURDF_description/urdf/submodules/3_wheeled/mobRob_3w_triSteer.xacro (robot description, xacro)
@@ -9,9 +9,9 @@
   <xacro:define_materials/>
   <!-- Define the robot -->
-  <xacro:chassis size="${chassis_size}" mass="${chassis_mass}" material="${chassis_material}" />
+  <xacro:chassis size="${chassis_size}" mass="${chassis_mass}" material="${chassis_material}" wheel_radius="${wheel_radius}" />
   <!-- Wheels -->
   <xacro:wheel name="front" radius="${wheel_radius}" width="${wheel_width}" mass="${wheel_mass}" material="${wheel_material}" x="0" y="0" z="0" parent="front_steering_link" />
-  <xacro:wheel name="rear_left" radius="${wheel_radius}" width="${wheel_width}" mass="${wheel_mass}" material="${wheel_material}" x="${rl_x}" y="${rl_y}" z="${rl_z}" parent="chassis" />
-  <xacro:wheel name="rear_right" radius="${wheel_radius}" width="${wheel_width}" mass="${wheel_mass}" material="${wheel_material}" x="${rr_x}" y="${rr_y}" z="${rr_z}" parent="chassis" />
+  <xacro:wheel name="rear_left" radius="${wheel_radius}" width="${wheel_width}" mass="${wheel_mass}" material="${wheel_material}" x="${rl_x}" y="${rl_y}" z="${rl_z}" parent="base_link" />
+  <xacro:wheel name="rear_right" radius="${wheel_radius}" width="${wheel_width}" mass="${wheel_mass}" material="${wheel_material}" x="${rr_x}" y="${rr_y}" z="${rr_z}" parent="base_link" />
   <!-- Include Gazebo Xacro files -->
   <xacro:include filename="$(find mobRobURDF_description)/urdf/gazebo_files/control/gazebo_ros2_control_3w_triSteer.xacro" />

File: src/mobRobURDF_description/urdf/submodules/3_wheeled/mobRob_3w_tricycle.xacro (robot description, xacro)
@@ -9,9 +9,9 @@
   <xacro:define_materials/>
   <!-- Define the robot -->
-  <xacro:chassis size="${chassis_size}" mass="${chassis_mass}" material="${chassis_material}" />
+  <xacro:chassis size="${chassis_size}" mass="${chassis_mass}" material="${chassis_material}" wheel_radius="${wheel_radius}" />
   <!-- Wheels -->
   <xacro:wheel name="front" radius="${wheel_radius}" width="${wheel_width}" mass="${wheel_mass}" material="${wheel_material}" x="0" y="0" z="0" parent="front_steering_link" />
-  <xacro:wheel name="rear_left" radius="${wheel_radius}" width="${wheel_width}" mass="${wheel_mass}" material="${wheel_material}" x="${rl_x}" y="${rl_y}" z="${rl_z}" parent="chassis" />
-  <xacro:wheel name="rear_right" radius="${wheel_radius}" width="${wheel_width}" mass="${wheel_mass}" material="${wheel_material}" x="${rr_x}" y="${rr_y}" z="${rr_z}" parent="chassis" />
+  <xacro:wheel name="rear_left" radius="${wheel_radius}" width="${wheel_width}" mass="${wheel_mass}" material="${wheel_material}" x="${rl_x}" y="${rl_y}" z="${rl_z}" parent="base_link" />
+  <xacro:wheel name="rear_right" radius="${wheel_radius}" width="${wheel_width}" mass="${wheel_mass}" material="${wheel_material}" x="${rr_x}" y="${rr_y}" z="${rr_z}" parent="base_link" />
   <!-- Include Gazebo Xacro files -->
   <xacro:include filename="$(find mobRobURDF_description)/urdf/gazebo_files/control/gazebo_ros2_control_3w_tricycle.xacro" />

File: src/mobRobURDF_description/urdf/submodules/3_wheeled/sensors.xacro (robot description, xacro)
@@ -27,5 +27,5 @@
     </link>
     <joint name="lidar_joint" type="fixed">
-      <parent link="chassis" />
+      <parent link="base_link" />
       <child link="lidar" />
       <origin xyz="0 0 ${z}" rpy="0 0 0" />
@@ -62,5 +62,5 @@
     </link>
     <joint name="camera_joint" type="fixed">
-      <parent link="chassis" />
+      <parent link="base_link" />
       <child link="camera" />
       <origin xyz="${x} 0 ${z}" rpy="0 0 0" />

File: src/mobRobURDF_description/urdf/submodules/4_wheeled/ackermann/base.xacro (robot description, xacro)
@@ -3,13 +3,14 @@
   <!-- Include the inertial_macros.xacro file -->
   <xacro:include filename="$(find mobRobURDF_description)/urdf/macros/inertial_macros.xacro" />
-  <!-- Base Link -->
-  <link name="base_link"></link>
+  <!-- Base Footprint (ground-projected origin; massless, sits where the wheels touch the ground) -->
+  <link name="base_footprint"></link>
   <!-- Chassis Macro -->
-  <xacro:macro name="chassis" params="size mass material x_steer y_steer z_steer">
+  <xacro:macro name="chassis" params="size mass material wheel_radius x_steer y_steer z_steer">
     <xacro:property name="size_list" value="${list(map(float, size.split()))}" />
     <xacro:property name="l" value="${size_list[0]}" />
     <xacro:property name="w" value="${size_list[1]}" />
     <xacro:property name="h" value="${size_list[2]}" />
-    <link name="chassis">
+    <!-- Base Link (physical robot body / chassis) -->
+    <link name="base_link">
       <inertial>
         <mass value="${mass}" />
@@ -31,9 +32,11 @@
       </collision>
     </link>
-    <!-- Fixed Joint between base_link and chassis -->
-    <joint name="base_to_chassis" type="fixed">
-      <parent link="base_link" />
-      <child link="chassis" />
-      <origin xyz="0 0 ${h/2}" rpy="0 0 0" />
+    <!-- Fixed Joint between base_footprint and base_link.
+         Raised by h/2 + wheel_radius so base_footprint lands exactly at the
+         ground contact point (wheel centres sit at z = wheel_radius). -->
+    <joint name="base_footprint_to_base_link" type="fixed">
+      <parent link="base_footprint" />
+      <child link="base_link" />
+      <origin xyz="0 0 ${h/2 + float(wheel_radius)}" rpy="0 0 0" />
     </joint>
     <!-- Front Steering Link (Left) for 4-Wheeled Robot (when ackermann control is chosen) -->
@@ -48,5 +51,5 @@
     <!-- Revolute Joint for Steering (z-axis rotation | Left) -->
     <joint name="chassis_to_front_left_steering" type="revolute">
-      <parent link="chassis" />
+      <parent link="base_link" />
       <child link="front_left_steering_link" />
       <origin xyz="${x_steer} ${y_steer} ${z_steer}" rpy="0 0 0" /> <!-- Position at front wheel base -->
@@ -65,5 +68,5 @@
     <!-- Revolute Joint for Steering (z-axis rotation | Right) -->
     <joint name="chassis_to_front_right_steering" type="revolute">
-      <parent link="chassis" />
+      <parent link="base_link" />
       <child link="front_right_steering_link" />
       <origin xyz="${x_steer} -${y_steer} ${z_steer}" rpy="0 0 0" /> <!-- Position at front wheel base -->

File: src/mobRobURDF_description/urdf/submodules/4_wheeled/ackermann/mobRob_4w_acker.xacro (robot description, xacro)
@@ -9,10 +9,10 @@
   <xacro:define_materials/>
   <!-- Define the robot -->
-  <xacro:chassis size="${chassis_size}" mass="${chassis_mass}" material="${chassis_material}" x_steer="${fl_x}" y_steer="${fl_y}" z_steer="${fl_z}" />
+  <xacro:chassis size="${chassis_size}" mass="${chassis_mass}" material="${chassis_material}" wheel_radius="${wheel_radius}" x_steer="${fl_x}" y_steer="${fl_y}" z_steer="${fl_z}" />
   <!-- Wheels -->
   <xacro:wheel name="front_left" radius="${wheel_radius}" width="${wheel_width}" mass="${wheel_mass}" material="${wheel_material}" x="0" y="0" z="0" parent="front_left_steering_link" />
   <xacro:wheel name="front_right" radius="${wheel_radius}" width="${wheel_width}" mass="${wheel_mass}" material="${wheel_material}" x="0" y="0" z="0" parent="front_right_steering_link" />
-  <xacro:wheel name="rear_left" radius="${wheel_radius}" width="${wheel_width}" mass="${wheel_mass}" material="${wheel_material}" x="${rl_x}" y="${rl_y}" z="${rl_z}" parent="chassis" />
-  <xacro:wheel name="rear_right" radius="${wheel_radius}" width="${wheel_width}" mass="${wheel_mass}" material="${wheel_material}" x="${rr_x}" y="${rr_y}" z="${rr_z}" parent="chassis" />
+  <xacro:wheel name="rear_left" radius="${wheel_radius}" width="${wheel_width}" mass="${wheel_mass}" material="${wheel_material}" x="${rl_x}" y="${rl_y}" z="${rl_z}" parent="base_link" />
+  <xacro:wheel name="rear_right" radius="${wheel_radius}" width="${wheel_width}" mass="${wheel_mass}" material="${wheel_material}" x="${rr_x}" y="${rr_y}" z="${rr_z}" parent="base_link" />
   <!-- Include Gazebo Xacro files -->
   <xacro:include filename="$(find mobRobURDF_description)/urdf/gazebo_files/control/gazebo_ros2_control_4w_acker.xacro" />

File: src/mobRobURDF_description/urdf/submodules/4_wheeled/base.xacro (robot description, xacro)
@@ -3,13 +3,14 @@
   <!-- Include the inertial_macros.xacro file -->
   <xacro:include filename="$(find mobRobURDF_description)/urdf/macros/inertial_macros.xacro" />
-  <!-- Base Link -->
-  <link name="base_link"></link>
+  <!-- Base Footprint (ground-projected origin; massless, sits where the wheels touch the ground) -->
+  <link name="base_footprint"></link>
   <!-- Chassis Macro -->
-  <xacro:macro name="chassis" params="size mass material">
+  <xacro:macro name="chassis" params="size mass material wheel_radius">
     <xacro:property name="size_list" value="${list(map(float, size.split()))}" />
     <xacro:property name="l" value="${size_list[0]}" />
     <xacro:property name="w" value="${size_list[1]}" />
     <xacro:property name="h" value="${size_list[2]}" />
-    <link name="chassis">
+    <!-- Base Link (physical robot body / chassis) -->
+    <link name="base_link">
       <inertial>
         <mass value="${mass}" />
@@ -31,9 +32,11 @@
       </collision>
     </link>
-    <!-- Fixed Joint between base_link and chassis -->
-    <joint name="base_to_chassis" type="fixed">
-      <parent link="base_link" />
-      <child link="chassis" />
-      <origin xyz="0 0 ${h/2}" rpy="0 0 0" />
+    <!-- Fixed Joint between base_footprint and base_link.
+         Raised by h/2 + wheel_radius so base_footprint lands exactly at the
+         ground contact point (wheel centres sit at z = wheel_radius). -->
+    <joint name="base_footprint_to_base_link" type="fixed">
+      <parent link="base_footprint" />
+      <child link="base_link" />
+      <origin xyz="0 0 ${h/2 + float(wheel_radius)}" rpy="0 0 0" />
     </joint>
   </xacro:macro>

File: src/mobRobURDF_description/urdf/submodules/4_wheeled/mobRob_4w_diff.xacro (robot description, xacro)
@@ -9,5 +9,5 @@
   <xacro:define_materials/>
   <!-- Define the robot -->
-  <xacro:chassis size="${chassis_size}" mass="${chassis_mass}" material="${chassis_material}" />
+  <xacro:chassis size="${chassis_size}" mass="${chassis_mass}" material="${chassis_material}" wheel_radius="${wheel_radius}" />
   <!-- Wheels -->
   <xacro:wheel name="front_left" radius="${wheel_radius}" width="${wheel_width}" mass="${wheel_mass}" material="${wheel_material}" x="${fl_x}" y="${fl_y}" z="${fl_z}" />

File: src/mobRobURDF_description/urdf/submodules/4_wheeled/mobRob_4w_mec.xacro (robot description, xacro)
@@ -9,5 +9,5 @@
   <xacro:define_materials/>
   <!-- Define the robot -->
-  <xacro:chassis size="${chassis_size}" mass="${chassis_mass}" material="${chassis_material}" />
+  <xacro:chassis size="${chassis_size}" mass="${chassis_mass}" material="${chassis_material}" wheel_radius="${wheel_radius}" />
   <!-- Wheels — sphere collision for reliable mecanum strafing (visual stays a cylinder) -->
   <xacro:wheel name="front_left" radius="${wheel_radius}" width="${wheel_width}" mass="${wheel_mass}" material="${wheel_material}" x="${fl_x}" y="${fl_y}" z="${fl_z}" collision_geom="sphere" />
