Commit message: Changed chassis to base_link and base_link to base_footprint

File: src/mobRobURDF_description/urdf/submodules/4_wheeled/wheels.xacro (robot description, xacro)
@@ -36,5 +36,5 @@
     </link>
     <joint name="${name}_joint" type="continuous">
-      <parent link="chassis" />
+      <parent link="base_link" />
       <child link="${name}_wheel" />
       <origin xyz="${x} ${y} ${z}" rpy="0 0 0" />

Commit message: Fixed the issue with colors not getting applied

File: src/mobRobURDF_description/urdf/gazebo_files/gazebo_colors.xacro (robot description, xacro)
@@ -6,10 +6,23 @@
   <xacro:macro name="gz_link_color" params="link_name color">
     <xacro:property name="_rgba" value="${
-      '0.5  0.5  0.5  1' if color == 'Gray'  else
-      '0.05 0.05 0.05 1' if color == 'Black' else
-      '1.0  0.0  0.0  1' if color == 'Red'   else
-      '0.0  0.2  1.0  1' if color == 'Blue'  else
-      '0.0  0.8  0.0  1' if color == 'Green' else
-      '1.0  1.0  1.0  1'
+      '0.50 0.50 0.50 1' if color == 'Gray'      else
+      '0.75 0.75 0.75 1' if color == 'Silver'    else
+      '0.25 0.25 0.25 1' if color == 'Dark Gray' else
+      '0.05 0.05 0.05 1' if color == 'Black'     else
+      '1.0  1.0  1.0  1' if color == 'White'     else
+      '1.0  0.0  0.0  1' if color == 'Red'       else
+      '0.50 0.00 0.00 1' if color == 'Maroon'    else
+      '1.0  0.50 0.0  1' if color == 'Orange'    else
+      '1.0  1.0  0.0  1' if color == 'Yellow'    else
+      '0.0  0.80 0.0  1' if color == 'Green'     else
+      '0.50 1.0  0.0  1' if color == 'Lime'      else
+      '0.0  0.50 0.50 1' if color == 'Teal'      else
+      '0.0  1.0  1.0  1' if color == 'Cyan'      else
+      '0.0  0.2  1.0  1' if color == 'Blue'      else
+      '0.0  0.0  0.50 1' if color == 'Navy'      else
+      '0.50 0.0  0.50 1' if color == 'Purple'    else
+      '1.0  0.40 0.70 1' if color == 'Pink'      else
+      '0.60 0.30 0.10 1' if color == 'Brown'     else
+      '0.50 0.50 0.50 1'
     }"/>
     <gazebo reference="${link_name}">

File: src/mobRobURDF_description/urdf/mobRob.urdf.xacro (robot description, xacro)
@@ -9,7 +9,10 @@
   <xacro:property name="wheel_mass" value="0.5"/>
   <xacro:property name="wheel_material" value="Dark Gray"/>
-  <xacro:property name="front_x" value="0.6"/>
-  <xacro:property name="front_y" value="0"/>
-  <xacro:property name="front_z" value="-0.15"/>
+  <xacro:property name="fl_x" value="0.4533333333333333"/>
+  <xacro:property name="fl_y" value="0.46"/>
+  <xacro:property name="fl_z" value="-0.15"/>
+  <xacro:property name="fr_x" value="0.4533333333333333"/>
+  <xacro:property name="fr_y" value="-0.46"/>
+  <xacro:property name="fr_z" value="-0.15"/>
   <xacro:property name="rl_x" value="-0.4533333333333333"/>
   <xacro:property name="rl_y" value="0.46"/>
@@ -18,8 +21,8 @@
   <xacro:property name="rr_y" value="-0.46"/>
   <xacro:property name="rr_z" value="-0.15"/>
-  <xacro:property name="controller_type" value="tricycle"/>
+  <xacro:property name="controller_type" value="diff_4w"/>
   <xacro:property name="hardware_plugin" value="gz_ros2_control/GazeboSimSystem"/>
   <xacro:property name="use_gazebo_sim" value="1"/>
-  <xacro:include filename="$(find mobRobURDF_description)/urdf/submodules/3_wheeled/mobRob_3w_tricycle.xacro"/>
+  <xacro:include filename="$(find mobRobURDF_description)/urdf/submodules/4_wheeled/mobRob_4w_diff.xacro"/>
   <xacro:include filename="$(find mobRobURDF_description)/urdf/user_sensors.xacro"/>
 </robot>
